File: Eagle_Files/Extruder_Board1.2.brd (EAGLE design)
At the start: 38.1 x 46.5 mm, 61 parts, among them J1 SFW24R-1STE1LF, U1 ATMEGA48PA-MMHR28M1-L, U2 MCP6001T-I/OTSOT-23-5_MC-L, U3 LM358PWRDFN-8

Commit message: Fixed accidental short of pin to ground
Parts:
- removed GND1: TPTP13SQ, testpad:TP13SQ
- added ⏚: TPTP13SQ, testpad:TP13SQ
- moved 5V 17.5 mm to (12.1, 8.26), flipped to the bottom, turned to 0 degrees
- moved SCK 7.75 mm to (14.0, 6.35), flipped to the bottom, turned to 0 degrees
- moved MISO 5.89 mm to (14.0, 8.26), flipped to the bottom, turned to 0 degrees
- moved MOSI 5.31 mm to (12.1, 6.35), flipped to the bottom, turned to 0 degrees
- moved RST 1.47 mm to (14.0, 4.45), flipped to the bottom
Connections:
- net +5V: no longer 5V.TP
- net GAIN_FB: now also R2.1
- net GND: now also ⏚.TP; no longer GND1.TP, R2.1
- net VCC_REG: now also 5V.TP
Routing:
- net RST: track 13.2 -> 59.5 mm, vias 1 -> 3
- net SPI_MOSI: track 0.00 -> 25.8 mm, vias 0 -> 3
- net SPI_SCK: track 0.00 -> 25.7 mm, vias 0 -> 3
- net VCC_REG: track 8.23 -> 31.7 mm, vias 0 -> 1
- net SPI_MISO: track 0.00 -> 22.8 mm, vias 0 -> 3
- net GAIN_FB: track 1.34 -> 13.0 mm, vias 0 -> 3
- net TRG_LED: track 49.9 -> 51.2 mm
