File: Eagle_Files/Extruder_Board1.2.sch (EAGLE design)
At the start: 60 parts, among them J1 SFW24R-1STE1LF, U1 ATMEGA48PA-MMHR28M1-L, U2 MCP6001T-I/OTSOT-23-5_MC-L, U3 LM358PWRDFN-8

Commit message: Fixed accidental short of pin to ground
Parts:
- renumbered GND1 to ⏚
Connections:
- net +5V: no longer 5V.TP
- net GAIN_FB: now also R2.1
- net GND: no longer R2.1
- net VCC_REG: now also 5V.TP
Other:
- moved on the sheet: R17
Changed lines of the file:
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@@
 <setting verticaltext="up"/>
 </settings>
-<grid distance="1.27" unitdist="mm" unit="mm" style="lines" multiple="1" display="no" altdistance="0.127" altunitdist="mm" altunit="mm"/>
+<grid distance="1.27" unitdist="mm" unit="mm" style="lines" multiple="1" display="no" altdistance="0.01" altunitdist="inch" altunit="mm"/>
 <layers>
 <layer number="1" name="Top" color="4" fill="1" visible="no" active="no"/>
@@
 <part name="R17" library="PiezoFFC" library_urn="urn:adsk.eagle:library:6897166" deviceset="SMD-RES-0R-5%-1/16W(0402)" device="" package3d_urn="urn:adsk.eagle:package:7115182/2" value="3.3K"/>
 <part name="R19" library="PiezoFFC" library_urn="urn:adsk.eagle:library:6897166" deviceset="SMD-RES-0R-5%-1/16W(0402)" device="" package3d_urn="urn:adsk.eagle:package:7115182/2" value="1M"/>
-<part name="GND1" library="testpad" library_urn="urn:adsk.eagle:library:385" deviceset="TP" device="TP13SQ" package3d_urn="urn:adsk.eagle:package:27974/1" value="TPTP13SQ"/>
+<part name="⏚" library="testpad" library_urn="urn:adsk.eagle:library:385" deviceset="TP" device="TP13SQ" package3d_urn="urn:adsk.eagle:package:27974/1" value="TPTP13SQ"/>
 </parts>
 <sheets>
@@
 <attribute name="VALUE" x="194.945" y="177.165" size="1.778" layer="96"/>
 </instance>
-<instance part="R17" gate="G$1" x="199.39" y="195.58" smashed="yes" rot="R90">
-<attribute name="NAME" x="199.39" y="191.77" size="1.27" layer="95" ratio="10" rot="R90"/>
-<attribute name="VALUE" x="201.93" y="191.77" size="1.27" layer="96" ratio="10" rot="R90"/>
+<instance part="R17" gate="G$1" x="199.39" y="190.5" smashed="yes" rot="R90">
+<attribute name="NAME" x="199.39" y="186.69" size="1.27" layer="95" ratio="10" rot="R90"/>
+<attribute name="VALUE" x="201.93" y="186.69" size="1.27" layer="96" ratio="10" rot="R90"/>
 </instance>
 <instance part="R19" gate="G$1" x="191.77" y="204.47" smashed="yes" rot="R90">
@@
 <attribute name="VALUE" x="193.04" y="205.74" size="1.27" layer="96" ratio="10" rot="R90"/>
 </instance>
-<instance part="GND1" gate="G$1" x="238.76" y="123.19" smashed="yes" rot="R270">
+<instance part="⏚" gate="G$1" x="238.76" y="123.19" smashed="yes" rot="R270">
 <attribute name="NAME" x="240.03" y="123.19" size="1.778" layer="95"/>
 <attribute name="TP_SIGNAL_NAME" x="237.49" y="121.92" size="1.778" layer="97" rot="R270"/>
@@
 <wire x1="215.9" y1="100.33" x2="215.9" y2="102.87" width="0.1524" layer="91"/>
 <wire x1="215.9" y1="102.87" x2="238.76" y2="102.87" width="0.1524" layer="91"/>
-<pinref part="GND1" gate="G$1" pin="TP"/>
+<pinref part="⏚" gate="G$1" pin="TP"/>
 <wire x1="236.22" y1="123.19" x2="215.9" y2="123.19" width="0.1524" layer="91"/>
 <wire x1="215.9" y1="123.19" x2="215.9" y2="102.87" width="0.1524" layer="91"/>
@@
 <wire x1="196.85" y1="200.66" x2="196.85" y2="198.12" width="0.1524" layer="91"/>
 <junction x="196.85" y="184.15"/>
-<pinref part="R17" gate="G$1" pin="1"/>
-<pinref part="R2" gate="G$1" pin="1"/>
 <wire x1="196.85" y1="198.12" x2="196.85" y2="184.15" width="0.1524" layer="91"/>
-<wire x1="199.39" y1="191.77" x2="199.39" y2="189.23" width="0.1524" layer="91"/>
-<wire x1="199.39" y1="189.23" x2="212.09" y2="189.23" width="0.1524" layer="91"/>
-<pinref part="U2" gate="A" pin="VSS"/>
-<wire x1="212.09" y1="189.23" x2="213.36" y2="189.23" width="0.1524" layer="91"/>
-<wire x1="212.09" y1="193.04" x2="212.09" y2="189.23" width="0.1524" layer="91"/>
-<junction x="212.09" y="189.23"/>
-<wire x1="196.85" y1="184.15" x2="212.09" y2="184.15" width="0.1524" layer="91"/>
-<wire x1="212.09" y1="184.15" x2="212.09" y2="189.23" width="0.1524" layer="91"/>
+<wire x1="196.85" y1="184.15" x2="199.39" y2="184.15" width="0.1524" layer="91"/>
 <pinref part="D8" gate="G$1" pin="A"/>
+<wire x1="199.39" y1="184.15" x2="212.09" y2="184.15" width="0.1524" layer="91"/>
 <wire x1="181.61" y1="214.63" x2="182.88" y2="214.63" width="0.1524" layer="91"/>
 <wire x1="181.61" y1="205.74" x2="181.61" y2="214.63" width="0.1524" layer="91"/>
@@
 <wire x1="191.77" y1="198.12" x2="196.85" y2="198.12" width="0.1524" layer="91"/>
 <junction x="196.85" y="198.12"/>
+<pinref part="R17" gate="G$1" pin="1"/>
+<wire x1="199.39" y1="186.69" x2="199.39" y2="184.15" width="0.1524" layer="91"/>
+<junction x="199.39" y="184.15"/>
+<pinref part="U2" gate="A" pin="VSS"/>
+<wire x1="212.09" y1="193.04" x2="212.09" y2="184.15" width="0.1524" layer="91"/>
 </segment>
 </net>
@@
 <junction x="60.96" y="130.81"/>
 </segment>
+<segment>
+<pinref part="5V" gate="G$1" pin="TP"/>
+<wire x1="236.22" y1="125.73" x2="224.79" y2="125.73" width="0.1524" layer="91"/>
+<label x="223.52" y="125.73" size="1.778" layer="95"/>
+</segment>
 </net>
 <net name="E0_1B" class="0">
@@
 <wire x1="238.76" y1="100.33" x2="218.44" y2="100.33" width="0.1524" layer="91"/>
 <label x="228.6" y="100.33" size="1.778" layer="95"/>
-<pinref part="5V" gate="G$1" pin="TP"/>
-<label x="228.6" y="125.73" size="1.778" layer="95"/>
 <pinref part="P+8" gate="1" pin="+5V"/>
-<wire x1="236.22" y1="125.73" x2="218.44" y2="125.73" width="0.1524" layer="91"/>
-<wire x1="218.44" y1="125.73" x2="218.44" y2="139.7" width="0.1524" layer="91"/>
-<wire x1="218.44" y1="100.33" x2="218.44" y2="125.73" width="0.1524" layer="91"/>
-<junction x="218.44" y="125.73"/>
+<wire x1="218.44" y1="100.33" x2="218.44" y2="139.7" width="0.1524" layer="91"/>
 </segment>
 <segment>
@@
 <pinref part="R17" gate="G$1" pin="2"/>
 <pinref part="U2" gate="A" pin="VIN-"/>
-<wire x1="199.39" y1="199.39" x2="199.39" y2="200.66" width="0.1524" layer="91"/>
-</segment>
-</net>
+<wire x1="199.39" y1="194.31" x2="199.39" y2="195.58" width="0.1524" layer="91"/>
+<pinref part="R2" gate="G$1" pin="1"/>
+<wire x1="199.39" y1="195.58" x2="199.39" y2="200.66" width="0.1524" layer="91"/>
+<wire x1="213.36" y1="189.23" x2="201.93" y2="189.23" width="0.1524" layer="91"/>
+<wire x1="201.93" y1="189.23" x2="201.93" y2="195.58" width="0.1524" layer="91"/>
+<wire x1="201.93" y1="195.58" x2="199.39" y2="195.58" width="0.1524" layer="91"/>
+<junction x="199.39" y="195.58"/>
+</segment>
+</net>
