File: Eagle_Files/Extruder_Board_programmer.brd (EAGLE design)
At the start: 39.6 x 46.5 mm, 21 parts, among them J1 10118192-0001LF, U1 CP2102N-A01-GQFN20

Commit message: Adjusted trace placement, added logo to bottom of board
Parts:
- added U$2: (no value), PiezoFFC:LOGO-PYR0BALL-SS-20MM
Routing:
- net 5V_DC: track 67.0 -> 67.7 mm
Changed lines of the file:
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@@
 <attribute name="NAME" x="4.1825" y="17.6345" size="0.8128" layer="25" font="vector" rot="R90" align="top-left"/>
 </element>
+<element name="U$2" library="PiezoFFC" library_urn="urn:adsk.eagle:library:6897166" package="LOGO-PYR0BALL-SS-20MM" package3d_urn="urn:adsk.eagle:package:5522046/1" value="" x="12.413" y="33.9525" smashed="yes" rot="MR270"/>
 </elements>
 <signals>
@@
 <wire x1="33.052465625" y1="33.304034375" x2="33.0844625" y2="33.304034375" width="0.1524" layer="1"/>
 <wire x1="25.887459375" y1="22.47310625" x2="25.604875" y2="22.190521875" width="0.1524" layer="1"/>
-<wire x1="25.604875" y1="22.190521875" x2="24.486396875" y2="22.190521875" width="0.1524" layer="1"/>
-<wire x1="24.486396875" y1="22.190521875" x2="23.244" y2="20.948125" width="0.1524" layer="1"/>
+<wire x1="25.604875" y1="22.190521875" x2="23.343396875" y2="22.190521875" width="0.1524" layer="1"/>
+<wire x1="23.343396875" y1="22.190521875" x2="23.244" y2="22.091125" width="0.1524" layer="1"/>
 <wire x1="23.241903125" y1="18.257503125" x2="23.241903125" y2="20.884625" width="0.4064" layer="1"/>
 <contactref element="R1" pad="2"/>
 <wire x1="23.244" y1="20.4655" x2="23.244" y2="20.884625" width="0.1524" layer="1"/>
-<wire x1="23.244" y1="20.884625" x2="23.244" y2="20.948125" width="0.1524" layer="1"/>
+<wire x1="23.244" y1="20.884625" x2="23.244" y2="22.091125" width="0.1524" layer="1"/>
 <wire x1="20" y1="15.0156" x2="20" y2="14" width="0.4064" layer="1"/>
 <wire x1="20" y1="15.0156" x2="23.241903125" y2="18.257503125" width="0.4064" layer="1"/>
@@
 <wire x1="15.55" y1="21.25" x2="16.723" y2="21.25" width="0.1524" layer="16"/>
 <wire x1="16.723" y1="21.25" x2="21.0185" y2="16.9545" width="0.1524" layer="16"/>
-<wire x1="24.437890625" y1="21.0235375" x2="24.437890625" y2="18.739309375" width="0.1524" layer="1"/>
+<wire x1="24.437890625" y1="21.0235375" x2="24.247390625" y2="20.8330375" width="0.1524" layer="1"/>
+<wire x1="24.247390625" y1="20.8330375" x2="24.247390625" y2="18.548809375" width="0.1524" layer="1"/>
 <wire x1="21.0185" y1="15.31991875" x2="21.0185" y2="14.2875" width="0.1524" layer="1"/>
-<wire x1="24.437890625" y1="18.739309375" x2="21.0185" y2="15.31991875" width="0.1524" layer="1"/>
+<wire x1="24.247390625" y1="18.548809375" x2="21.0185" y2="15.31991875" width="0.1524" layer="1"/>
 <wire x1="22.209878125" y1="12.68488125" x2="22.209878125" y2="12.684878125" width="0" layer="19" extent="1-1"/>
 </signal>
