File: Eagle_Files/AVR_Board_programmer.brd (EAGLE design)
At the start: 39.6 x 46.5 mm, 22 parts, among them J1 10118192-0001LF, U1 CP2102N-A01-GQFN20

Commit message: Renamed boards, Fixed programmer
 - Renamed boards to more closely match change in spec/design revision
 - Added required components to usb serial board stack
   - Fixes https://github.com/pyr0ball/pyr0piezo/issues/9
 - Minor change to voltage values to stay consistent with local tests
Parts:
- added C1, C2: 0.1uF, PiezoFFC:CAPC1005X50
- added R4: 10K, PiezoFFC:R0402
- U1: value CP2102N-A01-GQFN20 -> CP2102N-A01-GQFN28; device PiezoFFC:SILABS_QFN20 -> PiezoFFC:QFN50P500X500X80-29N
- moved U$2 10.1 mm to (14.4, 24.0), turned to 180 degrees
- moved U1 2.16 mm to (14.4, 24.1), turned to 45 degrees
Connections:
- new net PGM_RST: C1.2, R4.2, U1.28
- net 5V_DC: now also C2.2
- net GND: now also C2.1, U1.29; no longer U1.12, U1.21
- net RST: now also C1.1
- net RXD: now also U1.26; no longer U1.18
- net TXD: now also U1.25; no longer U1.17
- net TXT: now also U1.18; no longer U1.20
- net VBUS: now also R4.1
Routing:
- net RST: track 8.10 -> 29.0 mm
- net TXT: track 27.0 -> 36.2 mm
- net RXT: track 26.3 -> 31.6 mm
- net GND: track 3.51 -> 0.00 mm
- net VBUS: track 17.4 -> 20.3 mm, vias 0 -> 1
- net TXD: track 48.3 -> 45.8 mm
- net RXD: track 42.7 -> 40.6 mm
- net PGM_RST: track 0.00 -> 1.04 mm
- net 5V_DC: track 67.7 -> 68.3 mm

Commit message: Added ICSP Header/breakout to programmer
Also added secondary footprint for alternate TVS Diode
(ESD protection component) that's about 1/10th the cost
of the one currently used (suggested by the UART Bridge's
Datasheet.
Parts:
- added D2: TVS_DIODE_CM1293A, PiezoFFC:SC-74-6
- added ICSP0: ICSP_HEADERICSP-2MM, PiezoFFC:HDRV6W50P200_3X2_400X600X550B
- added ICSP1: ICSP_HEADERICSP_2.54MM_RIGHT, PiezoFFC:HDRRA6W64P254_2X3_762X254X508B
Connections:
- new net SPI_MISO: ICSP0.5, ICSP1.6
- new net SPI_MOSI: ICSP0.3, ICSP1.2
- new net SPI_SCK: ICSP0.4, ICSP1.5
- net 5V_DC: now also D2.5
- net D+: now also D2.3
- net D-: now also D2.1
- net GND: now also D2.2, ICSP0.2, ICSP1.3
- net RST: now also ICSP0.1, ICSP1.4
- net VBUS: now also ICSP0.6, ICSP1.1
Routing:
- net RST: track 29.0 -> 64.5 mm
- net VBUS: track 20.3 -> 46.1 mm
- net SPI_MISO: track 0.00 -> 13.1 mm
- net SPI_SCK: track 0.00 -> 12.9 mm
- net SPI_MOSI: track 0.00 -> 12.5 mm
- net D-: track 19.8 -> 24.7 mm
- net D+: track 18.5 -> 22.7 mm
- net 5V_DC: track 68.3 -> 71.1 mm, vias 1 -> 2

Commit message: Fixed airwires and overlaps caused by swapping IC
Reminder to always do a DRC after changin BOM!
Routing:
- net PGM_RST: track 1.04 -> 6.87 mm, vias 0 -> 1
- net GND: track 0.00 -> 2.57 mm
- net D-: track 24.7 -> 25.3 mm
- net VBUS: track 46.1 -> 46.7 mm
- net 5V_DC: vias 2 -> 3
