File: Eagle_Files/AVR_Board_programmer1.0.1.brd (EAGLE design)
At the start: 39.6 x 46.5 mm, 29 parts, among them J1 10118192-0001LF, U1 CP2102N-A01-GQFN28

Commit message: added ICSP header for standalone units
Parts:
- added C3: 0.1uF, PiezoFFC:CAPC1005X50
- added C4, C5: 4.7uF, PiezoFFC:CAPC2012X130
- added D3: ZENER_DIODE_PLZ5V1C, PiezoFFC:DO-219AC
- added R5: 10K, PiezoFFC:R0402
- moved ICSP2 37.7 mm to (19.6, 24.6), flipped to the bottom, turned to 135 degrees
- moved U$1 5.39 mm to (16.4, 33.0)
- moved C2 4.12 mm to (12.4, 18.9), turned to 135 degrees
- moved D1 2.83 mm to (27.8, 19.1)
- moved ICSP1 2.20 mm to (2.81, 15.6), flipped to the bottom
- moved ICSP0 2.00 mm to (13.9, 4.55), flipped to the bottom
Connections:
- removed net VBUS: ICSP0.6, ICSP1.1, ICSP2.6, R1.1, R2.2, R4.1, TTL.5, U1.8
- new net N$1: C2.2, C5.1, R1.1, R2.2, U1.8
- new net RST_PULLUP: R5.1, U1.9
- net 5V_DC: now also C3.2, C4.1, D3.P$2, ICSP0.6, ICSP1.1, ICSP2.6, R4.1, TTL.5; no longer C2.2
- net GND: now also C3.1, C4.2, C5.2, D3.P$1
- net VDD: now also R5.2
Routing:
- net VBUS: track 46.7 -> 0.00 mm, vias 1 -> 0
- net SPI_MOSI: track 12.5 -> 36.0 mm, vias 0 -> 2
- net 5V_DC: track 71.1 -> 93.7 mm
- net SPI_MISO: track 13.1 -> 33.4 mm, vias 0 -> 1
- net SPI_SCK: track 12.9 -> 31.8 mm, vias 0 -> 1
- net N$1: track 0.00 -> 5.69 mm
- net RST: track 64.5 -> 60.0 mm, vias 0 -> 1
- net VDD: track 0.00 -> 3.76 mm, vias 0 -> 1
- net RST_PULLUP: track 0.00 -> 1.92 mm, vias 0 -> 1
- net D+: track 22.7 -> 23.8 mm
- net PGM_RST: track 6.87 -> 5.73 mm
Other:
- board text added: "+5V"
- board text added: "MISO"
- board text added: "MOSI"
- board text added: "RST"
- board text added: "SCK"
- board text added: "⏚"

Commit message: moved usb to bottom of board, fixed caps
Decoupling capacitors were connected on
the wrong voltage regulation input
Parts:
- moved ICSP1 2.54 mm to (5.35, 15.6), flipped to the top
- moved C4 0.41 mm to (17.1, 18.4)
- flipped D3 to the bottom, turned to 180 degrees
- flipped J1 to the bottom, turned to 315 degrees
Connections:
- net N$2 renamed PWR_IND
- removed net N$1: C2.2, C5.1, R1.1, R2.2, U1.8
- new net VBUS: R1.1, R2.2, U1.8
- net VDD: now also C2.2, C5.1
Routing:
- net VDD: track 3.76 -> 9.53 mm, vias 1 -> 2
- net N$1: track 5.69 -> 0.00 mm
- net SPI_SCK: track 31.8 -> 36.2 mm
- net VBUS: track 0.00 -> 3.31 mm
- net D-: track 25.1 -> 22.1 mm, vias 1 -> 2
- net SPI_MISO: track 33.4 -> 35.6 mm
- net SPI_MOSI: track 36.0 -> 34.0 mm
- net RST: track 60.0 -> 61.9 mm, vias 1 -> 2
- net D+: track 23.8 -> 22.5 mm, vias 1 -> 2
- net 5V_DC: track 93.7 -> 94.3 mm, vias 3 -> 5
Other:
- board text added: "RXD"
- board text added: "TXD"

Commit message: Optimized trace layout, serpentined usb
Parts:
- removed D1: SP0503BAHTG, PiezoFFC:SOT143
- removed U$2: (no value), PiezoFFC:LOGO-PYR0BALL-SS-20MM
- +5V, GND, RST., RXD, TXD: value TP -> TPSPRING_CONTACT_3.5X1.1; device PiezoFFC:TP13SQ-HOLE -> PiezoFFC:SPRING_CONTACT_3.48X1.10
- ICSP0, ICSP2: value ICSP_HEADERICSP-2MM -> ICSP_HEADERSPRING_3.48X1.1; device PiezoFFC:HDRV6W50P200_3X2_400X600X550B -> PiezoFFC:ICSP_3X2_3.48X1.1_SPRING_CONTACTS
- ICSP1: device PiezoFFC:HDRRA6W64P254_2X3_762X254X508B -> PiezoFFC:ICSP_2X3_2.54_RIGHT
- moved ICSP0 2.00 mm to (11.9, 4.55), flipped to the top
- moved ICSP2 1.98 mm to (20.8, 26.1), flipped to the top, turned to 225 degrees
- moved R8 0.18 mm to (33.5, 33.1)
- flipped +5V to the top, turned to 225 degrees
- flipped GND to the top, turned to 225 degrees
- flipped RST. to the top, turned to 225 degrees
- flipped RXD to the top, turned to 225 degrees
- flipped TXD to the top, turned to 225 degrees
Connections:
- net 5V_DC: now also +5V.TH, ICSP0.5, ICSP0.P$5, ICSP2.5, ICSP2.P$5; no longer D1.2, ICSP0.6, ICSP2.6
- net D+: no longer D1.4
- net D-: no longer D1.3
- net GND: now also GND.TH, ICSP0.1, ICSP0.P$1, ICSP2.1, ICSP2.P$1; no longer D1.1, ICSP0.2, ICSP2.2
- net RST: now also ICSP0.2, ICSP0.P$2, ICSP2.2, ICSP2.P$2, RST..TH; no longer ICSP0.1, ICSP2.1
- net RXD: now also RXD.TH
- net SPI_MISO: now also ICSP0.6, ICSP0.P$6, ICSP2.6, ICSP2.P$6; no longer ICSP0.5, ICSP2.5
- net SPI_MOSI: now also ICSP0.4, ICSP0.P$4, ICSP2.4, ICSP2.P$4; no longer ICSP0.3, ICSP2.3
- net SPI_SCK: now also ICSP0.3, ICSP0.P$3, ICSP2.3, ICSP2.P$3; no longer ICSP0.4, ICSP2.4
- net TXD: now also TXD.TH
Routing:
- net D+: track 22.5 -> 15.0 mm
- net 5V_DC: track 94.3 -> 87.5 mm, vias 5 -> 3
- net D-: track 22.1 -> 17.2 mm, vias 2 -> 0
- net SPI_SCK: track 36.2 -> 36.9 mm, vias 1 -> 0
- net VDD: track 9.53 -> 8.88 mm
- net SPI_MISO: track 35.6 -> 36.1 mm
- net RST: track 61.9 -> 62.3 mm, vias 2 -> 1
- net SPI_MOSI: track 34.0 -> 34.4 mm, vias 2 -> 1
Other:
- board text removed: "- +"
