File: Eagle_Files/AVR_Board_programmer1.0.1.sch (EAGLE design)
At the start: 27 parts, among them J1 10118192-0001LF, U1 CP2102N-A01-GQFN28

Commit message: added ICSP header for standalone units
Parts:
- added C3: 0.1uF, PiezoFFC:CERAMIC-1NF-50V-10%-X7R(0402)CAP_0402
- added C4, C5: 4.7uF, PiezoFFC:SEEED-CAPACITOR_CERAMIC-10UF-25V-10%-X5R(0805)CAP_0805-3D
- added D3: ZENER_DIODE_PLZ5V1C, PiezoFFC:ZENER_DIODE_PLZ5V1C
- added R5: 10K, PiezoFFC:SMD-RES-0R-5%-1/16W(0402)
Connections:
- removed net VBUS: ICSP0.VCC, ICSP1.VCC, ICSP2.VCC, R1.1, R2.2, R4.1, TTL.P$5, U1.VBUS
- new net N$1: C2.2, C5.1, R1.1, R2.2, U1.VBUS
- new net RST_PULLUP: R5.1, U1.!RST
- new net VDD: R5.2, U1.VDD
- net 5V_DC: now also C3.2, C4.1, D3.C, ICSP0.VCC, ICSP1.VCC, ICSP2.VCC, R4.1, TTL.P$5; no longer C2.2
- net GND: now also C3.1, C4.2, C5.2, D3.A
Other:
- moved on the sheet: R2

Commit message: moved usb to bottom of board, fixed caps
Decoupling capacitors were connected on
the wrong voltage regulation input
Connections:
- net N$2 renamed PWR_IND
- removed net N$1: C2.2, C5.1, R1.1, R2.2, U1.VBUS
- new net VBUS: R1.1, R2.2, U1.VBUS
- net VDD: now also C2.2, C5.1

Commit message: Optimized trace layout, serpentined usb
Parts:
- removed D1: SP0503BAHTG, PiezoFFC:SP0503BAHTG
- +5V, GND, RST., RXD, TXD: value TP -> TPSPRING_CONTACT_3.5X1.1; device PiezoFFC:TP -> PiezoFFC:TPSPRING_CONTACT_3.5X1.1
- ICSP0, ICSP2: value ICSP_HEADERICSP-2MM -> ICSP_HEADERSPRING_3.48X1.1; device PiezoFFC:ICSP_HEADERICSP-2MM -> PiezoFFC:ICSP_HEADERSPRING_3.48X1.1
Connections:
- net 5V_DC: no longer D1.2
- net D+: no longer D1.4
- net D-: no longer D1.3
- net GND: no longer D1.1
