File: Eagle_Files/PiezoStandalone1.1.brd (EAGLE design)
At the start: 42.9 x 15.4 mm, 48 parts, among them J1 CON-MOLEX-3P-1.25MM048, U1 ATMEGA48PA-MMHR28M1-L, U2 L78L05ACU, U3 LM2902LM2902QT

Commit message: v1.1 Piezo Standalone board
 - Added overvolt/overcurrent protection
via zener diode and fuse
 - Swapped LM358 dual channel opamp + MCP6001 Single Channel opamp for LM2902 Quad Channel.
 - Added jumper to bypass Vreg for < 6V input
Parts:
- added D1: ZENER_DIODE_PLZ5V1C, PiezoFFC:DO-219AC
- added F1: 500mA, PiezoFFC:R0402
- added SJ1: (no value), PiezoFFC:SJM
- moved U$1 5.71 mm to (23.5, 5.08)
- moved U$2 3.02 mm to (13.6, 9.59), turned to 45 degrees
- moved U2 0.64 mm to (11.1, 4.22)
- moved R16 0.13 mm to (15.6, 8.84)
Connections:
- new net VCC_FUSE: F1.2, SJ1.1, U2.3
- net +5V: now also D1.P$2, SJ1.2
- net GND: now also D1.P$1
- net VCC_REG: now also F1.1; no longer U2.3
Routing:
- net VCC_FUSE: track 0.00 -> 2.84 mm, vias 0 -> 1
- net +5V: track 57.1 -> 59.2 mm
- net VCC_REG: track 7.17 -> 5.58 mm
Other:
- board text added: "+ -"
- board text removed: "- +"

Commit message: Added missing 0.1uF cap on AVR Vcc
Parts:
- added C4: 0.1uF, PiezoFFC:CAPC1005X50
Connections:
- net +5V: now also C4.2
- net GND: now also C4.1
Changed lines of the file:
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@@
 <attribute name="NAME" x="12.34265625" y="8.6777125" size="0.6096" layer="26" font="vector" ratio="11" rot="MR225"/>
+</element>
+<element name="C4" library="PiezoFFC" library_urn="urn:adsk.eagle:library:6897166" package="CAPC1005X50" package3d_urn="urn:adsk.eagle:package:5248669/4" value="0.1uF" x="24.765" y="2.7305" smashed="yes" rot="MR90">
+<attribute name="NAME" x="24.765" y="3.6294" size="0.6096" layer="26" font="vector" ratio="11" rot="MR0" align="bottom-center"/>
 </element>
 </elements>
@@
 <via x="11.722309375" y="8.846896875" extent="1-16" drill="0.3"/>
 <via x="18" y="5.925" extent="1-16" drill="0.3"/>
-<via x="9.876815625" y="2.81019375" extent="1-16" drill="0.3"/>
+<via x="11.146815625" y="6.30269375" extent="1-16" drill="0.3"/>
 <via x="17.970796875" y="4.338" extent="1-16" drill="0.3"/>
 <contactref element="C1" pad="1"/>
@@
 <wire x1="26.42" y1="5.965" x2="26.67" y2="5.715" width="0.1524" layer="1"/>
 <contactref element="D1" pad="P$1"/>
+<contactref element="C4" pad="1"/>
 </signal>
 <signal name="Z_MIN_TRIG">
@@
 <wire x1="12.1702125" y1="7.1337875" x2="12.26315" y2="7.04085" width="0.4064" layer="16"/>
 <wire x1="12.26315" y1="7.04085" x2="12.26315" y2="6.151853125" width="0.4064" layer="16"/>
+<contactref element="C4" pad="2"/>
+<wire x1="24.7515" y1="3.253" x2="24.765" y2="3.2305" width="0" layer="19" extent="1-16"/>
 </signal>
 <signal name="GAIN_FB">

Commit message: fixed footprint for LM2902, optimized traces
Parts:
- J1: value CON-MOLEX-3P-1.25MM048 -> CON-MOLEX-4P-1.25MM048; device PiezoFFC:53048-03 -> PiezoFFC:53048-04
- R2: value 3.3K -> 3K3
- U3: value LM2902LM2902QT -> LM2902QT; device PiezoFFC:QFN50P300X300X100-17N -> PiezoFFC:QFN16
- moved R10 6.04 mm to (26.7, 9.21), turned to 90 degrees
- moved R5 6.02 mm to (26.7, 8.37), turned to 270 degrees
- moved R15 1.08 mm to (21.3, 9.28)
- moved D8 1.00 mm to (32.9, 7.19)
Connections:
- net GND: no longer U3.17
- net V_FOLLOW: now also U3.13, U3.14; no longer U3.5, U3.6
- net V_FOLLOW_DIV: now also U3.12; no longer U3.4
Routing:
- net V_FOLLOW: track 8.99 -> 7.07 mm
- net Z_TRG: track 5.85 -> 7.01 mm
- net PZ+: track 11.1 -> 10.0 mm
- net +5V: track 59.2 -> 60.2 mm
- net VCC_REG: track 5.58 -> 6.32 mm
- net Z_MIN_TRIG: track 18.5 -> 19.1 mm
- net PZ_AMP_OUT: track 6.78 -> 6.23 mm
- net GND: track 6.65 -> 6.53 mm, vias 24 -> 25
