File: Eagle_Files/PiezoStandalone_PT100_1.1.1.brd (EAGLE design)
At the start: 42.9 x 15.4 mm, 69 parts, among them J1 CON-MOLEX-4P-1.25MM048, U1 ATMEGA48PA-MMHR28M1-L, U2 L78L05ACU, U3 LM2902QT

Commit message: Added labels to controller connector
Parts:
- moved J2 28.3 mm to (26.5, 6.95), flipped to the bottom, turned to 180 degrees
Routing:
- net PT100_OUT: track 0.00 -> 30.2 mm, vias 0 -> 3
- net PT100_JUMP: track 0.00 -> 1.02 mm
- net GAIN_OUT: track 9.33 -> 9.95 mm
- net GND: vias 26 -> 28
Other:
- board text added: "PTC"
- board text added: "Vcc"
- board text added: "Z"
- board text added: "⏚"

Commit message: Fixed airwires and overlaps
Routing:
- net PZ+: track 8.66 -> 11.8 mm
- net PT_IN-: track 5.35 -> 6.87 mm
- net PT100_JUMP: track 1.02 -> 1.74 mm

Commit message: Fixed spacing for zener diode
Parts:
- moved D1 0.30 mm to (14.2, 7.68)
- moved R16 0.19 mm to (15.7, 8.94)

Commit message: Gave some extra space to zener diode
related to https://github.com/pyr0ball/pyr0piezo/issues/12
Parts:
- moved D1 0.45 mm to (14.2, 8.13)
- moved R11 0.22 mm to (14.5, 5.06)
Changed lines of the file:
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@@
 </layers>
 <board>
-<fusionsync huburn="a.cGVyc29uYWw6dWUyYTEyMDdh" projecturn="a.cGVyc29uYWw6dWUyYTEyMDdhIzIwMTgxMTI5MTYyOTY3NjMx" f3durn="urn:adsk.wipprod:dm.lineage:nsLuw-r7TDSCqnqJ3mJIQg" pcbguid="3bd29ec8-00c9-4374-8a01-bcbe035150bd" lastpulledtime="" lastsyncedchangeguid="a4ad0e1a-098f-745d-9187-822f9d61ba5b"/>
+<fusionsync huburn="a.cGVyc29uYWw6dWUyYTEyMDdh" projecturn="a.cGVyc29uYWw6dWUyYTEyMDdhIzIwMTgxMTI5MTYyOTY3NjMx" f3durn="urn:adsk.wipprod:dm.lineage:nsLuw-r7TDSCqnqJ3mJIQg" pcbguid="3bd29ec8-00c9-4374-8a01-bcbe035150bd" lastpulledtime="" lastsyncedchangeguid="c40632c8-a1ac-543f-1eb5-0abfdd09adff"/>
 <plain>
 <text x="34.715253125" y="10.10183125" size="1.27" layer="22" ratio="11" rot="R180">+  -</text>
@@
 <attribute name="VALUE" x="22.066" y="3.6055" size="0.4064" layer="27" font="vector" ratio="11"/>
 </element>
-<element name="R11" library="PiezoFFC" library_urn="urn:adsk.eagle:library:6897166" package="R0402" package3d_urn="urn:adsk.eagle:package:7115182/2" value="220R" x="14.51" y="5.284" smashed="yes" rot="R270">
-<attribute name="MPN" value="RC0402JR-070RL" x="14.51" y="5.284" size="1.778" layer="27" rot="R270" display="off"/>
-<attribute name="NAME" x="13.5575" y="5.6015" size="0.6096" layer="25" font="vector" ratio="11" rot="R180"/>
-<attribute name="VALUE" x="15.145" y="4.903" size="0.4064" layer="27" font="vector" ratio="11" rot="R180"/>
+<element name="R11" library="PiezoFFC" library_urn="urn:adsk.eagle:library:6897166" package="R0402" package3d_urn="urn:adsk.eagle:package:7115182/2" value="220R" x="14.51" y="5.06175" smashed="yes" rot="R270">
+<attribute name="MPN" value="RC0402JR-070RL" x="14.51" y="5.06175" size="1.778" layer="27" rot="R270" display="off"/>
+<attribute name="NAME" x="13.5575" y="5.37925" size="0.6096" layer="25" font="vector" ratio="11" rot="R180"/>
+<attribute name="VALUE" x="15.145" y="4.68075" size="0.4064" layer="27" font="vector" ratio="11" rot="R180"/>
 </element>
 <element name="R12" library="PiezoFFC" library_urn="urn:adsk.eagle:library:6897166" package="R0402" package3d_urn="urn:adsk.eagle:package:7115182/2" value="330R" x="14.51" y="4.1405" smashed="yes" rot="R270">
@@
 <element name="U$1" library="PiezoFFC" library_urn="urn:adsk.eagle:library:6897166" package="LOGO-PYR0BALL-SS-6MM" value="" x="23.495" y="5.08" smashed="yes" rot="MR0"/>
 <element name="U$2" library="PiezoFFC" library_urn="urn:adsk.eagle:library:6897166" package="LOGO-PYR0BALL-SS-6MM" value="" x="13.589" y="9.5885" smashed="yes" rot="R45"/>
-<element name="D1" library="PiezoFFC" library_urn="urn:adsk.eagle:library:6897166" package="DO-219AC" package3d_urn="urn:adsk.eagle:package:8452796/2" value="ZENER_DIODE_PLZ5V1C" x="14.19225" y="7.6835" smashed="yes" rot="R270"/>
+<element name="D1" library="PiezoFFC" library_urn="urn:adsk.eagle:library:6897166" package="DO-219AC" package3d_urn="urn:adsk.eagle:package:8452796/2" value="ZENER_DIODE_PLZ5V1C" x="14.1605" y="8.128" smashed="yes" rot="R270"/>
 <element name="F1" library="PiezoFFC" library_urn="urn:adsk.eagle:library:6897166" package="R0402" package3d_urn="urn:adsk.eagle:package:7115182/2" value="500mA" x="10.668" y="8.001" smashed="yes" rot="R90">
 <attribute name="MPN" value="RC0402JR-070RL" x="4.953" y="3.556" size="1.778" layer="27" rot="R90" display="off"/>
@@
 <contactref element="D1" pad="P$2"/>
 <wire x1="31.75" y1="3.175" x2="31.6865" y2="3.1115" width="0.1524" layer="16"/>
-<wire x1="14.19225" y1="6.5335" x2="13.97" y2="6.31125" width="0.1524" layer="1"/>
-<wire x1="13.97" y1="6.31125" x2="13.97" y2="5.9055" width="0.254" layer="1"/>
+<wire x1="14.1605" y1="6.978" x2="13.97" y2="6.7875" width="0.1524" layer="1"/>
+<wire x1="13.97" y1="6.7875" x2="13.97" y2="5.9055" width="0.254" layer="1"/>
 <wire x1="12.563796875" y1="6.1985" x2="12.309796875" y2="6.1985" width="0.1524" layer="1"/>
 <contactref element="SJ1" pad="2"/>
@@
 <contactref element="R11" pad="1"/>
 <contactref element="U1" pad="5"/>
-<wire x1="16.84379375" y1="4.6875" x2="15.569" y2="4.6875" width="0.1524" layer="1"/>
-<wire x1="15.569" y1="4.6875" x2="14.9725" y2="5.284" width="0.1524" layer="1"/>
+<wire x1="16.84379375" y1="4.6875" x2="15.34675" y2="4.6875" width="0.1524" layer="1"/>
+<wire x1="15.34675" y1="4.6875" x2="14.9725" y2="5.06175" width="0.1524" layer="1"/>
 <wire x1="22.6555" y1="4.5225" x2="22.6555" y2="4.459" width="0.1524" layer="1"/>
 <wire x1="22.6555" y1="4.459" x2="22.4015" y2="4.205" width="0.1524" layer="1"/>
@@
 <wire x1="15.8221625" y1="4.9807" x2="15.5676625" y2="5.2352" width="0.1524" layer="16"/>
 <wire x1="15.5676625" y1="5.2352" x2="14.99045" y2="5.2352" width="0.1524" layer="16"/>
-<wire x1="14.99045" y1="5.2352" x2="14.99045" y2="5.26605" width="0.1524" layer="1"/>
-<wire x1="14.99045" y1="5.26605" x2="14.9725" y2="5.284" width="0.1524" layer="1"/>
+<wire x1="14.99045" y1="5.2352" x2="14.99045" y2="5.0797" width="0.1524" layer="1"/>
+<wire x1="14.99045" y1="5.0797" x2="14.9725" y2="5.06175" width="0.1524" layer="1"/>
 </signal>
 <signal name="VADJ_R1">
@@
 <wire x1="15.494" y1="4.1275" x2="14.9855" y2="4.1275" width="0.1524" layer="1"/>
 <wire x1="14.9855" y1="4.1275" x2="14.9725" y2="4.1405" width="0.1524" layer="1"/>
-<wire x1="14.9725" y1="4.1405" x2="14.478" y2="4.635" width="0.1524" layer="1"/>
-<wire x1="14.478" y1="4.635" x2="14.478" y2="4.8895" width="0.1524" layer="1"/>
-<wire x1="14.478" y1="4.8895" x2="14.0843" y2="5.2832" width="0.1524" layer="1"/>
-<wire x1="14.0843" y1="5.2832" x2="14.0475" y2="5.2832" width="0.1524" layer="1"/>
-<wire x1="14.0475" y1="5.284" x2="14.0835" y2="5.284" width="0.1524" layer="1"/>
-<wire x1="14.0835" y1="5.284" x2="14.0843" y2="5.2832" width="0.1524" layer="1"/>
+<wire x1="14.9725" y1="4.1405" x2="14.0475" y2="5.0655" width="0.1524" layer="1"/>
+<wire x1="14.0475" y1="5.06175" x2="14.0475" y2="5.0655" width="0.1524" layer="1"/>
 </signal>
 <signal name="VADJ_R2">
