File: Eagle_Files/Direct-Extruder-FFC-Breakout_1.0.0.brd (EAGLE design)
At the start: 53.3 x 63.9 mm, 30 parts, among them J1 SFW24R-1STE1LF, Q2 2N2907, U1 LM317DCY, U2 L78L05ACU

Commit message: Pushing changed files saved after exporting gerber
Parts:
- removed R5: 0R, PiezoFFC:R0805
- added F1: 500mA, PiezoFFC:R0805
- moved C4 10.0 mm to (39.2, 38.7)
- moved FAN0 9.29 mm to (-2.27, 23.1)
- moved FAN1 9.29 mm to (-2.27, 13.8)
- moved C3 3.84 mm to (25.6, 25.3), turned to 90 degrees
- moved Q2 2.83 mm to (19.4, 26.3)
- moved R6 2.83 mm to (16.6, 19.9)
- moved R7 2.83 mm to (19.4, 21.1)
- moved U2 2.83 mm to (22.7, 17.8)
- moved C2 1.92 mm to (17.8, 50.9)
- moved 12V 1.00 mm to (32.9, 43.5)
- moved 5V 1.00 mm to (20.2, 43.5)
- moved C5 1.00 mm to (32.3, 35.6)
- moved R1 1.00 mm to (26.6, 39.7)
- moved R2 1.00 mm to (23.3, 39.7)
- moved R3 1.00 mm to (29.9, 39.7)
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Connections:
- new net IND_LED: R4.1, U1.2
- net +5V: now also F1.2; no longer R4.1, R5.2
- net E0_1A: now also E0.3; no longer E0.2
- net E0_1B: now also E0.4; no longer E0.1
- net E0_2A: now also E0.2; no longer E0.3
- net E0_2B: now also E0.1; no longer E0.4
- net TH0+: now also TH1.2; no longer TH1.1
- net TH0-: now also TH1.1; no longer TH1.2
- net VCC_REG: now also F1.1; no longer R5.1
Routing:
- net VCC: track 0.00 -> 134.7 mm
- net FAN1_GATE: track 0.00 -> 53.7 mm
- net FAN0_GATE: track 0.00 -> 50.6 mm
- net TH0-: track 0.00 -> 48.6 mm
- net Z_MIN_TRIG: track 0.00 -> 48.2 mm, vias 0 -> 1
- net TH0+: track 0.00 -> 47.5 mm
- net HE0-: track 0.00 -> 46.3 mm
- net E0_1B: track 0.00 -> 32.2 mm
- net E0_1A: track 0.00 -> 29.0 mm
- net V_INT: track 0.00 -> 26.6 mm
- net E0_2A: track 0.00 -> 25.9 mm
- net VCC_REG: track 0.00 -> 23.5 mm, vias 0 -> 1
- net E0_2B: track 0.00 -> 23.0 mm
- net +5V: track 0.00 -> 14.6 mm
- net LED_R: track 0.00 -> 8.87 mm
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
Commit message: Modified footprints and added 3D Models for caps
Parts:
- C2, C4: value 220uf -> 100uf; device PiezoFFC:PC-D5.3MM -> PiezoFFC:ALU-C-D5.3MM_LEFT
- C3: value 220uf -> 100uf; device PiezoFFC:PC-D5.3MM -> PiezoFFC:ALU-C-D5.3MM_RIGHT
- moved F1 0.50 mm to (28.5, 20.0), turned to 180 degrees
- moved R7 0.12 mm to (19.3, 21.2), turned to 90 degrees
- turned R6 to 0 degrees
