File: Eagle_Files/Direct-Extruder-FFC-Breakout_1.0.0.sch (EAGLE design)
At the start: 29 parts, among them J1 SFW24R-1STE1LF, Q2 2N2907, U1 LM317DCY, U2 L78L05ACU

Commit message: Pushing changed files saved after exporting gerber
Parts:
- F1: value 0R -> 500mA
- renumbered R5 to F1
Connections:
- new net IND_LED: R4.1, U1.OUTPUT_2
- net +5V: no longer R4.1
- net E0_1A: now also E0-3.S; no longer E0-2.S
- net E0_1B: now also E0-4.S; no longer E0-1.S
- net E0_2A: now also E0-2.S; no longer E0-3.S
- net E0_2B: now also E0-1.S; no longer E0-4.S
- net TH0+: now also TH1-2.S; no longer TH1-1.S
- net TH0-: now also TH1-1.S; no longer TH1-2.S
Changed lines of the file:
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@@
 <part name="AGND3" library="supply1" library_urn="urn:adsk.eagle:library:371" deviceset="AGND" device=""/>
 <part name="R4" library="PiezoFFC" library_urn="urn:adsk.eagle:library:6897166" deviceset="SEEED-RESISTOR_SMD-RES-1.5K-1%-1/10W(0603)" device="DETAILED_MODEL" package3d_urn="urn:adsk.eagle:package:5224535/3" value="1K"/>
-<part name="P+2" library="supply1" library_urn="urn:adsk.eagle:library:371" deviceset="+5V" device=""/>
 <part name="5V" library="PiezoFFC" library_urn="urn:adsk.eagle:library:6897166" deviceset="LED" device="CHIP-LED0805" package3d_urn="urn:adsk.eagle:package:15818/2"/>
 <part name="12V" library="PiezoFFC" library_urn="urn:adsk.eagle:library:6897166" deviceset="LED" device="CHIP-LED0805" package3d_urn="urn:adsk.eagle:package:15818/2"/>
@@
 <part name="H3" library="PiezoFFC" library_urn="urn:adsk.eagle:library:6897166" deviceset="HOLES_MOUNT-PAD-ROUND" device="3.2" package3d_urn="urn:adsk.eagle:package:5224590/1"/>
 <part name="H4" library="PiezoFFC" library_urn="urn:adsk.eagle:library:6897166" deviceset="HOLES_MOUNT-PAD-ROUND" device="3.2" package3d_urn="urn:adsk.eagle:package:5224590/1"/>
-<part name="R5" library="PiezoFFC" library_urn="urn:adsk.eagle:library:6897166" deviceset="SMD-RES-2K-5%-1/8W(0805)" device="" package3d_urn="urn:adsk.eagle:package:32799/1" value="0R"/>
+<part name="F1" library="PiezoFFC" library_urn="urn:adsk.eagle:library:6897166" deviceset="SMD-RES-2K-5%-1/8W(0805)" device="" package3d_urn="urn:adsk.eagle:package:32799/1" value="500mA"/>
 </parts>
 <sheets>
@@
 <attribute name="VALUE" x="64.77" y="158.75" size="1.27" layer="96" ratio="10"/>
 </instance>
-<instance part="P+2" gate="1" x="60.96" y="168.91" smashed="yes">
-<attribute name="VALUE" x="59.69" y="170.18" size="1.778" layer="96"/>
-</instance>
 <instance part="5V" gate="G$1" x="73.66" y="148.59" smashed="yes" rot="R270">
 <attribute name="NAME" x="69.088" y="145.034" size="1.778" layer="95"/>
@@
 <attribute name="NAME" x="335.534" y="132.6642" size="1.778" layer="95"/>
 </instance>
-<instance part="R5" gate="G$1" x="118.11" y="102.87" smashed="yes" rot="R180">
+<instance part="F1" gate="G$1" x="118.11" y="102.87" smashed="yes" rot="R180">
 <attribute name="NAME" x="119.38" y="101.6" size="1.27" layer="95" ratio="10" rot="R180"/>
 <attribute name="VALUE" x="119.38" y="105.41" size="1.27" layer="96" ratio="10" rot="R180"/>
@@
 </segment>
 <segment>
-<pinref part="E0" gate="-4" pin="S"/>
-<wire x1="245.11" y1="121.92" x2="257.81" y2="121.92" width="0.1524" layer="91"/>
-<label x="250.19" y="121.92" size="1.778" layer="95"/>
+<wire x1="245.11" y1="114.3" x2="256.54" y2="114.3" width="0.1524" layer="91"/>
+<label x="250.19" y="114.3" size="1.778" layer="95"/>
+<pinref part="E0" gate="-1" pin="S"/>
 </segment>
 </net>
@@
 </segment>
 <segment>
-<pinref part="E0" gate="-3" pin="S"/>
-<wire x1="245.11" y1="119.38" x2="257.81" y2="119.38" width="0.1524" layer="91"/>
-<label x="250.19" y="119.38" size="1.778" layer="95"/>
+<wire x1="245.11" y1="116.84" x2="256.54" y2="116.84" width="0.1524" layer="91"/>
+<label x="250.19" y="116.84" size="1.778" layer="95"/>
+<pinref part="E0" gate="-2" pin="S"/>
 </segment>
 </net>
@@
 </segment>
 <segment>
-<pinref part="E0" gate="-2" pin="S"/>
-<wire x1="245.11" y1="116.84" x2="257.81" y2="116.84" width="0.1524" layer="91"/>
-<label x="250.19" y="116.84" size="1.778" layer="95"/>
+<wire x1="245.11" y1="119.38" x2="256.54" y2="119.38" width="0.1524" layer="91"/>
+<label x="250.19" y="119.38" size="1.778" layer="95"/>
+<pinref part="E0" gate="-3" pin="S"/>
 </segment>
 </net>
@@
 </segment>
 <segment>
-<pinref part="E0" gate="-1" pin="S"/>
-<wire x1="245.11" y1="114.3" x2="257.81" y2="114.3" width="0.1524" layer="91"/>
-<label x="250.19" y="114.3" size="1.778" layer="95"/>
+<wire x1="245.11" y1="121.92" x2="256.54" y2="121.92" width="0.1524" layer="91"/>
+<label x="250.19" y="121.92" size="1.778" layer="95"/>
+<pinref part="E0" gate="-4" pin="S"/>
 </segment>
 </net>
@@
 <wire x1="121.92" y1="102.87" x2="138.43" y2="102.87" width="0.1524" layer="91"/>
 <label x="123.19" y="102.87" size="1.778" layer="95"/>
-<pinref part="R5" gate="G$1" pin="1"/>
+<pinref part="F1" gate="G$1" pin="1"/>
 </segment>
 </net>
@@
 </segment>
 <segment>
-<pinref part="TH1" gate="-2" pin="S"/>
-<wire x1="245.11" y1="162.56" x2="257.81" y2="162.56" width="0.1524" layer="91"/>
-<label x="252.73" y="162.56" size="1.778" layer="95"/>
+<wire x1="245.11" y1="160.02" x2="255.27" y2="160.02" width="0.1524" layer="91"/>
+<label x="250.19" y="160.02" size="1.778" layer="95"/>
+<pinref part="TH1" gate="-1" pin="S"/>
 </segment>
 </net>
@@
 </segment>
 <segment>
-<pinref part="TH1" gate="-1" pin="S"/>
-<wire x1="245.11" y1="160.02" x2="257.81" y2="160.02" width="0.1524" layer="91"/>
-<label x="252.73" y="160.02" size="1.778" layer="95"/>
+<wire x1="245.11" y1="162.56" x2="255.27" y2="162.56" width="0.1524" layer="91"/>
+<label x="250.19" y="162.56" size="1.778" layer="95"/>
+<pinref part="TH1" gate="-2" pin="S"/>
 </segment>
 </net>
@@
 <net name="+5V" class="0">
 <segment>
-<pinref part="P+2" gate="1" pin="+5V"/>
-<wire x1="60.96" y1="166.37" x2="60.96" y2="161.29" width="0.1524" layer="91"/>
-<pinref part="R4" gate="G$1" pin="1"/>
-<wire x1="60.96" y1="161.29" x2="64.77" y2="161.29" width="0.1524" layer="91"/>
-</segment>
-<segment>
 <pinref part="U2" gate="G$1" pin="OUT"/>
 <wire x1="106.68" y1="87.63" x2="107.95" y2="87.63" width="0.1524" layer="91"/>
@@
 <pinref part="P+1" gate="1" pin="+5V"/>
 <wire x1="107.95" y1="105.41" x2="107.95" y2="102.87" width="0.1524" layer="91"/>
-<pinref part="R5" gate="G$1" pin="2"/>
+<pinref part="F1" gate="G$1" pin="2"/>
 </segment>
 </net>
@@
 </segment>
 </net>
+<net name="IND_LED" class="0">
+<segment>
+<pinref part="R4" gate="G$1" pin="1"/>
+<wire x1="60.96" y1="161.29" x2="64.77" y2="161.29" width="0.1524" layer="91"/>
+<label x="63.5" y="161.29" size="1.778" layer="95" rot="R180"/>
+</segment>
+<segment>
+<pinref part="U1" gate="A" pin="OUTPUT_2"/>
+<wire x1="146.05" y1="166.37" x2="146.05" y2="179.07" width="0.1524" layer="91"/>
+<label x="146.05" y="170.18" size="1.778" layer="95" rot="R90"/>
+</segment>
+</net>

Commit message: Modified footprints and added 3D Models for caps
Parts:
- C2, C4: value 220uf -> 100uf; device PiezoFFC:DIP-ALUMINUM-100UF-16V(D5-H7MM) -> PiezoFFC:DIP-ALUMINUM-100UF-16V(D5-H7MM)LEFT
- C3: value 220uf -> 100uf; device PiezoFFC:DIP-ALUMINUM-100UF-16V(D5-H7MM) -> PiezoFFC:DIP-ALUMINUM-100UF-16V(D5-H7MM)RIGHT
Changed lines of the file:
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@@
 <setting verticaltext="up"/>
 </settings>
-<grid distance="1.27" unitdist="mm" unit="mm" style="lines" multiple="1" display="no" altdistance="0.01" altunitdist="inch" altunit="inch"/>
+<grid distance="0.1" unitdist="inch" unit="inch" style="lines" multiple="1" display="no" altdistance="0.01" altunitdist="inch" altunit="inch"/>
 <layers>
 <layer number="1" name="Top" color="4" fill="1" visible="no" active="no"/>
@@
 <part name="J1" library="PiezoFFC" library_urn="urn:adsk.eagle:library:6897166" deviceset="SFW24R-1STE1LF" device="" package3d_urn="urn:adsk.eagle:package:6899317/2"/>
 <part name="AGND1" library="supply1" library_urn="urn:adsk.eagle:library:371" deviceset="AGND" device=""/>
-<part name="U1" library="PiezoFFC" library_urn="urn:adsk.eagle:library:6897166" deviceset="LM317DCY" device=""/>
-<part name="SW1" library="PiezoFFC" library_urn="urn:adsk.eagle:library:6897166" deviceset="SEEED-SWITCH_DIP-TOGGLE-SWITCH-2CH-(2X3P-2.54)" device="DPDT_254_6P_UPDATE" package3d_urn="urn:adsk.eagle:package:5224531/3"/>
+<part name="U1" library="PiezoFFC" library_urn="urn:adsk.eagle:library:6897166" deviceset="LM317DCY" device="" package3d_urn="urn:adsk.eagle:package:7346255/2"/>
+<part name="SW1" library="PiezoFFC" library_urn="urn:adsk.eagle:library:6897166" deviceset="SEEED-SWITCH_DIP-TOGGLE-SWITCH-2CH-(2X3P-2.54)" device="DPDT_254_6P_UPDATE" package3d_urn="urn:adsk.eagle:package:5224531/4"/>
 <part name="E0" library="PiezoFFC" library_urn="urn:adsk.eagle:library:6897166" deviceset="C-GRID-04" device="-70553" package3d_urn="urn:adsk.eagle:package:6902618/2"/>
-<part name="Z_MIN" library="PiezoFFC" library_urn="urn:adsk.eagle:library:6897166" deviceset="C-GRID-02" device="-70553"/>
-<part name="FAN1" library="PiezoFFC" library_urn="urn:adsk.eagle:library:6897166" deviceset="C-GRID-02" device="-70553"/>
-<part name="FAN0" library="PiezoFFC" library_urn="urn:adsk.eagle:library:6897166" deviceset="C-GRID-02" device="-70553"/>
-<part name="TH1" library="PiezoFFC" library_urn="urn:adsk.eagle:library:6897166" deviceset="C-GRID-02" device="-70553"/>
-<part name="HE0" library="PiezoFFC" library_urn="urn:adsk.eagle:library:6897166" deviceset="KK-156-2" device=""/>
+<part name="Z_MIN" library="PiezoFFC" library_urn="urn:adsk.eagle:library:6897166" deviceset="C-GRID-02" device="-70553" package3d_urn="urn:adsk.eagle:package:7346257/2"/>
+<part name="FAN1" library="PiezoFFC" library_urn="urn:adsk.eagle:library:6897166" deviceset="C-GRID-02" device="-70553" package3d_urn="urn:adsk.eagle:package:7346257/2"/>
+<part name="FAN0" library="PiezoFFC" library_urn="urn:adsk.eagle:library:6897166" deviceset="C-GRID-02" device="-70553" package3d_urn="urn:adsk.eagle:package:7346257/2"/>
+<part name="TH1" library="PiezoFFC" library_urn="urn:adsk.eagle:library:6897166" deviceset="C-GRID-02" device="-70553" package3d_urn="urn:adsk.eagle:package:7346257/2"/>
+<part name="HE0" library="PiezoFFC" library_urn="urn:adsk.eagle:library:6897166" deviceset="KK-156-2" device="" package3d_urn="urn:adsk.eagle:package:7346264/2"/>
 <part name="AGND2" library="supply1" library_urn="urn:adsk.eagle:library:371" deviceset="AGND" device=""/>
-<part name="PWR" library="PiezoFFC" library_urn="urn:adsk.eagle:library:6897166" deviceset="KK-156-2" device=""/>
+<part name="PWR" library="PiezoFFC" library_urn="urn:adsk.eagle:library:6897166" deviceset="KK-156-2" device="" package3d_urn="urn:adsk.eagle:package:7346264/2"/>
 <part name="R1" library="PiezoFFC" library_urn="urn:adsk.eagle:library:6897166" deviceset="SEEED-RESISTOR_SMD-RES-1.5K-1%-1/10W(0603)" device="DETAILED_MODEL" package3d_urn="urn:adsk.eagle:package:5224535/3" value="240R"/>
 <part name="R2" library="PiezoFFC" library_urn="urn:adsk.eagle:library:6897166" deviceset="SEEED-RESISTOR_SMD-RES-1.5K-1%-1/10W(0603)" device="DETAILED_MODEL" package3d_urn="urn:adsk.eagle:package:5224535/3" value="715R"/>
@@
 <part name="5V" library="PiezoFFC" library_urn="urn:adsk.eagle:library:6897166" deviceset="LED" device="CHIP-LED0805" package3d_urn="urn:adsk.eagle:package:15818/2"/>
 <part name="12V" library="PiezoFFC" library_urn="urn:adsk.eagle:library:6897166" deviceset="LED" device="CHIP-LED0805" package3d_urn="urn:adsk.eagle:package:15818/2"/>
-<part name="U2" library="PiezoFFC" library_urn="urn:adsk.eagle:library:6897166" deviceset="L78L05ACU" device="" package3d_urn="urn:adsk.eagle:package:6899241/4"/>
+<part name="U2" library="PiezoFFC" library_urn="urn:adsk.eagle:library:6897166" deviceset="L78L05ACU" device="" package3d_urn="urn:adsk.eagle:package:6899241/5"/>
 <part name="AGND4" library="supply1" library_urn="urn:adsk.eagle:library:371" deviceset="AGND" device=""/>
 <part name="Q2" library="PiezoFFC" library_urn="urn:adsk.eagle:library:6897166" deviceset="2N2907" device="" package3d_urn="urn:adsk.eagle:package:28523/2"/>
-<part name="R6" library="PiezoFFC" library_urn="urn:adsk.eagle:library:6897166" deviceset="SMD-RES-2K-5%-1/8W(0805)" device="" package3d_urn="urn:adsk.eagle:package:32799/1" value="1R"/>
-<part name="R7" library="PiezoFFC" library_urn="urn:adsk.eagle:library:6897166" deviceset="SMD-RES-2K-5%-1/8W(0805)" device="" package3d_urn="urn:adsk.eagle:package:32799/1" value="10R"/>
-<part name="C2" library="PiezoFFC" library_urn="urn:adsk.eagle:library:6897166" deviceset="DIP-ALUMINUM-100UF-16V(D5-H7MM)" device="" package3d_urn="urn:adsk.eagle:package:32406/1" value="220uf"/>
-<part name="C3" library="PiezoFFC" library_urn="urn:adsk.eagle:library:6897166" deviceset="DIP-ALUMINUM-100UF-16V(D5-H7MM)" device="" package3d_urn="urn:adsk.eagle:package:32406/1" value="220uf"/>
-<part name="C4" library="PiezoFFC" library_urn="urn:adsk.eagle:library:6897166" deviceset="DIP-ALUMINUM-100UF-16V(D5-H7MM)" device="" package3d_urn="urn:adsk.eagle:package:32406/1" value="220uf"/>
+<part name="R6" library="PiezoFFC" library_urn="urn:adsk.eagle:library:6897166" deviceset="SMD-RES-2K-5%-1/8W(0805)" device="" package3d_urn="urn:adsk.eagle:package:8443791/2" value="1R"/>
+<part name="R7" library="PiezoFFC" library_urn="urn:adsk.eagle:library:6897166" deviceset="SMD-RES-2K-5%-1/8W(0805)" device="" package3d_urn="urn:adsk.eagle:package:8443791/2" value="10R"/>
+<part name="C2" library="PiezoFFC" library_urn="urn:adsk.eagle:library:6897166" deviceset="DIP-ALUMINUM-100UF-16V(D5-H7MM)" device="LEFT" package3d_urn="urn:adsk.eagle:package:8885168/4" value="100uf"/>
+<part name="C3" library="PiezoFFC" library_urn="urn:adsk.eagle:library:6897166" deviceset="DIP-ALUMINUM-100UF-16V(D5-H7MM)" device="RIGHT" package3d_urn="urn:adsk.eagle:package:8885515/3" value="100uf"/>
+<part name="C4" library="PiezoFFC" library_urn="urn:adsk.eagle:library:6897166" deviceset="DIP-ALUMINUM-100UF-16V(D5-H7MM)" device="LEFT" package3d_urn="urn:adsk.eagle:package:8885168/4" value="100uf"/>
 <part name="C5" library="PiezoFFC" library_urn="urn:adsk.eagle:library:6897166" deviceset="SEEED-CAPACITOR_CERAMIC-10UF-25V-10%-X5R(0805)" device="CAP_0805-3D" package3d_urn="urn:adsk.eagle:package:5225034/2" value="10uF"/>
 <part name="P+1" library="supply1" library_urn="urn:adsk.eagle:library:371" deviceset="+5V" device=""/>
 <part name="AGND5" library="supply1" library_urn="urn:adsk.eagle:library:371" deviceset="AGND" device=""/>
-<part name="H1" library="PiezoFFC" library_urn="urn:adsk.eagle:library:6897166" deviceset="HOLES_MOUNT-PAD-ROUND" device="3.2" package3d_urn="urn:adsk.eagle:package:5224590/1"/>
-<part name="H2" library="PiezoFFC" library_urn="urn:adsk.eagle:library:6897166" deviceset="HOLES_MOUNT-PAD-ROUND" device="3.2" package3d_urn="urn:adsk.eagle:package:5224590/1"/>
-<part name="H3" library="PiezoFFC" library_urn="urn:adsk.eagle:library:6897166" deviceset="HOLES_MOUNT-PAD-ROUND" device="3.2" package3d_urn="urn:adsk.eagle:package:5224590/1"/>
-<part name="H4" library="PiezoFFC" library_urn="urn:adsk.eagle:library:6897166" deviceset="HOLES_MOUNT-PAD-ROUND" device="3.2" package3d_urn="urn:adsk.eagle:package:5224590/1"/>
-<part name="F1" library="PiezoFFC" library_urn="urn:adsk.eagle:library:6897166" deviceset="SMD-RES-2K-5%-1/8W(0805)" device="" package3d_urn="urn:adsk.eagle:package:32799/1" value="500mA"/>
+<part name="H1" library="PiezoFFC" library_urn="urn:adsk.eagle:library:6897166" deviceset="HOLES_MOUNT-PAD-ROUND" device="3.2" package3d_urn="urn:adsk.eagle:package:5224590/2"/>
+<part name="H2" library="PiezoFFC" library_urn="urn:adsk.eagle:library:6897166" deviceset="HOLES_MOUNT-PAD-ROUND" device="3.2" package3d_urn="urn:adsk.eagle:package:5224590/2"/>
+<part name="H3" library="PiezoFFC" library_urn="urn:adsk.eagle:library:6897166" deviceset="HOLES_MOUNT-PAD-ROUND" device="3.2" package3d_urn="urn:adsk.eagle:package:5224590/2"/>
+<part name="H4" library="PiezoFFC" library_urn="urn:adsk.eagle:library:6897166" deviceset="HOLES_MOUNT-PAD-ROUND" device="3.2" package3d_urn="urn:adsk.eagle:package:5224590/2"/>
+<part name="F1" library="PiezoFFC" library_urn="urn:adsk.eagle:library:6897166" deviceset="SMD-RES-2K-5%-1/8W(0805)" device="" package3d_urn="urn:adsk.eagle:package:8443791/2" value="500mA"/>
 </parts>
 <sheets>
@@
 <instance part="C3" gate="G$1" x="107.95" y="78.74" smashed="yes" rot="R270">
 <attribute name="NAME" x="105.41" y="77.47" size="1.27" layer="95" ratio="10" rot="R90"/>
-<attribute name="VALUE" x="110.49" y="80.01" size="1.27" layer="96" ratio="10" rot="R270"/>
 </instance>
 <instance part="C4" gate="G$1" x="151.13" y="142.24" smashed="yes" rot="R270">
