File: Eagle_Files/Extruder_Board1.1.0.sch (EAGLE design)
At the start: 60 parts, among them J1 SFW24R-1STE1LF, U1 ATMEGA48PA-MMHR28M1-L, U2 LM2902QT

Commit message: Pushing changed files saved after exporting gerber
Parts:
- renumbered R14 to F1
Other:
- note removed: "Feedback LED's"
Changed lines of the file:
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@@
 <part name="R12" library="PiezoFFC" library_urn="urn:adsk.eagle:library:6897166" deviceset="SMD-RES-0R-5%-1/16W(0402)" device="" package3d_urn="urn:adsk.eagle:package:7115182/2" value="330R"/>
 <part name="R13" library="PiezoFFC" library_urn="urn:adsk.eagle:library:6897166" deviceset="SMD-RES-0R-5%-1/16W(0402)" device="" package3d_urn="urn:adsk.eagle:package:7115182/2" value="100R"/>
-<part name="R14" library="PiezoFFC" library_urn="urn:adsk.eagle:library:6897166" deviceset="SEEED-RESISTOR_SMD-RES-1.5K-1%-1/10W(0603)" device="DETAILED_MODEL" package3d_urn="urn:adsk.eagle:package:5224535/3" value="0R"/>
+<part name="F1" library="PiezoFFC" library_urn="urn:adsk.eagle:library:6897166" deviceset="SEEED-RESISTOR_SMD-RES-1.5K-1%-1/10W(0603)" device="DETAILED_MODEL" package3d_urn="urn:adsk.eagle:package:5224535/3" value="0R"/>
 <part name="P+8" library="supply1" library_urn="urn:adsk.eagle:library:371" deviceset="+5V" device=""/>
 <part name="ADJ-" library="PiezoFFC" library_urn="urn:adsk.eagle:library:6897166" deviceset="TP" device="TP10R" package3d_urn="urn:adsk.eagle:package:27959/1" value="TPTP10R"/>
@@
 <wire x1="322.58" y1="181.61" x2="322.58" y2="224.79" width="0.1524" layer="94"/>
 <text x="180.34" y="201.93" size="1.778" layer="94" rot="R90">Piezo In</text>
-<text x="218.44" y="73.66" size="3.81" layer="94">Feedback LED's</text>
 <wire x1="228.6" y1="224.79" x2="228.6" y2="181.61" width="0.1524" layer="94"/>
 <wire x1="228.6" y1="181.61" x2="223.52" y2="176.53" width="0.1524" layer="94"/>
@@
 <attribute name="VALUE" x="354.33" y="200.66" size="1.27" layer="96" ratio="10"/>
 </instance>
-<instance part="R14" gate="G$1" x="71.12" y="130.81" smashed="yes">
+<instance part="F1" gate="G$1" x="71.12" y="130.81" smashed="yes">
 <attribute name="NAME" x="67.31" y="132.08" size="1.27" layer="95" ratio="10"/>
 <attribute name="VALUE" x="67.31" y="128.27" size="1.27" layer="96" ratio="10"/>
@@
 <wire x1="50.8" y1="127" x2="50.8" y2="130.81" width="0.1524" layer="91"/>
 <junction x="50.8" y="130.81"/>
-<pinref part="R14" gate="G$1" pin="1"/>
+<pinref part="F1" gate="G$1" pin="1"/>
 <wire x1="67.31" y1="130.81" x2="60.96" y2="130.81" width="0.1524" layer="91"/>
 <pinref part="D1" gate="G$1" pin="C"/>
@@
 <wire x1="99.06" y1="128.27" x2="99.06" y2="130.81" width="0.1524" layer="91"/>
 <junction x="99.06" y="130.81"/>
-<pinref part="R14" gate="G$1" pin="2"/>
+<pinref part="F1" gate="G$1" pin="2"/>
 <pinref part="P+5" gate="1" pin="+5V"/>
 <wire x1="83.82" y1="137.16" x2="83.82" y2="130.81" width="0.1524" layer="91"/>

Commit message: fixed some spacing and labelling
Parts:
- R6: value (none) -> 1K
Connections:
- net N$2 renamed PWR_LED
- net E0_1A: now also E0-2.S, J1.33, J1.44; no longer E0-3.S, J1.55, J1.66
- net E0_1B: now also E0-1.S, J1.11, J1.22; no longer E0-4.S, J1.77, J1.88
- net E0_2A: now also E0-3.S, J1.55, J1.66; no longer E0-2.S, J1.33, J1.44
- net E0_2B: now also E0-4.S, J1.77, J1.88; no longer E0-1.S, J1.11, J1.22
Changed lines of the file:
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@@
 <setting verticaltext="up"/>
 </settings>
-<grid distance="1.27" unitdist="mm" unit="mm" style="lines" multiple="1" display="no" altdistance="0.01" altunitdist="inch" altunit="inch"/>
+<grid distance="0.1" unitdist="inch" unit="inch" style="lines" multiple="1" display="no" altdistance="0.01" altunitdist="inch" altunit="inch"/>
 <layers>
 <layer number="1" name="Top" color="4" fill="1" visible="no" active="no"/>
@@
 <part name="TRG" library="PiezoFFC" library_urn="urn:adsk.eagle:library:6897166" deviceset="SEEED-LED_SMD-LED-CLEAR-BLUE(0603)" device="LED_0603" package3d_urn="urn:adsk.eagle:package:5224536/3"/>
 <part name="PWR" library="PiezoFFC" library_urn="urn:adsk.eagle:library:6897166" deviceset="SEEED-LED_SMD-LED-CLEAR-BLUE(0603)" device="LED_0603" package3d_urn="urn:adsk.eagle:package:5224536/3"/>
-<part name="R6" library="PiezoFFC" library_urn="urn:adsk.eagle:library:6897166" deviceset="SMD-RES-0R-5%-1/16W(0402)" device="" package3d_urn="urn:adsk.eagle:package:7115182/2"/>
+<part name="R6" library="PiezoFFC" library_urn="urn:adsk.eagle:library:6897166" deviceset="SMD-RES-0R-5%-1/16W(0402)" device="" package3d_urn="urn:adsk.eagle:package:7115182/2" value="1K"/>
 <part name="R8" library="PiezoFFC" library_urn="urn:adsk.eagle:library:6897166" deviceset="SMD-RES-0R-5%-1/16W(0402)" device="" package3d_urn="urn:adsk.eagle:package:7115182/2" value="1K"/>
 <part name="R1" library="PiezoFFC" library_urn="urn:adsk.eagle:library:6897166" deviceset="SMD-RES-0R-5%-1/16W(0402)" device="" package3d_urn="urn:adsk.eagle:package:7115182/2" value="1M"/>
@@
 </segment>
 </net>
-<net name="E0_1B" class="0">
+<net name="E0_2B" class="0">
 <segment>
 <pinref part="J1" gate="A" pin="88"/>
@@
 </segment>
 </net>
-<net name="E0_1A" class="0">
+<net name="E0_2A" class="0">
 <segment>
 <pinref part="J1" gate="A" pin="66"/>
@@
 </segment>
 </net>
-<net name="E0_2A" class="0">
+<net name="E0_1A" class="0">
 <segment>
 <pinref part="J1" gate="A" pin="44"/>
@@
 </segment>
 </net>
-<net name="E0_2B" class="0">
+<net name="E0_1B" class="0">
 <segment>
 <pinref part="J1" gate="A" pin="22"/>
@@
 </segment>
 </net>
-<net name="N$2" class="0">
+<net name="PWR_LED" class="0">
 <segment>
 <pinref part="R8" gate="G$1" pin="2"/>
