File: Eagle_Files/Direct-Extruder-FFC-Breakout_2.0.0.brd (EAGLE design)
At the start: 53.3 x 63.9 mm, 30 parts, among them J1 FFC_MOLEX_0.5MM, Q2 2N2907, U1 LM317DCY, U2 L78L05ACU

Commit message: Added X-motor and X-min breakouts
Added in preparation for https://github.com/pyr0ball/pyr0piezo/issues/18
Parts:
- added I2C: (no value), PiezoFFC:HDRVR4W64P254_1X4_1016X254X575B
- added UART: JST-2.54MM_5P-2.54JST_2.54MM_5P_F, PiezoFFC:HDRVR5W64P254_1X5_1270X254X575B
- added X_MIN: C-GRID-02-70553, PiezoFFC:70553-02
- added X_MOT: C-GRID-04-70553, PiezoFFC:70553-04
- C2: device PiezoFFC:PC-D5.3MM -> PiezoFFC:ALU-C-D5.3MM_LEFT
- C3, C4: device PiezoFFC:PC-D5.3MM -> PiezoFFC:ALU-C-D5.3MM_RIGHT
- moved E0 12.5 mm to (48.1, 1.73)
- moved H3 11.5 mm to (59.8, 5.18)
- moved H4 11.5 mm to (59.8, 58.8)
- moved J1 11.5 mm to (62.5, 32.0)
- moved C4 8.35 mm to (37.8, 37.7), turned to 90 degrees
- moved C3 3.74 mm to (23.2, 25.3), turned to 90 degrees
- moved Z_MIN 1.50 mm to (22.5, 1.73)
Connections:
- new net PT_100_OUT: J1.28
- new net RST: J1.23, UART.5
- new net RXD: J1.22, UART.4
- new net SCL: I2C.4, J1.20
- new net SDA: I2C.3, J1.19
- new net TXD: J1.21, UART.3
- new net X_1A: J1.13, J1.14, X_MOT.2
- new net X_1B: J1.11, J1.12, X_MOT.1
- new net X_2A: J1.15, J1.16, X_MOT.3
- new net X_2B: J1.17, J1.18, X_MOT.4
- new net X_MIN_TRIG: J1.27, X_MIN.2
- net AGND: now also I2C.2, UART.2, X_MIN.1
- net VCC_REG: now also I2C.1, J1.24, J1.25, UART.1; no longer J1.12, J1.13
- net Z_MIN_TRIG: now also J1.26; no longer J1.11
Routing:
- net X_MIN_TRIG: track 0.00 -> 71.6 mm
- net X_2B: track 0.00 -> 36.2 mm
- net X_2A: track 0.00 -> 33.3 mm
- net X_1A: track 0.00 -> 30.3 mm
- net Z_MIN_TRIG: track 33.7 -> 61.8 mm
- net X_1B: track 0.00 -> 27.4 mm
- net VCC_REG: track 22.6 -> 43.4 mm
- net V_INT: track 40.0 -> 51.7 mm
- net TH0-: track 46.3 -> 57.8 mm
- net TH0+: track 46.2 -> 57.7 mm
- net FAN1_GATE: track 46.9 -> 58.4 mm
- net FAN0_GATE: track 55.9 -> 67.4 mm
- net TXD: track 0.00 -> 10.0 mm
- net VCC: track 138.1 -> 148.1 mm
- net HE0-: track 56.1 -> 65.5 mm
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Other:
- board size 53.3 x 63.9 mm -> 64.8 x 63.9 mm
- board text added: "+5V ⏚ SDA SCL"
- board text added: "+5V ⏚ TXD RXD RST"
