File: Eagle_Files/Direct-Extruder-FFC-Breakout_2.0.0.sch (EAGLE design)
At the start: 29 parts, among them J1 FFC_MOLEX_0.5MM, Q2 2N2907, U1 LM317DCY, U2 L78L05ACU

Commit message: Added X-motor and X-min breakouts
Added in preparation for https://github.com/pyr0ball/pyr0piezo/issues/18
Parts:
- added I2C: (no value), PiezoFFC:SEEED-CONNECTOR_DIP-BLACK-FEMALE-HEADER-VERT(4P-2.54)JST-2.54MM_4P
- added UART: JST-2.54MM_5P-2.54JST_2.54MM_5P_F, PiezoFFC:JST-2.54MM_5P-2.54JST_2.54MM_5P_F
- added X_MIN: C-GRID-02-70553, PiezoFFC:C-GRID-02-70553
- added X_MOT: C-GRID-04-70553, PiezoFFC:C-GRID-04-70553
- C2: device PiezoFFC:DIP-ALUMINUM-100UF-16V(D5-H7MM) -> PiezoFFC:DIP-ALUMINUM-100UF-16V(D5-H7MM)LEFT
- C3, C4: device PiezoFFC:DIP-ALUMINUM-100UF-16V(D5-H7MM) -> PiezoFFC:DIP-ALUMINUM-100UF-16V(D5-H7MM)RIGHT
Connections:
- new net PT_100_OUT: J1.30
- new net RST: J1.25, UART.P$5
- new net RXD: J1.24, UART.P$4
- new net SCL: I2C.P$4, J1.22
- new net SDA: I2C.P$3, J1.21
- new net TXD: J1.23, UART.P$3
- new net X_1A: J1.15, J1.16, X_MOT-2.S
- new net X_1B: J1.13, J1.14, X_MOT-1.S
- new net X_2A: J1.17, J1.18, X_MOT-3.S
- new net X_2B: J1.19, J1.20, X_MOT-4.S
- new net X_MIN_TRIG: J1.29, X_MIN-2.S
- net AGND: now also I2C.P$2, UART.P$2, X_MIN-1.S
- net VCC_REG: now also I2C.P$1, J1.26, J1.27, UART.P$1; no longer J1.14, J1.15
- net Z_MIN_TRIG: now also J1.28; no longer J1.13
Other:
- moved on the sheet: E0-1, E0-2, E0-3, E0-4
