File: Eagle_Files/Pyr0-Piezo-FFC-Creality-X-Board.2.0.0.sch (EAGLE design)
At the start: 8 parts, among them J1 FFC_MOLEX_0.5MM, J2 FFC_MOLEX_0.5MM

Commit message: Finished first iteration of x-gantry board
First version to address https://github.com/pyr0ball/pyr0piezo/issues/18
Parts:
- added D1: (no value), PiezoFFC:SEEED-LED_SMD-LED-CLEAR-BLUE(0603)LED_0603
- added R1, R2: 1K, PiezoFFC:SMD-RES-2K-5%-1/8W(0805)
- X_MIN: value C-GRID-03-70553 -> LIMIT_SWITCHMICRO_SPDT_5.08; device PiezoFFC:C-GRID-03-70553 -> PiezoFFC:LIMIT_SWITCHMICRO_SPDT_5.08
Connections:
- new net X_MIN_LED: D1.+, R1.1
- new net X_PULLDOWN: R2.1, X_MIN.COM
- net AGND: now also X_MIN.NO
- net VCC_REG: now also R1.2
- net X_MIN_TRIG: now also D1.-, R2.2
Changed lines of the file:
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@@
 <?xml version="1.0" encoding="utf-8"?>
 <!DOCTYPE eagle SYSTEM "eagle.dtd">
-<eagle version="9.3.1">
+<eagle version="9.3.0">
 <drawing>
 <settings>
@@
 <setting verticaltext="up"/>
 </settings>
-<grid distance="0.1" unitdist="inch" unit="inch" style="lines" multiple="1" display="no" altdistance="0.01" altunitdist="inch" altunit="inch"/>
+<grid distance="1.27" unitdist="mm" unit="mm" style="lines" multiple="1" display="no" altdistance="0.01" altunitdist="inch" altunit="inch"/>
 <layers>
 <layer number="1" name="Top" color="4" fill="1" visible="no" active="no"/>
@@
 <part name="J2" library="PiezoFFC" library_urn="urn:adsk.eagle:library:6897166" deviceset="FFC_MOLEX_0.5MM" device="" package3d_urn="urn:adsk.eagle:package:8786753/3"/>
 <part name="X-MOT" library="PiezoFFC" library_urn="urn:adsk.eagle:library:6897166" deviceset="C-GRID-04" device="-70553" package3d_urn="urn:adsk.eagle:package:6902618/2"/>
-<part name="X_MIN" library="PiezoFFC" library_urn="urn:adsk.eagle:library:6897166" deviceset="C-GRID-03" device="-70553" package3d_urn="urn:adsk.eagle:package:7346260/2"/>
 <part name="AGND1" library="supply1" library_urn="urn:adsk.eagle:library:371" deviceset="AGND" device=""/>
 <part name="AGND2" library="supply1" library_urn="urn:adsk.eagle:library:371" deviceset="AGND" device=""/>
@@
 <part name="P+1" library="supply1" library_urn="urn:adsk.eagle:library:371" deviceset="VCC" device=""/>
 <part name="P+2" library="supply1" library_urn="urn:adsk.eagle:library:371" deviceset="VCC" device=""/>
+<part name="X_MIN" library="PiezoFFC" library_urn="urn:adsk.eagle:library:6897166" deviceset="LIMIT_SWITCH" device="MICRO_SPDT_5.08" package3d_urn="urn:adsk.eagle:package:9246121/2"/>
+<part name="R1" library="PiezoFFC" library_urn="urn:adsk.eagle:library:6897166" deviceset="SMD-RES-2K-5%-1/8W(0805)" device="" package3d_urn="urn:adsk.eagle:package:8443791/2" value="1K"/>
+<part name="AGND4" library="supply1" library_urn="urn:adsk.eagle:library:371" deviceset="AGND" device=""/>
+<part name="D1" library="PiezoFFC" library_urn="urn:adsk.eagle:library:6897166" deviceset="SEEED-LED_SMD-LED-CLEAR-BLUE(0603)" device="LED_0603" package3d_urn="urn:adsk.eagle:package:5224536/3"/>
+<part name="R2" library="PiezoFFC" library_urn="urn:adsk.eagle:library:6897166" deviceset="SMD-RES-2K-5%-1/8W(0805)" device="" package3d_urn="urn:adsk.eagle:package:8443791/2" value="1K"/>
 </parts>
 <sheets>
@@
 <attribute name="NAME" x="17.78" y="60.198" size="1.524" layer="95"/>
 </instance>
-<instance part="X_MIN" gate="-1" x="15.24" y="53.34" smashed="yes">
-<attribute name="NAME" x="17.78" y="52.578" size="1.524" layer="95"/>
-<attribute name="VALUE" x="14.478" y="54.737" size="1.778" layer="96"/>
-</instance>
-<instance part="X_MIN" gate="-2" x="15.24" y="50.8" smashed="yes">
-<attribute name="NAME" x="17.78" y="50.038" size="1.524" layer="95"/>
-</instance>
-<instance part="X_MIN" gate="-3" x="15.24" y="48.26" smashed="yes">
-<attribute name="NAME" x="17.78" y="47.498" size="1.524" layer="95"/>
-</instance>
 <instance part="AGND1" gate="VR1" x="-7.62" y="-25.4" smashed="yes">
 <attribute name="VALUE" x="-10.16" y="-30.48" size="1.778" layer="96" rot="R90"/>
@@
 <instance part="P+2" gate="VCC" x="-68.58" y="17.78" smashed="yes">
 <attribute name="VALUE" x="-71.12" y="15.24" size="1.778" layer="96" rot="R90"/>
+</instance>
+<instance part="X_MIN" gate="G$1" x="44.45" y="40.64" smashed="yes">
+<attribute name="NAME" x="39.37" y="45.72" size="1.9304" layer="95"/>
+</instance>
+<instance part="R1" gate="G$1" x="11.43" y="26.67" smashed="yes" rot="R180">
+<attribute name="NAME" x="12.7" y="25.4" size="1.27" layer="95" ratio="10" rot="R180"/>
+<attribute name="VALUE" x="11.43" y="29.21" size="1.27" layer="96" ratio="10" rot="R180"/>
+</instance>
+<instance part="AGND4" gate="VR1" x="57.15" y="30.48" smashed="yes">
+<attribute name="VALUE" x="54.61" y="25.4" size="1.778" layer="96" rot="R90"/>
+</instance>
+<instance part="D1" gate="G$1" x="20.32" y="31.75" smashed="yes" rot="R90">
+<attribute name="NAME" x="22.86" y="33.02" size="1.27" layer="95" ratio="10" rot="R270"/>
+<attribute name="VALUE" x="25.4" y="26.67" size="1.27" layer="96" ratio="10" rot="R90"/>
+</instance>
+<instance part="R2" gate="G$1" x="27.94" y="40.64" smashed="yes" rot="R180">
+<attribute name="NAME" x="29.21" y="39.37" size="1.27" layer="95" ratio="10" rot="R180"/>
+<attribute name="VALUE" x="27.94" y="43.18" size="1.27" layer="96" ratio="10" rot="R180"/>
 </instance>
 </instances>
@@
 <junction x="-73.66" y="20.32"/>
 </segment>
+<segment>
+<pinref part="X_MIN" gate="G$1" pin="NO"/>
+<pinref part="AGND4" gate="VR1" pin="AGND"/>
+<wire x1="53.34" y1="36.83" x2="57.15" y2="36.83" width="0.1524" layer="91"/>
+<wire x1="57.15" y1="36.83" x2="57.15" y2="33.02" width="0.1524" layer="91"/>
+</segment>
 </net>
 <net name="X_1B_NC" class="0">
@@
 <junction x="-91.44" y="2.54"/>
 <label x="-101.6" y="0" size="1.778" layer="95"/>
+</segment>
+<segment>
+<pinref part="R1" gate="G$1" pin="2"/>
+<wire x1="7.62" y1="26.67" x2="0" y2="26.67" width="0.1524" layer="91"/>
+<wire x1="0" y1="26.67" x2="0" y2="30.48" width="0.1524" layer="91"/>
+<label x="0" y="30.48" size="1.778" layer="95" rot="R90" xref="yes"/>
 </segment>
 </net>
@@
 <label x="-104.14" y="-5.08" size="1.778" layer="95"/>
 </segment>
-</net>
+<segment>
+<label x="6.35" y="40.64" size="1.778" layer="95"/>
+<pinref part="D1" gate="G$1" pin="-"/>
+<wire x1="20.32" y1="40.64" x2="13.97" y2="40.64" width="0.1524" layer="91"/>
+<wire x1="20.32" y1="35.56" x2="20.32" y2="40.64" width="0.1524" layer="91"/>
+<pinref part="R2" gate="G$1" pin="2"/>
+<wire x1="24.13" y1="40.64" x2="20.32" y2="40.64" width="0.1524" layer="91"/>
+<junction x="20.32" y="40.64"/>
+</segment>
+</net>
+<net name="X_MIN_LED" class="0">
+<segment>
+<pinref part="R1" gate="G$1" pin="1"/>
+<pinref part="D1" gate="G$1" pin="+"/>
+<wire x1="15.24" y1="26.67" x2="20.32" y2="26.67" width="0.1524" layer="91"/>
+<wire x1="20.32" y1="26.67" x2="20.32" y2="27.94" width="0.1524" layer="91"/>
+</segment>
+</net>
+<net name="X_PULLDOWN" class="0">
+<segment>
+<pinref part="X_MIN" gate="G$1" pin="COM"/>
+<pinref part="R2" gate="G$1" pin="1"/>
+<wire x1="34.29" y1="40.64" x2="31.75" y2="40.64" width="0.1524" layer="91"/>
+</segment>
+</net>
