File: Eagle_Files/Extruder_Board2.0.0.brd (EAGLE design)
At the start: 42.6 x 46.5 mm, 61 parts, among them J2 FFC_MOLEX_0.5MM, U1 ATMEGA48PA-MMHR28M1-L, U2 MCP6001T-I/OTSOT-23-5_MC-L, U3 LM358PWRDFN-8

Commit message: Brought FFC board up to v2.x spec.
Still ToDo: route traces for PT100 input to amp
Parts:
- removed A_OUT: TPTP10R, PiezoFFC:TP10R
- removed R17: 3.3K, PiezoFFC:R0402
- removed U2: MCP6001T-I/OTSOT-23-5_MC-L, PiezoFFC:SOT-23-5_MC-L
- removed U3: LM358PWRDFN-8, PiezoFFC:SON50P200X200X60-9N
- added C10, C11, C8, C9: 0.1uF, PiezoFFC:CAPC1005X50
- added C12: 1uF, PiezoFFC:CAPC1005X50
- added C13: 10nF, PiezoFFC:CAPC1005X50
- added C4, C6: 10uF, PiezoFFC:CAPC1005X50
- added C5, C7: 3.3uF, PiezoFFC:CAPC1609X80
- added PT100: CON-MOLEX-2P-1.27MM048, PiezoFFC:53048-02
- added PZ+: TPTP13SQ, PiezoFFC:TP13SQ
- added R14: 2K2, PiezoFFC:R0402
- added U4: LM2902QT, PiezoFFC:QFN16
- ADJ+, ADJ-: value TPTP10R -> TPTP13SQ; device PiezoFFC:TP10R -> PiezoFFC:TP13SQ
- D1: value 1N4148DFN-1006-2 -> ZENER_DIODE_PLZ5V1C; device PiezoFFC:DIOC1006X70 -> PiezoFFC:DO-219AC
- H1, H2, H3: value HOLES_MOUNT-PAD-ROUND2.8 -> HOLES_MOUNT-PAD-ROUND3.2; device PiezoFFC:HOLES_2,8-PAD -> PiezoFFC:HOLES_3,2-PAD
- R11, R7: value 220R -> 10K
- R12: value 330R -> 2K2
- R15: value 680R -> 100R
- R4: value 10K -> 1K; device PiezoFFC:R0402 -> PiezoFFC:EXBN8V
- R5: value 330R -> 10K; device PiezoFFC:R0402 -> PiezoFFC:SEEED-RESISTOR_R0603
- R6: value (none) -> 4.7k
- R9: value 470R -> 1K
- moved R6 22.2 mm to (15.7, 41.7), turned to 180 degrees
- moved ADJ- 22.1 mm to (37.1, 29.7), flipped to the bottom, turned to 225 degrees
- moved R15 13.8 mm to (18.4, 16.5), flipped to the bottom, turned to 270 degrees
- moved R7 10.7 mm to (11.5, 15.8), flipped to the bottom, turned to 0 degrees
- moved R4 10.6 mm to (18.0, 24.0), turned to 0 degrees
- moved R12 9.59 mm to (10.4, 15.8), flipped to the bottom, turned to 180 degrees
- moved R11 9.04 mm to (13.0, 15.8), flipped to the bottom, turned to 0 degrees
- moved ADJ+ 7.46 mm to (38.3, 28.5), flipped to the bottom, turned to 45 degrees
- moved R2 6.84 mm to (30.4, 29.0), turned to 180 degrees
- moved R1 6.11 mm to (29.0, 29.4)
- moved R10 4.24 mm to (30.1, 23.0), turned to 270 degrees
- moved R19 4.13 mm to (33.5, 26.5), turned to 315 degrees
- moved D1 3.63 mm to (14.1, 29.6), turned to 270 degrees
- moved R13 3.18 mm to (25.7, 31.1)
- moved R5 2.73 mm to (21.3, 21.3), turned to 90 degrees
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Connections:
- removed net COMP-: ADJ+.TP, R1.2, R2.2, U2.1, U3.2
- removed net VADJ_R0: R11.2, R7.1, U1.5
- removed net VADJ_R1: R11.1, R12.2, U1.6
- removed net VADJ_R2: R12.1, R5.2, U1.7
- removed net VADJ_R3: R5.1, R9.2, U1.8
- removed net VADJ_SENSE: ADJ-.TP, R15.2, R7.2, U1.20, U3.3
- removed net V_FOLLOW: R1.1, U1.19, U3.6, U3.7
- new net GADJ_R0: R4.2, R4.8, U1.5
- new net GADJ_R1: R4.3, R4.7, U1.6
- new net GADJ_R2: R4.4, R4.6, U1.7
- new net GADJ_R3: R4.5, R9.2, U1.8
- new net GAIN_OUT: ADJ-.TP, R1.2, R2.2, U4.14, U4.16
- new net PT100+: C8.1, PT100.1, R12.1, R7.2
- new net PT100-: C9.2, PT100.2, R11.2, R14.2
- new net PT100_AMP+: C10.1, C12.2, R7.1, U4.4
- new net PT100_AMP-: C11.2, C12.1, R11.1, U4.5
- new net PT100_OUT: C13.2, R15.1
- new net PT100_R: R15.2, U4.6
- new net VCOMP_PWM: R5.2, U1.11
- new net VCOMP_SENSE: ADJ+.TP, C6.2, C7.2, R5.1, U1.20, U4.1
- new net V_FOL_PWM: R10.2, U1.1
- new net V_FOL_SENSE: R1.1, U1.19, U4.7, U4.8
- net +5V: now also U4.2; no longer R10.2, R15.1, U2.5, U3.8
- net ERR_LED: now also U1.2; no longer U1.1
- net GAIN_FB: now also R4.1, U4.13; no longer R17.2, U2.4
- net GND: now also C11.1, C13.1, C4.1, C5.1, C6.1, C7.1, C9.1, D1.P$1, H1.B3,2, H2.B3,2, H3.B3,2, PZ1.2, R14.1, U4.11; no longer D1.A, H1.B2,8, H2.B2,8, H3.B2,8, PZ1.1, R17.1, R4.1, U2.2, U3.4
- net PZ+: now also PZ+.TP, PZ1.1, U4.12; no longer PZ1.2, U2.3
- net PZ_AMP_OUT: now also U4.15; no longer A_OUT.TP, U3.1
- net RST: now also J2.38
- net SCL: now also J2.41
- net SDA: now also J2.42
- net TTL_RXD: now also J2.39
- net TTL_TXD: now also J2.40
- net VCC_REG: now also C10.2, C8.2, D1.P$2, R12.2; no longer D1.C
- net VREF_IN: now also C4.2, C5.2, U4.9; no longer R4.2, U3.5
- net Z_MIN_TRIG: now also U1.9; no longer U1.11
Routing:
- net VCOMP_SENSE: track 0.00 -> 38.7 mm, vias 0 -> 3
- net SCL: track 14.9 -> 46.3 mm, vias 1 -> 2
- net TRG_LED: track 51.4 -> 25.3 mm, vias 3 -> 2
- net SDA: track 16.0 -> 41.9 mm, vias 1 -> 3
- net VADJ_SENSE: track 21.6 -> 0.00 mm, vias 2 -> 0
- net TTL_TXD: track 15.5 -> 34.4 mm
- net RST: track 59.5 -> 77.9 mm
- net TTL_RXD: track 13.9 -> 32.3 mm
- net V_FOL_SENSE: track 0.00 -> 15.5 mm, vias 0 -> 3
- net V_FOL_PWM: track 0.00 -> 12.6 mm, vias 0 -> 2
- net GAIN_OUT: track 0.00 -> 12.3 mm, vias 0 -> 1
- net Z_MIN_TRIG: track 32.2 -> 44.4 mm
- net VCC_REG: track 43.3 -> 54.0 mm, vias 3 -> 4
- net COMP-: track 8.87 -> 0.00 mm, vias 1 -> 0
- net GAIN_FB: track 12.7 -> 21.4 mm, vias 3 -> 4
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
Commit message: Added pin assignments for serial/i2c comms on FFC
Builds necessary back-channel for https://github.com/pyr0ball/pyr0piezo/issues/2
Also added pin assignments used in https://github.com/pyr0ball/pyr0piezo/issues/18
Parts:
- moved C13 6.72 mm to (11.5, 19.6)
- moved R15 5.91 mm to (13.1, 19.1)
- moved R6 4.60 mm to (12.8, 38.1)
Connections:
- new net X_1A: J2.47, J2.48
- new net X_1B: J2.49, J2.50
- new net X_2A: J2.45, J2.46
- new net X_2B: J2.43, J2.44
- new net X_MIN_TRIG: J2.34
- net PT100_OUT: now also J2.33
- net Z_MIN_TRIG: now also J2.35; no longer J2.50
Routing:
- net PT100_AMP+: track 2.33 -> 37.2 mm, vias 0 -> 3
- net PT100_AMP-: track 2.33 -> 32.6 mm, vias 0 -> 3
- net PT100_R: track 2.21 -> 31.2 mm, vias 1 -> 3
- net Z_MIN_TRIG: track 44.4 -> 34.0 mm, vias 1 -> 2
- net PT100_OUT: track 0.00 -> 9.69 mm, vias 0 -> 2
- net RST: track 77.9 -> 70.3 mm
- net ERR_LED: track 22.9 -> 28.8 mm
- net TRG_LED: track 25.3 -> 30.0 mm
- net LED_VCC: track 29.1 -> 33.0 mm
- net VCC: track 23.3 -> 25.8 mm
- net HE0-: track 24.6 -> 22.5 mm
- net V_FOL_SENSE: track 15.5 -> 13.6 mm
- net GAIN_FB: track 21.4 -> 22.1 mm
- net GAIN_OUT: track 12.3 -> 13.0 mm
- net GND: vias 62 -> 72

Commit message: Updated library and components
Parts:
- U1: value ATMEGA48PA-MMHR28M1-L -> ATMEGA48/88/168/328PA; device PiezoFFC:28M1-L -> PiezoFFC:28M1
