File: Eagle_Files/PiezoStandalone_PT100_2.0.0.brd (EAGLE design)
At the start: 43 x 15.4 mm, 71 parts, among them J1 CON-MOLEX-4P-1.25MM048, U1 ATMEGA48PA-MMHR28M1-L, U2 L78L05ACU, U3 LM2902QT

Commit message: Swapped/repositioned components
 - Swapped individual 0402 resistors for 4x array. related to https://github.com/pyr0ball/pyr0piezo/issues/16
 - repositioned LPF capacitors for easier installation. related to https://github.com/pyr0ball/pyr0piezo/issues/15
Parts:
- removed R11, R12, R13, R9: 470R, PiezoFFC:R0402
- added RP1: 1K, PiezoFFC:EXBN8V-L
- moved C15 0.67 mm to (25.2, 1.81)
- moved C14 0.67 mm to (25.2, 2.64)
- moved R14 0.50 mm to (14.7, 2.65)
Connections:
- net GADJ_R0: now also RP1.2, RP1.8; no longer R11.1, R9.2
- net GADJ_R1: now also RP1.3, RP1.7; no longer R11.2, R12.1
- net GADJ_R2: now also RP1.4, RP1.6; no longer R12.2, R13.1
- net GADJ_R3: now also RP1.5; no longer R13.2
- net GAIN_ADJ: now also RP1.1; no longer R9.1
Routing:
- net GADJ_R0: track 28.5 -> 3.16 mm, vias 3 -> 0
- net GAIN_ADJ: track 2.91 -> 26.8 mm, vias 1 -> 4
- net VCOMP_SENSE: track 8.45 -> 9.82 mm
- net GADJ_R2: track 3.82 -> 3.11 mm

Commit message: Minor adjustments to silkscreen and traces
Parts:
- moved R16 0.38 mm to (15.6, 8.94)
- moved D1 0.06 mm to (14.1, 8.13)
Routing:
- net GND: track 3.67 -> 3.94 mm, vias 29 -> 31

Commit message: Added test pads for amp circuit debug
Parts:
- added ADJ+, ADJ-, PZ+: TPTP13SQ, PiezoFFC:TP13SQ
- moved R1 3.18 mm to (33.0, 9.20)
- moved R22 1.86 mm to (28.4, 5.75)
Connections:
- net GAIN_OUT: now also ADJ-.TP
- net PZ+: now also PZ+.TP
- net VCOMP_SENSE: now also ADJ+.TP
Routing:
- net GAIN_OUT: track 9.86 -> 22.0 mm
- net PZ+: track 11.8 -> 14.5 mm
- net PT100_JUMP: track 1.74 -> 4.29 mm
- net PT_AMP: track 3.56 -> 1.62 mm
- net GND: track 3.94 -> 5.63 mm

Commit message: Finished trace routing for amp diagnostics pads
Parts:
- moved ADJ+ 12.2 mm to (34.6, 13.4), turned to 90 degrees
- moved R20 1.80 mm to (35.1, 4.45), turned to 315 degrees
- moved R19 1.75 mm to (37.8, 7.08), turned to 135 degrees
- moved R18 0.85 mm to (34.0, 6.79)
- moved C6 0.83 mm to (34.6, 6.16)
- moved C5 0.81 mm to (36.1, 7.68)
- moved C8 0.81 mm to (36.8, 8.89)
- moved R17 0.81 mm to (35.5, 8.26)
- moved C9 0.76 mm to (33.3, 5.52)
- moved R1 0.19 mm to (33.1, 9.39)
Routing:
- net VCOMP_SENSE: track 9.82 -> 25.5 mm, vias 0 -> 1
- net PT_AMP-: track 7.03 -> 8.78 mm
- net +5V: track 68.1 -> 69.3 mm, vias 11 -> 10
- net GAIN_OUT: track 22.0 -> 21.0 mm
- net PT_IN-: track 6.87 -> 6.10 mm
- net PT_IN+: track 5.36 -> 6.13 mm
- net PT_AMP+: track 12.3 -> 12.9 mm
- net GND: track 5.63 -> 5.43 mm, vias 31 -> 33

Commit message: fixed some spacing and labelling
Parts:
- U1: value ATMEGA48PA-MMHR28M1-L -> ATMEGA48/88/168PA-MMHR28M1-L
Changed lines of the file:
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@@
 <drawing>
 <settings>
-<setting alwaysvectorfont="yes"/>
+<setting alwaysvectorfont="no"/>
 <setting verticaltext="up"/>
 </settings>
@@
 <attribute name="OC_NEWARK" value="57H4718" x="66.073890625" y="-12.06810625" size="1.778" layer="27" display="off"/>
 </element>
-<element name="U1" library="PiezoFFC" library_urn="urn:adsk.eagle:library:6897166" package="28M1-L" package3d_urn="urn:adsk.eagle:package:6899182/3" value="ATMEGA48PA-MMHR28M1-L" x="18.74879375" y="5.1375" smashed="yes">
+<element name="U1" library="PiezoFFC" library_urn="urn:adsk.eagle:library:6897166" package="28M1-L" package3d_urn="urn:adsk.eagle:package:6899182/3" value="ATMEGA48/88/168PA-MMHR28M1-L" x="18.74879375" y="5.1375" smashed="yes">
 <attribute name="MANUFACTURER_PART_NUMBER" value="ATMEGA48PAMMHR" x="35.2587875" y="-27.88249375" size="1.778" layer="27" display="off"/>
 <attribute name="NAME" x="16.290003125" y="6.258609375" size="1.016" layer="25" font="vector" ratio="11" rot="SR90"/>
@@
 <contactref element="PWR" pad="-"/>
 <contactref element="U1" pad="29"/>
-<contactref element="D8" pad="1"/>
 <contactref element="J1" pad="1"/>
 <contactref element="R1" pad="1"/>
@@
 <via x="29.0302125" y="9.147590625" extent="1-16" drill="0.3"/>
 <via x="33.898034375" y="5.425315625" extent="1-16" drill="0.3"/>
+<contactref element="D8" pad="1"/>
+<wire x1="38.766546875" y1="7.419521875" x2="39.94364375" y2="11.4935125" width="0" layer="19" extent="1-1"/>
+<wire x1="34.820215625" y1="4.772034375" x2="38.766546875" y2="7.419521875" width="0" layer="19" extent="16-16"/>
+<wire x1="33.898034375" y1="5.425315625" x2="34.820215625" y2="4.772034375" width="0" layer="19" extent="16-16"/>
+<wire x1="33.69105625" y1="5.17094375" x2="33.898034375" y2="5.425315625" width="0" layer="19" extent="16-16"/>
+<wire x1="34.222196875" y1="5.80594375" x2="33.898034375" y2="5.425315625" width="0" layer="19" extent="16-16"/>
+<wire x1="31.9512125" y1="6.290090625" x2="33.69105625" y2="5.17094375" width="0" layer="19" extent="16-16"/>
+<wire x1="32.1734625" y1="8.417340625" x2="31.9512125" y2="6.290090625" width="0" layer="19" extent="1-1"/>
+<wire x1="33.51671875" y1="9.386246875" x2="32.1734625" y2="8.417340625" width="0" layer="19" extent="16-16"/>
+<wire x1="34.025034375" y1="2.790065625" x2="34.820215625" y2="4.772034375" width="0" layer="19" extent="16-16"/>
+<wire x1="31.096790625" y1="11.617" x2="33.678890625" y2="10.811884375" width="0" layer="19" extent="1-1"/>
+<wire x1="29.977978125" y1="12.369921875" x2="31.096790625" y2="11.617" width="0" layer="19" extent="1-1"/>
+<wire x1="29.434621875" y1="13.405528125" x2="29.977978125" y2="12.369921875" width="0" layer="19" extent="1-16"/>
+<wire x1="29.454828125" y1="13.436321875" x2="29.434621875" y2="13.405528125" width="0" layer="19" extent="16-16"/>
+<wire x1="27.860271875" y1="10.14383125" x2="29.977978125" y2="12.369921875" width="0" layer="19" extent="1-1"/>
+<wire x1="27.1065" y1="10.0965" x2="27.860271875" y2="10.14383125" width="0" layer="19" extent="1-1"/>
+<wire x1="28.538275" y1="9.558828125" x2="27.860271875" y2="10.14383125" width="0" layer="19" extent="16-16"/>
+<wire x1="29.0302125" y1="9.147590625" x2="28.538275" y2="9.558828125" width="0" layer="19" extent="16-16"/>
+<wire x1="27.1065" y1="9.2075" x2="27.1065" y2="10.0965" width="0" layer="19" extent="1-1"/>
+<wire x1="26.32475" y1="7.824546875" x2="27.1065" y2="9.2075" width="0" layer="19" extent="1-1"/>
+<wire x1="26.0585" y1="11.4615" x2="27.1065" y2="10.0965" width="0" layer="19" extent="1-16"/>
+<wire x1="24.365790625" y1="11.58525" x2="26.0585" y2="11.4615" width="0" layer="19" extent="16-16"/>
+<wire x1="24.3377125" y1="8.683" x2="26.32475" y2="7.824546875" width="0" layer="19" extent="1-1"/>
+<wire x1="22.085690625" y1="11.054646875" x2="24.365790625" y2="11.58525" width="0" layer="19" extent="1-1"/>
+<wire x1="21.8929625" y1="6.74625" x2="24.3377125" y2="8.683" width="0" layer="19" extent="1-1"/>
+<wire x1="20.65379375" y1="5.1375" x2="21.8929625" y2="6.74625" width="0" layer="19" extent="1-1"/>
+<wire x1="19.553796875" y1="4.353503125" x2="20.65379375" y2="5.1375" width="0" layer="19" extent="1-1"/>
+<wire x1="18.74879375" y1="5.1375" x2="19.553796875" y2="4.353503125" width="0" layer="19" extent="1-1"/>
+<wire x1="17.3275" y1="6.1595" x2="18" y2="5.925" width="0" layer="19" extent="16-16"/>
+<wire x1="19.54579375" y1="5.937496875" x2="18.74879375" y2="5.1375" width="0" layer="19" extent="1-1"/>
+<wire x1="16.84379375" y1="5.1375" x2="17.3275" y2="6.1595" width="0" layer="19" extent="1-16"/>
+<wire x1="22.4938125" y1="4.122353125" x2="20.65379375" y2="5.1375" width="0" layer="19" extent="1-1"/>
+<wire x1="18.160040625" y1="2.22225625" x2="17.970796875" y2="4.338" width="0" layer="19" extent="1-1"/>
+<wire x1="16.348640625" y1="2.5238875" x2="18.160040625" y2="2.22225625" width="0" layer="19" extent="1-1"/>
+<wire x1="14.26925" y1="2.655" x2="16.348640625" y2="2.5238875" width="0" layer="19" extent="1-1"/>
+<wire x1="14.1962625" y1="2.232121875" x2="14.26925" y2="2.655" width="0" layer="19" extent="1-1"/>
+<wire x1="12.69805" y1="1.758375" x2="14.1962625" y2="2.232121875" width="0" layer="19" extent="1-1"/>
+<wire x1="11.03469375" y1="2.45573125" x2="12.69805" y2="1.758375" width="0" layer="19" extent="1-1"/>
+<wire x1="10.899503125" y1="2.494853125" x2="11.03469375" y2="2.45573125" width="0" layer="19" extent="16-16"/>
+<wire x1="11.064796875" y1="3.2775" x2="10.899503125" y2="2.494853125" width="0" layer="19" extent="1-16"/>
+<wire x1="9.58655" y1="1.726625" x2="10.899503125" y2="2.494853125" width="0" layer="19" extent="16-16"/>
+<wire x1="7.971815625" y1="1.85769375" x2="9.58655" y2="1.726625" width="0" layer="19" extent="1-1"/>
+<wire x1="9.491503125" y1="4.70979375" x2="11.064796875" y2="3.2775" width="0" layer="19" extent="1-16"/>
+<wire x1="9.6242625" y1="4.899121875" x2="9.491503125" y2="4.70979375" width="0" layer="19" extent="16-16"/>
+<wire x1="11.064796875" y1="5.9445" x2="9.6242625" y2="4.899121875" width="0" layer="19" extent="1-1"/>
+<wire x1="24.728946875" y1="4.59944375" x2="22.4938125" y2="4.122353125" width="0" layer="19" extent="16-16"/>
+<wire x1="24.849284375" y1="4.377565625" x2="24.728946875" y2="4.59944375" width="0" layer="19" extent="16-16"/>
+<wire x1="25.862175" y1="3.175" x2="24.849284375" y2="4.377565625" width="0" layer="19" extent="1-1"/>
+<wire x1="25.67775" y1="1.80975" x2="25.67775" y2="2.63525" width="0" layer="19" extent="1-1"/>
+<wire x1="28.575" y1="4.0005" x2="26.3605" y2="3.175" width="0" layer="19" extent="1-16"/>
+<wire x1="17.0990875" y1="9.21365625" x2="17.3275" y2="6.1595" width="0" layer="19" extent="16-16"/>
+<wire x1="14.200259375" y1="9.285609375" x2="17.0990875" y2="9.21365625" width="0" layer="19" extent="1-1"/>
+<wire x1="14.097" y1="9.278" x2="14.200259375" y2="9.285609375" width="0" layer="19" extent="1-1"/>
+<wire x1="18.421559375" y1="11.894896875" x2="17.0990875" y2="9.21365625" width="0" layer="19" extent="1-1"/>
+<wire x1="16.31975" y1="13.45413125" x2="18.421559375" y2="11.894896875" width="0" layer="19" extent="1-1"/>
+<wire x1="16.2445" y1="13.463" x2="16.31975" y2="13.45413125" width="0" layer="19" extent="16-16"/>
+<wire x1="4.463853125" y1="3.59795625" x2="7.971815625" y2="1.85769375" width="0" layer="19" extent="1-1"/>
+<wire x1="11.814225" y1="13.350271875" x2="16.2445" y2="13.463" width="0" layer="19" extent="16-16"/>
+<wire x1="10.80020625" y1="12.843159375" x2="11.814225" y2="13.350271875" width="0" layer="19" extent="16-16"/>
+<wire x1="10.2730125" y1="11.809059375" x2="10.80020625" y2="12.843159375" width="0" layer="19" extent="16-16"/>
+<wire x1="9.63870625" y1="10.205940625" x2="10.2730125" y2="11.809059375" width="0" layer="19" extent="16-16"/>
 </signal>
 <signal name="Z_MIN_TRIG">

Commit message: aligned caps for easier soldering
Parts:
- U1: value ATMEGA48/88/168PA-MMHR28M1-L -> ATMEGA48/88/168/328PA28M1-L
- moved C1 2.22 mm to (10.9, 5.42)
Routing:
- net +5V: track 69.3 -> 67.5 mm

Commit message: repositioned filter cap for easier soldering
Parts:
- moved C7 0.44 mm to (28.8, 4.22)
- moved C10 0.19 mm to (27.1, 3.17)
Routing:
- net PT_AMP+: track 12.9 -> 12.4 mm
