File: Eagle_Files/PiezoStandalone_PT100_2.0.0.sch (EAGLE design)
At the start: 69 parts, among them J1 CON-MOLEX-4P-1.25MM048, U1 ATMEGA48PA-MMHR28M1-L, U2 L78L05ACU, U3 LM2902QT

Commit message: Finished first iteration of x-gantry board
First version to address https://github.com/pyr0ball/pyr0piezo/issues/18
Changed lines of the file:
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@@
 <?xml version="1.0" encoding="utf-8"?>
 <!DOCTYPE eagle SYSTEM "eagle.dtd">
-<eagle version="9.3.1">
+<eagle version="9.3.0">
 <drawing>
 <settings>
@@
 </instance>
 <instance part="J2" gate="G$1" x="262.89" y="44.45" smashed="yes">
-<attribute name="NAME" x="259.08" y="45.72" size="1.27" layer="95" ratio="10"/>
+<attribute name="NAME" x="261.62" y="45.72" size="1.27" layer="95" ratio="10"/>
 <attribute name="VALUE" x="259.08" y="41.91" size="1.27" layer="96" ratio="10"/>
 </instance>

Commit message: fixed some spacing and labelling
Parts:
- U1: value ATMEGA48PA-MMHR28M1-L -> ATMEGA48/88/168PA-MMHR28M1-L; device PiezoFFC:ATMEGA48PA-MMHR28M1-L -> PiezoFFC:ATMEGA48/88/168PA-MMHR28M1-L
Other:
- note added: "ATMega88/168/328"
- note removed: "ATMega48"
- moved on the sheet: ADJ+, ADJ-, C10, C12, C13, C14, C15, C3, D8, R1, R10, R14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

Commit message: aligned caps for easier soldering
Parts:
- U1: value ATMEGA48/88/168PA-MMHR28M1-L -> ATMEGA48/88/168/328PA28M1-L; device PiezoFFC:ATMEGA48/88/168PA-MMHR28M1-L -> PiezoFFC:ATMEGA48/88/168/328PA28M1-L
Changed lines of the file:
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@@
 <parts>
 <part name="PZ1" library="PiezoFFC" library_urn="urn:adsk.eagle:library:6897166" deviceset="CON-MOLEX-2P-1.27MM" device="048" package3d_urn="urn:adsk.eagle:package:5807562/3"/>
-<part name="U1" library="PiezoFFC" library_urn="urn:adsk.eagle:library:6897166" deviceset="ATMEGA48/88/168PA-MMHR" device="28M1-L" package3d_urn="urn:adsk.eagle:package:6899182/3"/>
+<part name="U1" library="PiezoFFC" library_urn="urn:adsk.eagle:library:6897166" deviceset="ATMEGA48/88/168/328PA" device="28M1-L" package3d_urn="urn:adsk.eagle:package:6899182/3"/>
 <part name="U2" library="PiezoFFC" library_urn="urn:adsk.eagle:library:6897166" deviceset="L78L05ACU" device="" package3d_urn="urn:adsk.eagle:package:6899241/5"/>
 <part name="SUPPLY2" library="supply2" library_urn="urn:adsk.eagle:library:372" deviceset="GND" device=""/>
