File: Eagle_Files/FFC_Direct_Breakout/Pyr0-Piezo_Direct-Extruder-FFC-Breakout_1.0.0.brd (EAGLE design)
At the start: 53.3 x 63.9 mm, 30 parts, among them J1 SFW24R-1STE1LF, Q2 2N2907, U1 LM317DCY, U2 L78L05ACU

Commit message: Standardized naming conventions, organized
Moved each set of board files to individual folders
Parts:
- F1: value 500mA -> 2K
- R6: value 1R -> 2K
- R7: value 10R -> 2K
Changed lines of the file:
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@@
 <?xml version="1.0" encoding="utf-8"?>
 <!DOCTYPE eagle SYSTEM "eagle.dtd">
-<eagle version="9.3.0">
+<eagle version="9.3.1">
 <drawing>
 <settings>
-<setting alwaysvectorfont="yes"/>
+<setting alwaysvectorfont="no"/>
 <setting verticaltext="up"/>
 </settings>
@@
 <attribute name="VENDOR" value="FCI" x="43.18" y="66.44" size="1.778" layer="28" rot="MR90" display="off"/>
 </element>
-<element name="U1" library="PiezoFFC" library_urn="urn:adsk.eagle:library:6897166" package="SOT230P700X180-4N" package3d_urn="urn:adsk.eagle:package:7346255/2" value="LM317DCY" x="26.56" y="34.6" smashed="yes">
+<element name="U1" library="PiezoFFC" library_urn="urn:adsk.eagle:library:6897166" package="SOT230P700X180-4N" package3d_urn="urn:adsk.eagle:package:7346255/3" value="LM317DCY" x="26.56" y="34.6" smashed="yes">
 <attribute name="AVAILABILITY" value="Unavailable" x="26.56" y="34.6" size="1.778" layer="27" display="off"/>
 <attribute name="DESCRIPTION" value=" IC Regulator LM317/SOT223/LM317DCY TEXAS INSTRUMENT RoHS Ampere=1.5 SOT223 " x="26.56" y="34.6" size="1.778" layer="27" display="off"/>
@@
 <attribute name="VALUE" x="30.37" y="44.76" size="1.27" layer="27" rot="R270"/>
 </element>
-<element name="U2" library="PiezoFFC" library_urn="urn:adsk.eagle:library:6897166" package="SOT89" package3d_urn="urn:adsk.eagle:package:6899241/5" value="L78L05ACU" x="22.723" y="17.828" smashed="yes" rot="R180">
+<element name="U2" library="PiezoFFC" library_urn="urn:adsk.eagle:library:6897166" package="SOT89" package3d_urn="urn:adsk.eagle:package:6899241/6" value="L78L05ACU" x="22.723" y="17.828" smashed="yes" rot="R180">
 <attribute name="AVAILABILITY" value="Unavailable" x="22.723" y="17.828" size="1.778" layer="27" rot="R180" display="off"/>
 <attribute name="DESCRIPTION" value=" Voltage regulator; fixed; 5V; 0.1A; SOT89; SMD; Package: reel, tape " x="22.723" y="17.828" size="1.778" layer="27" rot="R180" display="off"/>
@@
 <attribute name="NAME" x="20.321" y="30.532" size="1.27" layer="25" font="vector" ratio="11" rot="R180"/>
 </element>
-<element name="R6" library="PiezoFFC" library_urn="urn:adsk.eagle:library:6897166" package="R0805" package3d_urn="urn:adsk.eagle:package:8443791/2" value="1R" x="16.56" y="19.824" smashed="yes">
+<element name="R6" library="PiezoFFC" library_urn="urn:adsk.eagle:library:6897166" package="R0805" package3d_urn="urn:adsk.eagle:package:8443791/3" value="2K" x="16.56" y="19.824" smashed="yes">
 <attribute name="MPN" value="RC0805JR-072KL" x="10.21" y="26.174" size="1.778" layer="27" display="off"/>
 <attribute name="NAME" x="16.425" y="20.829" size="0.889" layer="25" font="vector" ratio="11"/>
 <attribute name="VALUE" x="17.511" y="18.917" size="0.889" layer="21" font="vector" ratio="11" rot="R180"/>
 </element>
-<element name="R7" library="PiezoFFC" library_urn="urn:adsk.eagle:library:6897166" package="R0805" package3d_urn="urn:adsk.eagle:package:8443791/2" value="10R" x="19.33" y="21.234" smashed="yes" rot="R90">
+<element name="R7" library="PiezoFFC" library_urn="urn:adsk.eagle:library:6897166" package="R0805" package3d_urn="urn:adsk.eagle:package:8443791/3" value="2K" x="19.33" y="21.234" smashed="yes" rot="R90">
 <attribute name="MPN" value="RC0805JR-072KL" x="11.71" y="14.884" size="1.778" layer="27" rot="R90" display="off"/>
 <attribute name="NAME" x="20.175" y="22.601" size="0.889" layer="25" font="vector" ratio="11" rot="R270"/>
@@
 <element name="H3" library="PiezoFFC" library_urn="urn:adsk.eagle:library:6897166" package="HOLES_3,2-PAD" package3d_urn="urn:adsk.eagle:package:5224590/2" value="HOLES_MOUNT-PAD-ROUND3.2" x="48.26" y="5.18" smashed="yes"/>
 <element name="H4" library="PiezoFFC" library_urn="urn:adsk.eagle:library:6897166" package="HOLES_3,2-PAD" package3d_urn="urn:adsk.eagle:package:5224590/2" value="HOLES_MOUNT-PAD-ROUND3.2" x="48.26" y="58.82" smashed="yes"/>
-<element name="F1" library="PiezoFFC" library_urn="urn:adsk.eagle:library:6897166" package="R0805" package3d_urn="urn:adsk.eagle:package:8443791/2" value="500mA" x="28.5" y="20" smashed="yes" rot="R180">
+<element name="F1" library="PiezoFFC" library_urn="urn:adsk.eagle:library:6897166" package="R0805" package3d_urn="urn:adsk.eagle:package:8443791/3" value="2K" x="28.5" y="20" smashed="yes" rot="R180">
 <attribute name="MPN" value="RC0805JR-072KL" x="34.5" y="13" size="1.778" layer="27" rot="R180" display="off"/>
 <attribute name="NAME" x="27.895" y="20.916" size="0.889" layer="25" font="vector" ratio="11"/>
