File: Eagle_Files/FFC_Direct_Breakout/Pyr0-Piezo_Direct-Extruder-FFC-Breakout_2.0.1.brd (EAGLE design)
At the start: 64.8 x 63.9 mm, 34 parts, among them J1 FFC_MOLEX_0.5MM, Q2 2N2907, U1 LM317DCY, U2 L78L05ACU

Commit message: Added ESD protection diodes to motor connections
Parts:
- added D1, D10, D11, D12, D13, D14, D15, D16, D2, D3, D4, D5, D6, D7, D8, D9: DIODE_SCHOTTKY_SINGLE, PiezoFFC:DO-214AC
- Q2: value 2N2907 -> (none); device PiezoFFC:TO92 -> PiezoFFC:SOT23-BEC
- R5: value 0R -> 2K
- R6: value 1R -> 2K
- R7: value 10R -> 2K
- moved C3 4.12 mm to (27.2, 26.3), turned to 0 degrees
- moved Q2 0.23 mm to (17.3, 24.1), turned to 270 degrees
Connections:
- net +5V: now also Q2.C; no longer Q2.1
- net AGND: now also D1.A, D11.A, D13.A, D15.A, D3.A, D5.A, D7.A, D9.A
- net BYP_GATE: now also Q2.B; no longer Q2.2
- net E0_1A: now also D13.C, D14.A
- net E0_1B: now also D15.C, D16.A
- net E0_2A: now also D11.C, D12.A
- net E0_2B: now also D10.A, D9.C
- net VCC: now also D10.C, D12.C, D14.C, D16.C, D2.C, D4.C, D6.C, D8.C, Q2.E; no longer Q2.3
- net X_1A: now also D5.C, D6.A
- net X_1B: now also D7.C, D8.A
- net X_2A: now also D3.C, D4.A
- net X_2B: now also D1.C, D2.A
Routing:
- net VCC: track 148.1 -> 203.9 mm, vias 1 -> 2
- net X_1B: track 27.4 -> 53.6 mm
- net E0_1B: track 11.7 -> 28.4 mm
- net X_2A: track 33.3 -> 49.4 mm
- net E0_2A: track 17.1 -> 32.5 mm
- net X_1A: track 30.3 -> 39.4 mm
- net E0_1A: track 14.2 -> 22.4 mm
- net E0_2B: track 20.1 -> 28.2 mm
- net X_2B: track 36.2 -> 43.9 mm
- net +5V: track 16.9 -> 20.2 mm
- net BYP_GATE: track 6.28 -> 5.67 mm

Commit message: Beta production board sync
Routing:
- net VCC: track 203.9 -> 208.1 mm
- net HE0-: track 65.5 -> 66.5 mm
Changed lines of the file:
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@@
 <wire x1="52" y1="42.5" x2="47.5" y2="47" width="1.27" layer="1" curve="90"/>
 <wire x1="47.5" y1="47" x2="19" y2="47" width="1.27" layer="1"/>
-<wire x1="59.25" y1="39.25" x2="59.25" y2="39.75" width="0" layer="19" extent="1-1"/>
-<wire x1="58.75" y1="38" x2="59.25" y2="38" width="0" layer="19" extent="1-1"/>
+<wire x1="59.25" y1="39.75" x2="59.25" y2="39.25" width="0.1524" layer="1"/>
+<wire x1="59.25" y1="38" x2="58.75" y2="38" width="0.1524" layer="1"/>
 </signal>
 <signal name="VCC">
@@
 <wire x1="59.25" y1="46.25" x2="59.25" y2="46.75" width="0.1524" layer="1"/>
 <wire x1="54.05" y1="51.95" x2="59.25" y2="46.75" width="2.54" layer="1" curve="-90"/>
-<wire x1="59.25" y1="46.75" x2="59.25" y2="42.5" width="2.54" layer="1"/>
+<wire x1="59.25" y1="46.75" x2="59.25" y2="45" width="2.54" layer="1"/>
+<wire x1="59.25" y1="45" x2="59.25" y2="42.5" width="2.54" layer="1"/>
 <wire x1="19.51" y1="50.986" x2="19.5" y2="50.996" width="0.1524" layer="1" curve="-90"/>
 <wire x1="19.5" y1="50.996" x2="19.5" y2="51.95" width="0.1524" layer="1"/>
@@
 <wire x1="16.266" y1="25.666" x2="16.237" y2="25.637" width="0.8128" layer="16"/>
 <wire x1="16.237" y1="25.637" x2="16.237" y2="23.164" width="0.8128" layer="16"/>
-<wire x1="59.25" y1="44.75" x2="59.25" y2="45.25" width="0" layer="19" extent="1-1"/>
-<wire x1="59.25" y1="45.75" x2="59.25" y2="45.25" width="0" layer="19" extent="1-1"/>
-<wire x1="26" y1="16" x2="25.975" y2="16" width="0" layer="19" extent="16-16"/>
+<wire x1="25.975" y1="16" x2="26" y2="16" width="0.1524" layer="16"/>
+<wire x1="59.25" y1="45.75" x2="59.25" y2="45" width="0.1524" layer="1"/>
+<wire x1="59.25" y1="44.75" x2="59.25" y2="46.75" width="0.1524" layer="1"/>
+<wire x1="59.25" y1="45.25" x2="59.25" y2="46.75" width="0.1524" layer="1"/>
 </signal>
 <signal name="AGND">

Commit message: fixed incorrect resistor values on FFC Direct vreg #bugfix
Parts:
- R5: value 2K -> 0R
- R6: value 2K -> 1R
- R7: value 2K -> 10R
Changed lines of the file:
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@@
 <?xml version="1.0" encoding="utf-8"?>
 <!DOCTYPE eagle SYSTEM "eagle.dtd">
-<eagle version="9.3.2">
+<eagle version="9.4.2">
 <drawing>
 <settings>
-<setting alwaysvectorfont="yes"/>
+<setting alwaysvectorfont="no"/>
 <setting verticaltext="up"/>
 </settings>
@@
 <attribute name="NAME" x="21.532" y="23.179" size="1.27" layer="25" font="vector" ratio="11" rot="R90"/>
 </element>
-<element name="R6" library="PiezoFFC" library_urn="urn:adsk.eagle:library:6897166" package="R0805" package3d_urn="urn:adsk.eagle:package:8443791/3" value="2K" x="14.46" y="18.174" smashed="yes">
+<element name="R6" library="PiezoFFC" library_urn="urn:adsk.eagle:library:6897166" package="R0805" package3d_urn="urn:adsk.eagle:package:8443791/3" value="1R" x="14.46" y="18.174" smashed="yes">
 <attribute name="MPN" value="RC0805JR-072KL" x="8.11" y="24.524" size="1.778" layer="27" display="off"/>
 <attribute name="NAME" x="15.075" y="17.221" size="0.889" layer="25" font="vector" ratio="11" rot="R180"/>
 <attribute name="VALUE" x="13.317" y="17.539" size="0.889" layer="21" font="vector" ratio="11" rot="R90"/>
 </element>
-<element name="R7" library="PiezoFFC" library_urn="urn:adsk.eagle:library:6897166" package="R0805" package3d_urn="urn:adsk.eagle:package:8443791/3" value="2K" x="17.33" y="19.114" smashed="yes" rot="R90">
+<element name="R7" library="PiezoFFC" library_urn="urn:adsk.eagle:library:6897166" package="R0805" package3d_urn="urn:adsk.eagle:package:8443791/3" value="10R" x="17.33" y="19.114" smashed="yes" rot="R90">
 <attribute name="MPN" value="RC0805JR-072KL" x="9.71" y="12.764" size="1.778" layer="27" rot="R90" display="off"/>
 <attribute name="NAME" x="16.679" y="20.625" size="0.889" layer="25" font="vector" ratio="11"/>
@@
 <element name="H3" library="PiezoFFC" library_urn="urn:adsk.eagle:library:6897166" package="HOLES_3,2-PAD" package3d_urn="urn:adsk.eagle:package:5224590/2" value="HOLES_MOUNT-PAD-ROUND3.2" x="59.76" y="5.18" smashed="yes"/>
 <element name="H4" library="PiezoFFC" library_urn="urn:adsk.eagle:library:6897166" package="HOLES_3,2-PAD" package3d_urn="urn:adsk.eagle:package:5224590/2" value="HOLES_MOUNT-PAD-ROUND3.2" x="59.76" y="58.82" smashed="yes"/>
-<element name="R5" library="PiezoFFC" library_urn="urn:adsk.eagle:library:6897166" package="R0805" package3d_urn="urn:adsk.eagle:package:8443791/3" value="2K" x="27.1" y="18.65" smashed="yes" rot="R270">
+<element name="R5" library="PiezoFFC" library_urn="urn:adsk.eagle:library:6897166" package="R0805" package3d_urn="urn:adsk.eagle:package:8443791/3" value="0R" x="27.1" y="18.65" smashed="yes" rot="R270">
 <attribute name="MPN" value="RC0805JR-072KL" x="34.1" y="24.65" size="1.778" layer="27" rot="R270" display="off"/>
 <attribute name="NAME" x="29.005" y="17.634" size="0.889" layer="25" font="vector" ratio="11" rot="R180"/>
