File: Eagle_Files/FFC_Direct_Breakout/Pyr0-Piezo_Direct-Extruder-FFC-Breakout_2.0.1.sch (EAGLE design)
At the start: 33 parts, among them J1 FFC_MOLEX_0.5MM, Q2 2N2907, U1 LM317DCY, U2 L78L05ACU

Commit message: Added ESD protection diodes to motor connections
Parts:
- added D1, D10, D11, D12, D13, D14, D15, D16, D2, D3, D4, D5, D6, D7, D8, D9: DIODE_SCHOTTKY_SINGLE, PiezoFFC:DIODE_SCHOTTKY_SINGLE
- Q2: value 2N2907 -> (none); device PiezoFFC:2N2907 -> PiezoFFC:MMBT2907ALT1-PNP-SOT23-BEC
- R5: value 0R -> 2K
- R6: value 1R -> 2K
- R7: value 10R -> 2K
Connections:
- net AGND: now also D1.A, D11.A, D13.A, D15.A, D3.A, D5.A, D7.A, D9.A
- net E0_1A: now also D13.C, D14.A
- net E0_1B: now also D15.C, D16.A
- net E0_2A: now also D11.C, D12.A
- net E0_2B: now also D10.A, D9.C
- net VCC: now also D10.C, D12.C, D14.C, D16.C, D2.C, D4.C, D6.C, D8.C
- net X_1A: now also D5.C, D6.A
- net X_1B: now also D7.C, D8.A
- net X_2A: now also D3.C, D4.A
- net X_2B: now also D1.C, D2.A
Other:
- moved on the sheet: E0-1, E0-2, E0-3, E0-4, X_MOT-1, X_MOT-2, X_MOT-3, X_MOT-4

Commit message: fixed incorrect resistor values on FFC Direct vreg #bugfix
Parts:
- R5: value 2K -> 0R
- R6: value 2K -> 1R
- R7: value 2K -> 10R
Changed lines of the file:
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@@
 <?xml version="1.0" encoding="utf-8"?>
 <!DOCTYPE eagle SYSTEM "eagle.dtd">
-<eagle version="9.3.2">
+<eagle version="9.4.2">
 <drawing>
 <settings>
@@
 <part name="AGND4" library="supply1" library_urn="urn:adsk.eagle:library:371" deviceset="AGND" device=""/>
 <part name="Q2" library="PiezoFFC" library_urn="urn:adsk.eagle:library:6897166" deviceset="*-PNP-" device="SOT23-BEC" package3d_urn="urn:adsk.eagle:package:28748/2" technology="MMBT2907ALT1"/>
-<part name="R6" library="PiezoFFC" library_urn="urn:adsk.eagle:library:6897166" deviceset="SMD-RES-2K-5%-1/8W(0805)" device="" package3d_urn="urn:adsk.eagle:package:8443791/3" value="2K"/>
-<part name="R7" library="PiezoFFC" library_urn="urn:adsk.eagle:library:6897166" deviceset="SMD-RES-2K-5%-1/8W(0805)" device="" package3d_urn="urn:adsk.eagle:package:8443791/3" value="2K"/>
+<part name="R6" library="PiezoFFC" library_urn="urn:adsk.eagle:library:6897166" deviceset="SMD-RES-2K-5%-1/8W(0805)" device="" package3d_urn="urn:adsk.eagle:package:8443791/3" value="1R"/>
+<part name="R7" library="PiezoFFC" library_urn="urn:adsk.eagle:library:6897166" deviceset="SMD-RES-2K-5%-1/8W(0805)" device="" package3d_urn="urn:adsk.eagle:package:8443791/3" value="10R"/>
 <part name="C2" library="PiezoFFC" library_urn="urn:adsk.eagle:library:6897166" deviceset="DIP-ALUMINUM-100UF-16V(D5-H7MM)" device="LEFT" package3d_urn="urn:adsk.eagle:package:8885168/4" value="100uf"/>
 <part name="C3" library="PiezoFFC" library_urn="urn:adsk.eagle:library:6897166" deviceset="DIP-ALUMINUM-100UF-16V(D5-H7MM)" device="RIGHT" package3d_urn="urn:adsk.eagle:package:8885515/3" value="100uf"/>
@@
 <part name="H3" library="PiezoFFC" library_urn="urn:adsk.eagle:library:6897166" deviceset="HOLES_MOUNT-PAD-ROUND" device="3.2" package3d_urn="urn:adsk.eagle:package:5224590/2"/>
 <part name="H4" library="PiezoFFC" library_urn="urn:adsk.eagle:library:6897166" deviceset="HOLES_MOUNT-PAD-ROUND" device="3.2" package3d_urn="urn:adsk.eagle:package:5224590/2"/>
-<part name="R5" library="PiezoFFC" library_urn="urn:adsk.eagle:library:6897166" deviceset="SMD-RES-2K-5%-1/8W(0805)" device="" package3d_urn="urn:adsk.eagle:package:8443791/3" value="2K"/>
+<part name="R5" library="PiezoFFC" library_urn="urn:adsk.eagle:library:6897166" deviceset="SMD-RES-2K-5%-1/8W(0805)" device="" package3d_urn="urn:adsk.eagle:package:8443791/3" value="0R"/>
 <part name="J1" library="PiezoFFC" library_urn="urn:adsk.eagle:library:6897166" deviceset="FFC_MOLEX_0.5MM" device="" package3d_urn="urn:adsk.eagle:package:8786753/3"/>
 <part name="AGND6" library="supply1" library_urn="urn:adsk.eagle:library:371" deviceset="AGND" device=""/>
