File: Eagle_Files/Standalone/Pyr0-Piezo-Standalone_3.0.0.sch (EAGLE design)
At the start: 68 parts, among them J1 CON-MOLEX-6P-1.25MM048, J3 10118192-0001LF, U2 L78L05ACU, U3 LM2902QT, U4 ATSAMD21E*-MU

Commit message: Updated description. Sync files
Connections:
- net RST: now also U4.!RESET
- net SCL: now also U4.PA23
- net SDA: now also U4.PA22
- net Z_TRG: now also U4.PA15
Other:
- moved on the sheet: INT
