File: Eagle_Files/Standalone/Pyr0-Piezo-Standalone_2.1.0.brd (EAGLE design)
At the start: 43 x 15.4 mm, 66 parts, among them J1 CON-MOLEX-6P-1.25MM048, U2 L78L05ACU, U3 LM2902QT, U4 ATMEGA48/88/168/328PB

Commit message: Beta production board sync
Parts:
- D1: value ZENER_DIODE_PLZ5V1C -> DIODE_ZENER_PLZ5V1C
- moved C8 4.56 mm to (33.8, 5.49), turned to 135 degrees
- moved C5 4.29 mm to (34.4, 3.75), turned to 45 degrees
- moved C6 4.21 mm to (38.4, 7.81), turned to 225 degrees
- moved C9 4.05 mm to (36.4, 8.16), turned to 315 degrees
- moved R19 3.86 mm to (35.0, 4.38)
- moved R20 3.82 mm to (37.8, 7.21)
- moved R17 2.76 mm to (33.2, 6.67), turned to 45 degrees
- moved R18 2.10 mm to (35.1, 8.57), turned to 225 degrees
- moved TP2 1.37 mm to (35.5, 7.75)
- moved TP1 1.23 mm to (34.5, 6.92)
- moved R1 0.05 mm to (33.0, 9.35), turned to 270 degrees
Connections:
- net GND: now also PZ1.2; no longer PZ1.1
- net PT_IN+: now also PT100.1; no longer PT100.2
- net PT_IN-: now also PT100.2; no longer PT100.1
- net PZ+: now also PZ1.1; no longer PZ1.2
Routing:
- net +5V: track 67.4 -> 63.0 mm, vias 9 -> 8
- net PT_AMP+: track 12.9 -> 9.04 mm
- net PT_AMP-: track 8.75 -> 11.7 mm
- net PT_IN+: track 6.01 -> 7.78 mm
- net PZ+: track 14.3 -> 15.9 mm, vias 0 -> 1
- net GND: track 7.63 -> 6.13 mm
- net PT_IN-: track 6.10 -> 7.45 mm
