File: Eagle_Files/Standalone/Pyr0-Piezo-Standalone_2.1.0.sch (EAGLE design)
At the start: 64 parts, among them J1 CON-MOLEX-6P-1.25MM048, U2 L78L05ACU, U3 LM2902QT, U4 ATMEGA48/88/168/328PB

Commit message: Beta production board sync
Parts:
- D1: value ZENER_DIODE_PLZ5V1C -> DIODE_ZENER_PLZ5V1C; device PiezoFFC:ZENER_DIODE_PLZ5V1C -> PiezoFFC:DIODE_ZENER_PLZ5V1C
Connections:
- net GND: now also PZ1-2.S; no longer PZ1-1.S
- net PT_IN+: now also PT100-1.S; no longer PT100-2.S
- net PT_IN-: now also PT100-2.S; no longer PT100-1.S
- net PZ+: now also PZ1-1.S; no longer PZ1-2.S
Other:
- moved on the sheet: PT100-1, PT100-2, PZ1-1, PZ1-2
Changed lines of the file:
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@@
 <?xml version="1.0" encoding="utf-8"?>
 <!DOCTYPE eagle SYSTEM "eagle.dtd">
-<eagle version="9.3.0">
+<eagle version="9.3.2">
 <drawing>
 <settings>
-<setting alwaysvectorfont="no"/>
+<setting alwaysvectorfont="yes"/>
 <setting verticaltext="up"/>
 </settings>
@@
 <part name="R15" library="PiezoFFC" library_urn="urn:adsk.eagle:library:6897166" deviceset="SMD-RES-0R-5%-1/16W(0402)" device="" package3d_urn="urn:adsk.eagle:package:7115182/2" value="100R"/>
 <part name="⏚" library="testpad" library_urn="urn:adsk.eagle:library:385" deviceset="TP" device="TP13SQ" package3d_urn="urn:adsk.eagle:package:27974/1" value="TPTP13SQ"/>
-<part name="D1" library="PiezoFFC" library_urn="urn:adsk.eagle:library:6897166" deviceset="ZENER_DIODE_PLZ5V1C" device="" package3d_urn="urn:adsk.eagle:package:8452796/2"/>
+<part name="D1" library="PiezoFFC" library_urn="urn:adsk.eagle:library:6897166" deviceset="DIODE_ZENER_PLZ5V1C" device="" package3d_urn="urn:adsk.eagle:package:8452796/2"/>
 <part name="F1" library="PiezoFFC" library_urn="urn:adsk.eagle:library:6897166" deviceset="SMD-RES-0R-5%-1/16W(0402)" device="" package3d_urn="urn:adsk.eagle:package:7115182/2" value="500mA"/>
 <part name="SJ1" library="PiezoFFC" library_urn="urn:adsk.eagle:library:6897166" deviceset="SJ" device="M" package3d_urn="urn:adsk.eagle:package:8763769/3"/>
@@
 </plain>
 <instances>
-<instance part="PZ1" gate="-1" x="330.2" y="93.98" smashed="yes">
-<attribute name="NAME" x="331.47" y="93.472" size="1.524" layer="95" rot="R180"/>
-</instance>
-<instance part="PZ1" gate="-2" x="330.2" y="97.79" smashed="yes">
+<instance part="PZ1" gate="-1" x="330.2" y="97.79" smashed="yes">
 <attribute name="NAME" x="331.47" y="97.282" size="1.524" layer="95" rot="R180"/>
+</instance>
+<instance part="PZ1" gate="-2" x="330.2" y="95.25" smashed="yes">
+<attribute name="NAME" x="331.47" y="94.742" size="1.524" layer="95" rot="R180"/>
 </instance>
 <instance part="U2" gate="G$1" x="71.12" y="130.81" smashed="yes">
@@
 </instance>
 <instance part="U3" gate="P" x="340.36" y="199.39" smashed="yes"/>
-<instance part="PT100" gate="-1" x="203.2" y="43.18" smashed="yes" rot="R180">
-<attribute name="NAME" x="198.628" y="43.18" size="1.524" layer="95" rot="R270"/>
-</instance>
-<instance part="PT100" gate="-2" x="203.2" y="45.72" smashed="yes" rot="R180">
-<attribute name="NAME" x="200.152" y="45.72" size="1.524" layer="95" rot="R90"/>
+<instance part="PT100" gate="-1" x="203.2" y="45.72" smashed="yes" rot="R180">
+<attribute name="NAME" x="202.692" y="48.26" size="1.524" layer="95" rot="R90"/>
+</instance>
+<instance part="PT100" gate="-2" x="203.2" y="43.18" smashed="yes" rot="R180">
+<attribute name="NAME" x="201.168" y="40.64" size="1.524" layer="95" rot="R270"/>
 </instance>
 <instance part="C5" gate="G$1" x="212.09" y="52.07" smashed="yes" rot="R90">
@@
 </segment>
 <segment>
-<pinref part="PZ1" gate="-1" pin="S"/>
-<wire x1="327.66" y1="93.98" x2="323.85" y2="93.98" width="0.1524" layer="91"/>
 <pinref part="SUPPLY13" gate="GND" pin="GND"/>
-<wire x1="323.85" y1="93.98" x2="323.85" y2="88.9" width="0.1524" layer="91"/>
+<wire x1="323.85" y1="95.25" x2="323.85" y2="88.9" width="0.1524" layer="91"/>
+<pinref part="PZ1" gate="-2" pin="S"/>
+<wire x1="327.66" y1="95.25" x2="323.85" y2="95.25" width="0.1524" layer="91"/>
 </segment>
 </net>
@@
 </segment>
 <segment>
-<pinref part="PZ1" gate="-2" pin="S"/>
 <wire x1="323.85" y1="97.79" x2="325.12" y2="97.79" width="0.1524" layer="91"/>
 <label x="323.85" y="97.79" size="1.778" layer="95" rot="R180" xref="yes"/>
 <pinref part="PZ+" gate="G$1" pin="TP"/>
-<wire x1="325.12" y1="97.79" x2="327.66" y2="97.79" width="0.1524" layer="91"/>
 <wire x1="325.12" y1="100.33" x2="325.12" y2="97.79" width="0.1524" layer="91"/>
+<pinref part="PZ1" gate="-1" pin="S"/>
+<wire x1="327.66" y1="97.79" x2="325.12" y2="97.79" width="0.1524" layer="91"/>
 <junction x="325.12" y="97.79"/>
 </segment>
@@
 <net name="PT_IN+" class="0">
 <segment>
-<pinref part="PT100" gate="-2" pin="S"/>
-<wire x1="205.74" y1="45.72" x2="207.01" y2="45.72" width="0.1524" layer="91"/>
 <pinref part="TP1" gate="G$1" pin="TP"/>
 <wire x1="207.01" y1="45.72" x2="207.01" y2="46.99" width="0.1524" layer="91"/>
 <pinref part="R17" gate="G$1" pin="1"/>
-<wire x1="207.01" y1="45.72" x2="212.09" y2="45.72" width="0.1524" layer="91"/>
+<wire x1="207.01" y1="45.72" x2="208.28" y2="45.72" width="0.1524" layer="91"/>
+<wire x1="208.28" y1="45.72" x2="212.09" y2="45.72" width="0.1524" layer="91"/>
 <wire x1="212.09" y1="45.72" x2="218.44" y2="45.72" width="0.1524" layer="91"/>
 <wire x1="218.44" y1="45.72" x2="218.44" y2="48.26" width="0.1524" layer="91"/>
-<junction x="207.01" y="45.72"/>
 <pinref part="C5" gate="G$1" pin="1"/>
 <wire x1="212.09" y1="48.26" x2="212.09" y2="45.72" width="0.1524" layer="91"/>
@@
 <wire x1="218.44" y1="49.53" x2="218.44" y2="48.26" width="0.1524" layer="91"/>
 <junction x="218.44" y="48.26"/>
+<pinref part="PT100" gate="-1" pin="S"/>
+<wire x1="207.01" y1="45.72" x2="205.74" y2="45.72" width="0.1524" layer="91"/>
 </segment>
 </net>
 <net name="PT_IN-" class="0">
 <segment>
-<pinref part="PT100" gate="-1" pin="S"/>
-<wire x1="205.74" y1="43.18" x2="207.01" y2="43.18" width="0.1524" layer="91"/>
 <pinref part="TP2" gate="G$1" pin="TP"/>
 <wire x1="207.01" y1="43.18" x2="207.01" y2="41.91" width="0.1524" layer="91"/>
 <pinref part="R18" gate="G$1" pin="1"/>
-<wire x1="207.01" y1="43.18" x2="212.09" y2="43.18" width="0.1524" layer="91"/>
+<wire x1="207.01" y1="43.18" x2="208.28" y2="43.18" width="0.1524" layer="91"/>
+<wire x1="208.28" y1="43.18" x2="212.09" y2="43.18" width="0.1524" layer="91"/>
 <wire x1="212.09" y1="43.18" x2="218.44" y2="43.18" width="0.1524" layer="91"/>
 <wire x1="218.44" y1="43.18" x2="218.44" y2="40.64" width="0.1524" layer="91"/>
-<junction x="207.01" y="43.18"/>
 <pinref part="C6" gate="G$1" pin="2"/>
 <wire x1="212.09" y1="40.64" x2="212.09" y2="43.18" width="0.1524" layer="91"/>
@@
 <wire x1="218.44" y1="39.37" x2="218.44" y2="40.64" width="0.1524" layer="91"/>
 <junction x="218.44" y="40.64"/>
-</segment>
-</net>
+<pinref part="PT100" gate="-2" pin="S"/>
+<wire x1="205.74" y1="43.18" x2="207.01" y2="43.18" width="0.1524" layer="91"/>
+</segment>
+</net>
