File: Eagle_Files/Standalone/Pyr0-Piezo-Standalone1.0.2.brd (EAGLE design)
At the start: 42.9 x 15.4 mm, 52 parts, among them J1 CON-MOLEX-4P-1.25MM048, U1 ATMEGA48PA-MMHR28M1-L, U2 L78L05ACU, U3 LM2902QT

Commit message: Updated eagle files for 1.0.2 for Eagle 9.0.2
Parts:
- J1: value CON-MOLEX-4P-1.25MM048 -> CON-MOLEX-3P-1.25MM048; device PiezoFFC:53048-04 -> PiezoFFC:53048-03
Routing:
- net VCC_REG: track 6.32 -> 5.58 mm
- net Z_MIN_TRIG: track 19.1 -> 18.5 mm
Changed lines of the file:
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@@
 <?xml version="1.0" encoding="utf-8"?>
 <!DOCTYPE eagle SYSTEM "eagle.dtd">
-<eagle version="9.3.0">
+<eagle version="9.3.2">
 <drawing>
 <settings>
@@
 <attribute name="NAME" x="34.49166875" y="8.0337375" size="0.8128" layer="25" font="vector" rot="R315"/>
 </element>
-<element name="J1" library="PiezoFFC" library_urn="urn:adsk.eagle:library:6897166" package="53048-04" package3d_urn="urn:adsk.eagle:package:8078564/1" value="CON-MOLEX-4P-1.25MM048" x="7.429" y="9.764" smashed="yes" rot="R45">
-<attribute name="MF" value="MOLEX" x="7.429" y="9.764" size="1.778" layer="27" rot="R45" display="off"/>
-<attribute name="MPN" value="53048-0410" x="7.429" y="9.764" size="1.778" layer="27" rot="R45" display="off"/>
+<element name="J1" library="PiezoFFC" library_urn="urn:adsk.eagle:library:6897166" package="53048-03" package3d_urn="urn:adsk.eagle:package:7192338/2" value="CON-MOLEX-3P-1.25MM048" x="7.429" y="9.764" smashed="yes" rot="R45">
+<attribute name="MF" value="WALDOM/MOLEX" x="7.429" y="9.764" size="1.778" layer="27" rot="R45" display="off"/>
+<attribute name="MPN" value="53048-0310" x="7.429" y="9.764" size="1.778" layer="27" rot="R45" display="off"/>
 <attribute name="NAME" x="6.911978125" y="9.02291875" size="1.27" layer="25" rot="R45"/>
-<attribute name="OC_FARNELL" value="1462887" x="7.429" y="9.764" size="1.778" layer="27" rot="R45" display="off"/>
-<attribute name="OC_NEWARK" value="57H4721" x="7.429" y="9.764" size="1.778" layer="27" rot="R45" display="off"/>
+<attribute name="OC_FARNELL" value="9732918" x="7.429" y="9.764" size="1.778" layer="27" rot="R45" display="off"/>
+<attribute name="OC_NEWARK" value="38C9908" x="7.429" y="9.764" size="1.778" layer="27" rot="R45" display="off"/>
 </element>
 <element name="C3" library="PiezoFFC" library_urn="urn:adsk.eagle:library:6897166" package="CAPC1005X50" package3d_urn="urn:adsk.eagle:package:5248669/4" value="0.1uF" x="24.717" y="2.127" smashed="yes" rot="R180">
@@
 <wire x1="16.7996" y1="1.02424375" x2="9.64375625" y2="1.02424375" width="0.1524" layer="1"/>
 <wire x1="9.64375625" y1="1.02424375" x2="9.144" y2="1.524" width="0.1524" layer="1"/>
-<wire x1="7.870940625" y1="8.438171875" x2="7.429" y2="7.996234375" width="0.1524" layer="1"/>
+<wire x1="7.429" y1="7.99623125" x2="7.429" y2="7.996234375" width="0.1524" layer="1"/>
 <wire x1="17.425290625" y1="1.602" x2="18.112" y2="1.602" width="0.1524" layer="1"/>
 <wire x1="18.112" y1="1.602" x2="18.74879375" y2="2.23879375" width="0.1524" layer="1"/>
@@
 <contactref element="J1" pad="2"/>
 <wire x1="8.31288125" y1="8.88011875" x2="8.31288125" y2="8.81411875" width="0.4064" layer="1"/>
-<wire x1="8.754825" y1="9.32205625" x2="8.31288125" y2="8.88011875" width="0.1524" layer="1"/>
+<wire x1="8.31288125" y1="8.880115625" x2="8.31288125" y2="8.88011875" width="0.1524" layer="1"/>
 <wire x1="9.491503125" y1="6.10979375" x2="9.491503125" y2="7.70149375" width="0.4064" layer="16"/>
-<wire x1="9.491503125" y1="7.70149375" x2="8.754825" y2="9.32205625" width="0.4064" layer="16"/>
+<wire x1="9.491503125" y1="7.70149375" x2="8.31288125" y2="8.880115625" width="0.4064" layer="16"/>
 <contactref element="F1" pad="1"/>
 <wire x1="10.2055" y1="8.001" x2="9.192" y2="8.001" width="0.4064" layer="1"/>
