File: Eagle_Files/Standalone/Pyr0-Piezo-Standalone1.0.2.sch (EAGLE design)
At the start: 50 parts, among them J1 CON-MOLEX-4P-1.25MM048, U1 ATMEGA48PA-MMHR28M1-L, U2 L78L05ACU, U3 LM2902QT

Commit message: Updated eagle files for 1.0.2 for Eagle 9.0.2
Parts:
- J1: value CON-MOLEX-4P-1.25MM048 -> CON-MOLEX-3P-1.25MM048; device PiezoFFC:CON-MOLEX-4P-1.25MM048 -> PiezoFFC:CON-MOLEX-3P-1.25MM048
Changed lines of the file:
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@@
 <?xml version="1.0" encoding="utf-8"?>
 <!DOCTYPE eagle SYSTEM "eagle.dtd">
-<eagle version="9.3.0">
+<eagle version="9.3.2">
 <drawing>
 <settings>
-<setting alwaysvectorfont="no"/>
+<setting alwaysvectorfont="yes"/>
 <setting verticaltext="up"/>
 </settings>
@@
 <part name="D8" library="PiezoFFC" library_urn="urn:adsk.eagle:library:6897166" deviceset="BAV199" device="" package3d_urn="urn:adsk.eagle:package:6899267/1"/>
 <part name="SUPPLY10" library="supply2" library_urn="urn:adsk.eagle:library:372" deviceset="GND" device=""/>
-<part name="J1" library="PiezoFFC" library_urn="urn:adsk.eagle:library:6897166" deviceset="CON-MOLEX-4P-1.25MM" device="048" package3d_urn="urn:adsk.eagle:package:8078564/1"/>
+<part name="J1" library="PiezoFFC" library_urn="urn:adsk.eagle:library:6897166" deviceset="CON-MOLEX-3P-1.25MM" device="048" package3d_urn="urn:adsk.eagle:package:7192338/2"/>
 <part name="P+1" library="PiezoFFC" library_urn="urn:adsk.eagle:library:6897166" deviceset="+5V" device=""/>
 <part name="P+3" library="PiezoFFC" library_urn="urn:adsk.eagle:library:6897166" deviceset="+5V" device=""/>
