File: Eagle_Files/Standalone/Pyr0-Piezo-Standalone_2.0.1.brd (EAGLE design)
At the start: 43 x 15.4 mm, 71 parts, among them J1 CON-MOLEX-4P-1.25MM048, U1 ATMEGA48/88/168/328PA28M1-L, U2 L78L05ACU, U3 LM2902QT

Commit message: rotated fuse for easier soldering
Parts:
- moved F1 0.20 mm to (10.5, 8.16), turned to 315 degrees
Routing:
- net VCC_FUSE: track 2.84 -> 3.36 mm
Changed lines of the file:
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@@
 <layer number="43" name="vRestrict" color="2" fill="10" visible="no" active="yes"/>
 <layer number="44" name="Drills" color="7" fill="1" visible="no" active="yes"/>
-<layer number="45" name="Holes" color="7" fill="1" visible="no" active="yes"/>
+<layer number="45" name="Holes" color="7" fill="1" visible="yes" active="yes"/>
 <layer number="46" name="Milling" color="3" fill="1" visible="no" active="yes"/>
 <layer number="47" name="Measures" color="7" fill="1" visible="no" active="yes"/>
@@
 <element name="U$2" library="PiezoFFC" library_urn="urn:adsk.eagle:library:6897166" package="LOGO-PYR0BALL-SS-6MM" value="" x="13.589" y="9.5885" smashed="yes" rot="R45"/>
 <element name="D1" library="PiezoFFC" library_urn="urn:adsk.eagle:library:6897166" package="DO-219AC" package3d_urn="urn:adsk.eagle:package:8452796/2" value="ZENER_DIODE_PLZ5V1C" x="14.097" y="8.128" smashed="yes" rot="R270"/>
-<element name="F1" library="PiezoFFC" library_urn="urn:adsk.eagle:library:6897166" package="R0402" package3d_urn="urn:adsk.eagle:package:7115182/2" value="500mA" x="10.668" y="8.001" smashed="yes" rot="R90">
-<attribute name="MPN" value="RC0402JR-070RL" x="4.953" y="3.556" size="1.778" layer="27" rot="R90" display="off"/>
-<attribute name="NAME" x="11.811" y="7.5565" size="0.8128" layer="25" font="vector" ratio="11"/>
+<element name="F1" library="PiezoFFC" library_urn="urn:adsk.eagle:library:6897166" package="R0402" package3d_urn="urn:adsk.eagle:package:7115182/2" value="500mA" x="10.541" y="8.15975" smashed="yes" rot="R315">
+<attribute name="MPN" value="RC0402JR-070RL" x="11.439028125" y="15.34395" size="1.778" layer="27" rot="R315" display="off"/>
+<attribute name="NAME" x="9.418471875" y="7.665834375" size="0.8128" layer="25" font="vector" ratio="11" rot="R225"/>
 </element>
 <element name="SJ1" library="PiezoFFC" library_urn="urn:adsk.eagle:library:6897166" package="SJM" package3d_urn="urn:adsk.eagle:package:8763769/3" value="" x="11.811" y="7.493" smashed="yes" rot="MR225">
@@
 <contactref element="C2" pad="2"/>
 <contactref element="J1" pad="2"/>
-<wire x1="9.04313125" y1="9.03886875" x2="9.04313125" y2="9.03375" width="0.4064" layer="1"/>
-<wire x1="8.754825" y1="9.32205625" x2="9.04313125" y2="9.03375" width="0.4064" layer="1"/>
 <contactref element="F1" pad="1"/>
-<wire x1="10.2055" y1="8.001" x2="10.081" y2="8.001" width="0.4064" layer="1"/>
-<wire x1="10.081" y1="8.001" x2="9.04313125" y2="9.03886875" width="0.4064" layer="1"/>
 <wire x1="9.491503125" y1="8.585378125" x2="8.754825" y2="9.32205625" width="0.4064" layer="16"/>
 <wire x1="9.491503125" y1="6.10979375" x2="9.491503125" y2="8.585378125" width="0.4064" layer="16"/>
+<wire x1="10.36486875" y1="8.98995" x2="9.08693125" y2="8.98995" width="0.4064" layer="1"/>
+<wire x1="8.754825" y1="9.32205625" x2="9.08693125" y2="8.98995" width="0.4064" layer="1"/>
+<wire x1="10.868034375" y1="8.486784375" x2="10.36486875" y2="8.98995" width="0.4064" layer="1"/>
 </signal>
 <signal name="TTL_RXD">
@@
 <contactref element="F1" pad="2"/>
 <contactref element="U2" pad="3"/>
-<wire x1="9.565796875" y1="6.436296875" x2="9.565796875" y2="6.1985" width="0.4064" layer="1"/>
-<wire x1="11.1305" y1="8.001" x2="11.1305" y2="7.99633125" width="0.4064" layer="1"/>
-<wire x1="11.1305" y1="7.99633125" x2="10.52956875" y2="7.3954" width="0.4064" layer="1"/>
-<wire x1="10.52956875" y1="7.3954" x2="10.5249" y2="7.3954" width="0.4064" layer="1"/>
-<wire x1="10.5249" y1="7.3954" x2="9.565796875" y2="6.436296875" width="0.4064" layer="1"/>
 <contactref element="SJ1" pad="1"/>
 <wire x1="11.451790625" y1="7.852209375" x2="11.279290625" y2="7.852209375" width="0.4064" layer="16"/>
-<wire x1="11.279290625" y1="7.852209375" x2="11.1305" y2="8.001" width="0.4064" layer="16"/>
-<via x="11.1305" y="8.001" extent="1-16" drill="0.35"/>
+<via x="11.4522125" y="7.8644625" extent="1-16" drill="0.35"/>
+<wire x1="10.2139625" y1="7.8327125" x2="10.080625" y2="7.699375" width="0.4064" layer="1"/>
+<wire x1="10.080625" y1="7.699375" x2="9.565796875" y2="7.184546875" width="0.4064" layer="1"/>
+<wire x1="9.565796875" y1="7.184546875" x2="9.565796875" y2="6.1985" width="0.4064" layer="1"/>
+<wire x1="10.2457125" y1="7.8644625" x2="10.2139625" y2="7.8327125" width="0.4064" layer="1"/>
+<wire x1="11.4522125" y1="7.8644625" x2="11.10215625" y2="7.8644625" width="0.4064" layer="1"/>
+<wire x1="11.10215625" y1="7.8644625" x2="11.06710625" y2="7.8294125" width="0.4064" layer="1"/>
+<wire x1="11.06710625" y1="7.8294125" x2="10.6689625" y2="7.8294125" width="0.4064" layer="1"/>
+<wire x1="10.6689625" y1="7.8294125" x2="10.6339125" y2="7.8644625" width="0.4064" layer="1"/>
+<wire x1="10.6339125" y1="7.8644625" x2="10.2457125" y2="7.8644625" width="0.4064" layer="1"/>
+<wire x1="11.4522125" y1="7.8644625" x2="11.451790625" y2="7.852209375" width="0" layer="19" extent="16-16"/>
 </signal>
 <signal name="AMP_VCC">

Commit message: sync all boards for Rev.2.0.1 before gerberization
- added test pads for debugging amp circuit
Parts:
- moved C2 0.13 mm to (9.36, 5.41)
- moved C1 0.10 mm to (11.0, 5.42)
Changed lines of the file:
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@@
 <?xml version="1.0" encoding="utf-8"?>
 <!DOCTYPE eagle SYSTEM "eagle.dtd">
-<eagle version="9.3.1">
+<eagle version="9.3.2">
 <drawing>
 <settings>
-<setting alwaysvectorfont="yes"/>
+<setting alwaysvectorfont="no"/>
 <setting verticaltext="up"/>
 </settings>
@@
 <attribute name="VALUE" x="26.819478125" y="14.058915625" size="0.0254" layer="28" rot="MR270"/>
 </element>
-<element name="C1" library="PiezoFFC" library_urn="urn:adsk.eagle:library:6897166" package="CAPC1609X80" package3d_urn="urn:adsk.eagle:package:5248663/3" value="1uF" x="10.867753125" y="5.417353125" smashed="yes" rot="MR90">
-<attribute name="NAME" x="10.862415625" y="4.063046875" size="0.6096" layer="26" font="vector" rot="MR180" align="bottom-center"/>
-<attribute name="VALUE" x="10.653146875" y="5.441146875" size="0.6096" layer="28" font="vector" rot="MR270" align="top-center"/>
-</element>
-<element name="C2" library="PiezoFFC" library_urn="urn:adsk.eagle:library:6897166" package="CAPC1609X80" package3d_urn="urn:adsk.eagle:package:5248663/3" value="1uF" x="9.491503125" y="5.40979375" smashed="yes" rot="MR90">
-<attribute name="NAME" x="9.51453125" y="7.20939375" size="0.6096" layer="26" font="vector" ratio="11" rot="MR180" align="bottom-center"/>
-<attribute name="VALUE" x="8.90610625" y="5.471821875" size="0.6096" layer="28" font="vector" rot="MR90" align="top-center"/>
+<element name="C1" library="PiezoFFC" library_urn="urn:adsk.eagle:library:6897166" package="CAPC1609X80" package3d_urn="urn:adsk.eagle:package:5248663/3" value="1uF" x="10.963003125" y="5.417353125" smashed="yes" rot="MR90">
+<attribute name="NAME" x="10.957665625" y="4.063046875" size="0.6096" layer="26" font="vector" ratio="11" rot="MR180" align="bottom-center"/>
+<attribute name="VALUE" x="10.748396875" y="5.441146875" size="0.6096" layer="28" font="vector" rot="MR270" align="top-center"/>
+</element>
+<element name="C2" library="PiezoFFC" library_urn="urn:adsk.eagle:library:6897166" package="CAPC1609X80" package3d_urn="urn:adsk.eagle:package:5248663/3" value="1uF" x="9.364503125" y="5.40979375" smashed="yes" rot="MR90">
+<attribute name="NAME" x="9.38753125" y="7.20939375" size="0.6096" layer="26" font="vector" ratio="11" rot="MR180" align="bottom-center"/>
+<attribute name="VALUE" x="8.77910625" y="5.471821875" size="0.6096" layer="28" font="vector" rot="MR90" align="top-center"/>
 </element>
 <element name="INT" library="testpad" library_urn="urn:adsk.eagle:library:385" package="TP06R" package3d_urn="urn:adsk.eagle:package:27954/1" value="TPTP06R" x="17.003790625" y="8.150503125" smashed="yes">
@@
 <contactref element="J1" pad="2"/>
 <contactref element="F1" pad="1"/>
-<wire x1="9.491503125" y1="8.585378125" x2="8.754825" y2="9.32205625" width="0.4064" layer="16"/>
-<wire x1="9.491503125" y1="6.10979375" x2="9.491503125" y2="8.585378125" width="0.4064" layer="16"/>
+<wire x1="9.364503125" y1="8.712378125" x2="8.754825" y2="9.32205625" width="0.4064" layer="16"/>
+<wire x1="9.364503125" y1="6.10979375" x2="9.364503125" y2="8.712378125" width="0.4064" layer="16"/>
 <wire x1="10.36486875" y1="8.98995" x2="9.08693125" y2="8.98995" width="0.4064" layer="1"/>
 <wire x1="8.754825" y1="9.32205625" x2="9.08693125" y2="8.98995" width="0.4064" layer="1"/>
@@
 <via x="24.494634375" y="13.2122" extent="1-16" drill="0.35"/>
 <wire x1="12.66825" y1="5.9055" x2="12.2708" y2="5.9055" width="0.254" layer="1"/>
-<wire x1="14.596421875" y1="10.232734375" x2="13.52543125" y2="10.232734375" width="0.1524" layer="16"/>
-<wire x1="13.52543125" y1="10.232734375" x2="13.394965625" y2="10.3632" width="0.1524" layer="16"/>
+<wire x1="15.136171875" y1="10.042234375" x2="13.71593125" y2="10.042234375" width="0.1524" layer="16"/>
+<wire x1="13.71593125" y1="10.042234375" x2="13.394965625" y2="10.3632" width="0.1524" layer="16"/>
 <via x="17.5810375" y="13.227690625" extent="1-16" drill="0.35"/>
 <wire x1="24.4377125" y1="13.155278125" x2="24.494634375" y2="13.2122" width="0.1524" layer="1"/>
-<wire x1="17.5810375" y1="13.227690625" x2="17.5810375" y2="13.21735" width="0.1524" layer="16"/>
-<wire x1="17.5810375" y1="13.21735" x2="14.596421875" y2="10.232734375" width="0.1524" layer="16"/>
+<wire x1="17.5810375" y1="13.227690625" x2="17.5810375" y2="12.4871" width="0.1524" layer="16"/>
+<wire x1="17.5810375" y1="12.4871" x2="15.136171875" y2="10.042234375" width="0.1524" layer="16"/>
 <wire x1="17.5810375" y1="13.227690625" x2="17.92146875" y2="12.887259375" width="0.1524" layer="1"/>
 <wire x1="17.92146875" y1="12.887259375" x2="24.16969375" y2="12.887259375" width="0.1524" layer="1"/>
 <wire x1="24.16969375" y1="12.887259375" x2="24.494634375" y2="13.2122" width="0.1524" layer="1"/>
 <wire x1="13.394965625" y1="10.3632" x2="12.231775" y2="10.3632" width="0.1524" layer="16"/>
-<wire x1="12.231775" y1="10.3632" x2="10.409915625" y2="8.541340625" width="0.1524" layer="16"/>
-<wire x1="10.409915625" y1="8.541340625" x2="10.409915625" y2="6.303853125" width="0.1524" layer="16"/>
 <via x="12.309796875" y="6.1985" extent="1-16" drill="0.35"/>
 <contactref element="D8" pad="2"/>
@@
 <via x="21.424075" y="4.2375" extent="1-16" drill="0.35"/>
 <wire x1="16.3270125" y1="5.334" x2="20.327575" y2="5.334" width="0.1524" layer="16"/>
-<wire x1="10.409915625" y1="6.303853125" x2="10.867753125" y2="5.846015625" width="0.1524" layer="16"/>
-<wire x1="10.867753125" y1="5.814265625" x2="10.867753125" y2="6.117353125" width="0.1524" layer="16"/>
+<wire x1="10.963003125" y1="5.814265625" x2="10.963003125" y2="6.117353125" width="0.1524" layer="16"/>
 <wire x1="12.309796875" y1="6.1985" x2="12.26315" y2="6.151853125" width="0.1524" layer="16"/>
 <wire x1="12.26315" y1="6.151853125" x2="11.9255625" y2="5.814265625" width="0.1524" layer="16"/>
-<wire x1="11.9255625" y1="5.814265625" x2="10.899503125" y2="5.814265625" width="0.1524" layer="16"/>
+<wire x1="11.9255625" y1="5.814265625" x2="10.963003125" y2="5.814265625" width="0.1524" layer="16"/>
 <wire x1="24.431134375" y1="13.4027" x2="24.494634375" y2="13.3392" width="0.1524" layer="16"/>
 <wire x1="24.494634375" y1="13.3392" x2="24.494634375" y2="13.2122" width="0.1524" layer="16"/>
@@
 <wire x1="28.32311875" y1="2.766865625" x2="29.088896875" y2="3.53264375" width="0.1524" layer="1"/>
 <wire x1="28.32311875" y1="1.58961875" x2="28.32311875" y2="2.766865625" width="0.1524" layer="1"/>
-<wire x1="10.867753125" y1="6.117353125" x2="10.867753125" y2="5.846015625" width="0.1524" layer="16"/>
-<wire x1="10.867753125" y1="5.846015625" x2="10.899503125" y2="5.814265625" width="0.1524" layer="16"/>
 <contactref element="R20" pad="1"/>
 <contactref element="C9" pad="1"/>
@@
 <wire x1="33.59580625" y1="5.17094375" x2="32.4253625" y2="4.0005" width="0.1524" layer="16"/>
 <wire x1="32.4253625" y1="4.0005" x2="32.385" y2="4.0005" width="0.1524" layer="16"/>
+<wire x1="12.231775" y1="10.3632" x2="12.231775" y2="10.359425" width="0.1524" layer="16"/>
+<wire x1="12.231775" y1="10.359425" x2="11.8392" y2="9.96685" width="0.1524" layer="16"/>
+<wire x1="11.8392" y1="8.917671875" x2="11.43" y2="8.508471875" width="0.1524" layer="16"/>
+<wire x1="11.8392" y1="9.96685" x2="11.8392" y2="8.917671875" width="0.1524" layer="16"/>
+<wire x1="11.43" y1="8.508471875" x2="11.238071875" y2="8.508471875" width="0.1524" layer="16"/>
+<wire x1="11.238071875" y1="8.508471875" x2="10.795" y2="8.0654" width="0.1524" layer="16"/>
+<wire x1="10.804253125" y1="6.117353125" x2="10.963003125" y2="6.117353125" width="0.1524" layer="16"/>
+<wire x1="10.804253125" y1="6.117353125" x2="10.795" y2="6.12660625" width="0.1524" layer="16"/>
+<wire x1="10.795" y1="8.0654" x2="10.795" y2="6.12660625" width="0.1524" layer="16"/>
 </signal>
 <signal name="GAIN_OUT">

Commit message: Beta production board sync
Changed lines of the file:
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@@
 <contactref element="GND" pad="TP"/>
 <via x="24.3377125" y="8.683" extent="1-16" drill="0.3"/>
-<via x="17.0990875" y="9.21365625" extent="1-16" drill="0.3"/>
+<via x="15.5750875" y="11.78540625" extent="1-16" drill="0.3"/>
 <via x="19.54579375" y="5.937496875" extent="1-16" drill="0.3"/>
 <via x="31.6654625" y="7.972840625" extent="1-16" drill="0.3"/>

Commit message: Adjusted capacitor placement for easier soldering
Also optimized traces and ground plane
Parts:
- moved C7 2.09 mm to (30.8, 5.02), turned to 180 degrees
- moved C15 0.88 mm to (24.4, 2.13), turned to 90 degrees
- moved C14 0.51 mm to (25.2, 2.13), turned to 90 degrees
Routing:
- net PTAMP-: track 10.9 -> 12.4 mm
- net Z_TRG: track 7.01 -> 5.67 mm
- net V_FOL_PWM: track 13.3 -> 12.2 mm
- net GAIN_ADJ: track 26.6 -> 25.5 mm
- net GND: track 6.19 -> 5.37 mm
- net PT100_OUT: track 30.2 -> 29.5 mm
- net SCL: track 12.5 -> 12.0 mm
- net VCOMP_SENSE: track 25.5 -> 25.0 mm
