File: Eagle_Files/Standalone/Pyr0-Piezo-Standalone_2.1.1.brd (EAGLE design)
At the start: 43 x 15.4 mm, 66 parts, among them J1 CON-MOLEX-6P-1.25MM048, U2 L78L05ACU, U3 LM2902QT, U4 ATMEGA48/88/168/328PB

Commit message: fixed some file encoding issues
Routing:
- net SCL: track 11.7 -> 12.4 mm
Changed lines of the file:
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@@
 <?xml version="1.0" encoding="utf-8"?>
 <!DOCTYPE eagle SYSTEM "eagle.dtd">
-<eagle version="9.3.2">
+<eagle version="9.4.0">
 <drawing>
 <settings>
@@
 </signal>
 <signal name="SDA">
+<contactref element="J1" pad="1"/>
 <contactref element="U4" pad="3"/>
-<wire x1="16.71025" y1="6.084" x2="17.25" y2="6.084" width="0.1524" layer="1"/>
-<wire x1="16.2231" y1="6.57115" x2="16.71025" y2="6.084" width="0.1524" layer="1"/>
-<wire x1="16.2231" y1="6.57115" x2="16.2231" y2="7.46784375" width="0.1524" layer="1"/>
-<wire x1="15.77954375" y1="7.9114" x2="13.47465625" y2="7.9114" width="0.1524" layer="1"/>
-<wire x1="16.2231" y1="7.46784375" x2="15.77954375" y2="7.9114" width="0.1524" layer="1"/>
-<contactref element="J1" pad="1"/>
-<wire x1="13.47465625" y1="7.9114" x2="12.065" y2="9.32105625" width="0.1524" layer="1"/>
-<wire x1="12.065" y1="9.32105625" x2="12.065" y2="11.43" width="0.1524" layer="1"/>
-<wire x1="12.065" y1="11.43" x2="11.928665625" y2="11.43" width="0.1524" layer="1"/>
-<wire x1="11.928665625" y1="11.43" x2="11.411590625" y2="11.947075" width="0.1524" layer="1"/>
+<wire x1="17.25" y1="6.084" x2="16.80775" y2="6.084" width="0.1524" layer="1"/>
+<wire x1="16.2231" y1="7.46784375" x2="15.601" y2="8.08994375" width="0.1524" layer="1"/>
+<wire x1="16.80775" y1="6.084" x2="16.2231" y2="6.66865" width="0.1524" layer="1"/>
+<wire x1="16.2231" y1="6.66865" x2="16.2231" y2="7.46784375" width="0.1524" layer="1"/>
+<wire x1="15.601" y1="8.88613125" x2="15.56079375" y2="8.9263375" width="0.1524" layer="1"/>
+<wire x1="15.56079375" y1="8.9263375" x2="15.56079375" y2="10.27026875" width="0.1524" layer="1"/>
+<wire x1="15.56079375" y1="10.27026875" x2="15.2710125" y2="10.56005" width="0.1524" layer="1"/>
+<wire x1="15.2710125" y1="10.56005" x2="12.0777" y2="10.56005" width="0.1524" layer="1"/>
+<wire x1="15.601" y1="8.08994375" x2="15.601" y2="8.88613125" width="0.1524" layer="1"/>
+<wire x1="11.729090625" y1="11.629575" x2="11.411590625" y2="11.947075" width="0.1524" layer="1"/>
+<wire x1="11.729090625" y1="11.629575" x2="11.729090625" y2="10.908659375" width="0.1524" layer="1"/>
+<wire x1="12.0777" y1="10.56005" x2="11.729090625" y2="10.908659375" width="0.1524" layer="1"/>
 </signal>
 <signal name="SCL">
+<contactref element="J1" pad="2"/>
 <contactref element="U4" pad="6"/>
-<wire x1="17.25" y1="4.584" x2="16.371" y2="4.584" width="0.1524" layer="1"/>
-<wire x1="15.27175" y1="5.68325" x2="15.27175" y2="6.06425" width="0.1524" layer="1"/>
-<wire x1="16.371" y1="4.584" x2="15.27175" y2="5.68325" width="0.1524" layer="1"/>
-<wire x1="15.27175" y1="5.68325" x2="15.0424" y2="5.9126" width="0.1524" layer="1"/>
-<wire x1="15.0424" y1="5.9126" x2="15.0424" y2="5.9464" width="0.1524" layer="1"/>
+<wire x1="17.25" y1="4.584" x2="17.1086" y2="4.7254" width="0.1524" layer="1"/>
+<wire x1="15.58435" y1="5.42925" x2="15.5575" y2="5.42925" width="0.1524" layer="1"/>
+<wire x1="17.1086" y1="4.7254" x2="16.2882" y2="4.7254" width="0.1524" layer="1"/>
+<wire x1="16.2882" y1="4.7254" x2="15.58435" y2="5.42925" width="0.1524" layer="1"/>
+<wire x1="15.5575" y1="5.42925" x2="15.0424" y2="5.94435" width="0.1524" layer="1"/>
+<wire x1="15.0424" y1="5.94435" x2="15.0424" y2="5.9464" width="0.1524" layer="1"/>
 <via x="15.0424" y="5.9464" extent="1-16" drill="0.35"/>
-<wire x1="15.0424" y1="5.9464" x2="15.543896875" y2="6.447896875" width="0.1524" layer="16"/>
-<wire x1="15.543896875" y1="6.447896875" x2="15.543896875" y2="7.288896875" width="0.1524" layer="16"/>
-<via x="15.543896875" y="7.288896875" extent="1-16" drill="0.35"/>
-<wire x1="15.543896875" y1="7.288896875" x2="15.543896875" y2="7.292528125" width="0.1524" layer="1"/>
-<wire x1="15.543896875" y1="7.292528125" x2="15.229825" y2="7.6066" width="0.1524" layer="1"/>
-<wire x1="15.229825" y1="7.6066" x2="13.3484" y2="7.6066" width="0.1524" layer="1"/>
-<contactref element="J1" pad="2"/>
-<wire x1="13.3484" y1="7.6066" x2="11.7602" y2="9.1948" width="0.1524" layer="1"/>
-<wire x1="11.7602" y1="9.1948" x2="11.7602" y2="9.81075" width="0.1524" layer="1"/>
-<wire x1="11.7602" y1="9.81075" x2="10.52770625" y2="11.04324375" width="0.1524" layer="1"/>
-<wire x1="10.52770625" y1="11.04324375" x2="10.52770625" y2="11.063190625" width="0.1524" layer="1"/>
+<wire x1="15.0424" y1="5.9464" x2="15.57119375" y2="6.47519375" width="0.1524" layer="16"/>
+<wire x1="15.57119375" y1="6.47519375" x2="15.57119375" y2="7.2616" width="0.1524" layer="16"/>
+<via x="15.57119375" y="7.2616" extent="1-16" drill="0.35"/>
+<wire x1="15.57119375" y1="7.2616" x2="15.57119375" y2="7.68869375" width="0.1524" layer="1"/>
+<wire x1="15.57119375" y1="7.68869375" x2="15.2962" y2="7.9636875" width="0.1524" layer="1"/>
+<wire x1="15.2962" y1="7.9636875" x2="15.2962" y2="8.255" width="0.1524" layer="1"/>
+<wire x1="15.2962" y1="8.255" x2="15.25599375" y2="8.29520625" width="0.1524" layer="1"/>
+<wire x1="15.25599375" y1="8.29520625" x2="15.25599375" y2="10.14400625" width="0.1524" layer="1"/>
+<wire x1="15.25599375" y1="10.14400625" x2="15.14475" y2="10.25525" width="0.1524" layer="1"/>
+<wire x1="15.14475" y1="10.25525" x2="11.9514375" y2="10.25525" width="0.1524" layer="1"/>
+<wire x1="11.524496875" y1="10.682190625" x2="10.90870625" y2="10.682190625" width="0.1524" layer="1"/>
+<wire x1="10.90870625" y1="10.682190625" x2="10.52770625" y2="11.063190625" width="0.1524" layer="1"/>
+<wire x1="11.9514375" y1="10.25525" x2="11.524496875" y2="10.682190625" width="0.1524" layer="1"/>
 </signal>
 <signal name="Z_TRG">
@@
 <wire x1="15.58888125" y1="13.05661875" x2="15.06175" y2="13.58375" width="0.1524" layer="1"/>
 <wire x1="15.06175" y1="13.58375" x2="14.99825" y2="13.58375" width="0.1524" layer="1"/>
-<wire x1="15.86559375" y1="10.59381875" x2="15.58888125" y2="10.87053125" width="0.1524" layer="1"/>
-<wire x1="15.58888125" y1="10.87053125" x2="15.58888125" y2="13.05661875" width="0.1524" layer="1"/>
-<wire x1="15.86559375" y1="9.05259375" x2="15.86559375" y2="10.59381875" width="0.1524" layer="1"/>
+<wire x1="15.86559375" y1="10.43506875" x2="15.58888125" y2="10.71178125" width="0.1524" layer="1"/>
+<wire x1="15.58888125" y1="10.71178125" x2="15.58888125" y2="13.05661875" width="0.1524" layer="1"/>
+<wire x1="15.86559375" y1="9.05259375" x2="15.86559375" y2="10.43506875" width="0.1524" layer="1"/>
 </signal>
 <signal name="VCC_FUSE">
