File: Eagle_Files/FFC_Direct_Extruder/Pyr0-Piezo_Direct_Extruder_Board1.1.0.brd (EAGLE design)
At the start: 38.1 x 46.5 mm, 61 parts, among them J1 SFW24R-1STE1LF, U1 ATMEGA48PA-MMHR28M1-L, U2 LM2902QT

Commit message: Brought library additions to older rev boards
Parts:
- D1: value ZENER_DIODE_PLZ5V1C -> DIODE_ZENER_PLZ5V1C
- U1: value ATMEGA48PA-MMHR28M1-L -> ATMEGA48/88/168/328PA28M1-M; device PiezoFFC:28M1-L -> PiezoFFC:28M1-M
