File: Eagle_Files/FFC_Direct_Extruder/Pyr0-Piezo_Direct_Extruder_Board2.0.0.brd (EAGLE design)
At the start: 42.6 x 46.5 mm, 71 parts, among them J2 FFC_MOLEX_0.5MM, U1 ATMEGA48/88/168/328PA, U4 LM2902QT

Commit message: Brought library additions to older rev boards
Parts:
- D1: value ZENER_DIODE_PLZ5V1C -> DIODE_ZENER_PLZ5V1C
Changed lines of the file:
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@@
 <?xml version="1.0" encoding="utf-8"?>
 <!DOCTYPE eagle SYSTEM "eagle.dtd">
-<eagle version="9.3.0">
+<eagle version="9.3.2">
 <drawing>
 <settings>
@@
 <attribute name="VALUE" x="35.7877" y="30.35938125" size="0.0254" layer="28" rot="MR45"/>
 </element>
-<element name="D1" library="PiezoFFC" library_urn="urn:adsk.eagle:library:6897166" package="DO-219AC" package3d_urn="urn:adsk.eagle:package:8452796/2" value="ZENER_DIODE_PLZ5V1C" x="14.0915" y="29.5555" smashed="yes" rot="R270">
+<element name="D1" library="PiezoFFC" library_urn="urn:adsk.eagle:library:6897166" package="DO-219AC" package3d_urn="urn:adsk.eagle:package:8452796/2" value="DIODE_ZENER_PLZ5V1C" x="14.0915" y="29.5555" smashed="yes" rot="R270">
 <attribute name="NAME" x="14.1264" y="28.6665" size="0.6096" layer="25" font="vector" ratio="11" rot="R270" align="center-left"/>
 </element>
