File: Eagle_Files/Pyr0-Piezo_AVR_Programmer/Pyr0-Piezo_AVR_Board_Programmer_2.1.2.sch (EAGLE design)
At the start: 36 parts, among them J1 10118192-0001LF, U1 CP2102N-A01-GQFN28

Commit message: Complete overhaul of FFC board for v2.1.2 #bugfix
Parts:
- D2: value TVS_DIODE_CM1293A -> DIODE_TVS_ARRAY_CM1293A; device PiezoFFC:TVS_DIODE_CM1293A -> PiezoFFC:DIODE_TVS_ARRAY_CM1293A
- D3: value ZENER_DIODE_PLZ5V1C -> DIODE_ZENER_PLZ5V1C; device PiezoFFC:ZENER_DIODE_PLZ5V1C -> PiezoFFC:DIODE_ZENER_PLZ5V1C
Changed lines of the file:
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@@
 <part name="SUPPLY6" library="supply2" library_urn="urn:adsk.eagle:library:372" deviceset="GND" device=""/>
 <part name="R3" library="PiezoFFC" library_urn="urn:adsk.eagle:library:6897166" deviceset="SMD-RES-0R-5%-1/16W(0402)" device="" package3d_urn="urn:adsk.eagle:package:7115182/2"/>
-<part name="RXD" library="PiezoFFC" library_urn="urn:adsk.eagle:library:6897166" deviceset="TP" device="SPRING_CONTACT_3.5X1.1" package3d_urn="urn:adsk.eagle:package:8763770/2" value="TPSPRING_CONTACT_3.5X1.1"/>
-<part name="TXD" library="PiezoFFC" library_urn="urn:adsk.eagle:library:6897166" deviceset="TP" device="SPRING_CONTACT_3.5X1.1" package3d_urn="urn:adsk.eagle:package:8763770/2" value="TPSPRING_CONTACT_3.5X1.1"/>
-<part name="GND" library="PiezoFFC" library_urn="urn:adsk.eagle:library:6897166" deviceset="TP" device="SPRING_CONTACT_3.5X1.1" package3d_urn="urn:adsk.eagle:package:8763770/2" value="TPSPRING_CONTACT_3.5X1.1"/>
-<part name="+5V" library="PiezoFFC" library_urn="urn:adsk.eagle:library:6897166" deviceset="TP" device="SPRING_CONTACT_3.5X1.1" package3d_urn="urn:adsk.eagle:package:8763770/2" value="TPSPRING_CONTACT_3.5X1.1"/>
+<part name="RXD" library="PiezoFFC" library_urn="urn:adsk.eagle:library:6897166" deviceset="TP" device="SPRING_CONTACT_3.5X1.1" package3d_urn="urn:adsk.eagle:package:8763770/3" value="TPSPRING_CONTACT_3.5X1.1"/>
+<part name="TXD" library="PiezoFFC" library_urn="urn:adsk.eagle:library:6897166" deviceset="TP" device="SPRING_CONTACT_3.5X1.1" package3d_urn="urn:adsk.eagle:package:8763770/3" value="TPSPRING_CONTACT_3.5X1.1"/>
+<part name="GND" library="PiezoFFC" library_urn="urn:adsk.eagle:library:6897166" deviceset="TP" device="SPRING_CONTACT_3.5X1.1" package3d_urn="urn:adsk.eagle:package:8763770/3" value="TPSPRING_CONTACT_3.5X1.1"/>
+<part name="+5V" library="PiezoFFC" library_urn="urn:adsk.eagle:library:6897166" deviceset="TP" device="SPRING_CONTACT_3.5X1.1" package3d_urn="urn:adsk.eagle:package:8763770/3" value="TPSPRING_CONTACT_3.5X1.1"/>
 <part name="SUPPLY7" library="supply2" library_urn="urn:adsk.eagle:library:372" deviceset="GND" device=""/>
-<part name="RST." library="PiezoFFC" library_urn="urn:adsk.eagle:library:6897166" deviceset="TP" device="SPRING_CONTACT_3.5X1.1" package3d_urn="urn:adsk.eagle:package:8763770/2" value="TPSPRING_CONTACT_3.5X1.1"/>
+<part name="RST." library="PiezoFFC" library_urn="urn:adsk.eagle:library:6897166" deviceset="TP" device="SPRING_CONTACT_3.5X1.1" package3d_urn="urn:adsk.eagle:package:8763770/3" value="TPSPRING_CONTACT_3.5X1.1"/>
 <part name="PWR" library="PiezoFFC" library_urn="urn:adsk.eagle:library:6897166" deviceset="SEEED-LED_SMD-LED-CLEAR-BLUE(0603)" device="LED_0603" package3d_urn="urn:adsk.eagle:package:5224536/3"/>
 <part name="R8" library="PiezoFFC" library_urn="urn:adsk.eagle:library:6897166" deviceset="SMD-RES-0R-5%-1/16W(0402)" device="" package3d_urn="urn:adsk.eagle:package:7115182/2"/>
@@
 <part name="R2" library="PiezoFFC" library_urn="urn:adsk.eagle:library:6897166" deviceset="SMD-RES-0R-5%-1/16W(0402)" device="" package3d_urn="urn:adsk.eagle:package:7115182/2" value="47K"/>
 <part name="TTL" library="PiezoFFC" library_urn="urn:adsk.eagle:library:6897166" deviceset="JST-2.54MM_5P-2.54" device="JST_2.54MM_5P_F" package3d_urn="urn:adsk.eagle:package:5071743/2"/>
-<part name="U1" library="PiezoFFC" library_urn="urn:adsk.eagle:library:6897166" deviceset="CP2102N-A01-GQFN28" device="" package3d_urn="urn:adsk.eagle:package:8319976/2"/>
+<part name="U1" library="PiezoFFC" library_urn="urn:adsk.eagle:library:6897166" deviceset="CP2102N-A01-GQFN28" device="" package3d_urn="urn:adsk.eagle:package:8319976/3"/>
 <part name="R4" library="PiezoFFC" library_urn="urn:adsk.eagle:library:6897166" deviceset="SMD-RES-0R-5%-1/16W(0402)" device="" package3d_urn="urn:adsk.eagle:package:7115182/2" value="10K"/>
 <part name="C1" library="PiezoFFC" library_urn="urn:adsk.eagle:library:6897166" deviceset="CERAMIC-1NF-50V-10%-X7R(0402)" device="CAP_0402" package3d_urn="urn:adsk.eagle:package:5248669/4" value="0.1uF"/>
@@
 <part name="ICSP0" library="PiezoFFC" library_urn="urn:adsk.eagle:library:6897166" deviceset="ICSP_HEADER" device="SPRING_3.48X1.1" package3d_urn="urn:adsk.eagle:package:8763833/2" value="ICSP_HEADERSPRING_3.48X1.1"/>
 <part name="SUPPLY2" library="supply2" library_urn="urn:adsk.eagle:library:372" deviceset="GND" device=""/>
-<part name="D2" library="PiezoFFC" library_urn="urn:adsk.eagle:library:6897166" deviceset="TVS_DIODE_CM1293A" device="" package3d_urn="urn:adsk.eagle:package:8452336/3"/>
+<part name="D2" library="PiezoFFC" library_urn="urn:adsk.eagle:library:6897166" deviceset="DIODE_TVS_ARRAY_CM1293A" device="" package3d_urn="urn:adsk.eagle:package:8452336/4"/>
 <part name="ICSP2" library="PiezoFFC" library_urn="urn:adsk.eagle:library:6897166" deviceset="ICSP_HEADER" device="SPRING_3.48X1.1" package3d_urn="urn:adsk.eagle:package:8763833/2" value="ICSP_HEADERSPRING_3.48X1.1"/>
 <part name="C3" library="PiezoFFC" library_urn="urn:adsk.eagle:library:6897166" deviceset="CERAMIC-1NF-50V-10%-X7R(0402)" device="CAP_0402" package3d_urn="urn:adsk.eagle:package:5248669/4" value="0.1uF"/>
@@
 <part name="C5" library="PiezoFFC" library_urn="urn:adsk.eagle:library:6897166" deviceset="SEEED-CAPACITOR_CERAMIC-10UF-25V-10%-X5R(0805)" device="CAP_0805-3D" package3d_urn="urn:adsk.eagle:package:5225034/2" value="4.7uF"/>
 <part name="R5" library="PiezoFFC" library_urn="urn:adsk.eagle:library:6897166" deviceset="SMD-RES-0R-5%-1/16W(0402)" device="" package3d_urn="urn:adsk.eagle:package:7115182/2" value="10K"/>
-<part name="D3" library="PiezoFFC" library_urn="urn:adsk.eagle:library:6897166" deviceset="ZENER_DIODE_PLZ5V1C" device="" package3d_urn="urn:adsk.eagle:package:8452796/2"/>
-<part name="PZ+" library="PiezoFFC" library_urn="urn:adsk.eagle:library:6897166" deviceset="TP" device="SPRING_CONTACT_3.5X1.1" package3d_urn="urn:adsk.eagle:package:8763770/2" value="TPSPRING_CONTACT_3.5X1.1"/>
-<part name="VCOM" library="PiezoFFC" library_urn="urn:adsk.eagle:library:6897166" deviceset="TP" device="SPRING_CONTACT_3.5X1.1" package3d_urn="urn:adsk.eagle:package:8763770/2" value="TPSPRING_CONTACT_3.5X1.1"/>
-<part name="GOUT" library="PiezoFFC" library_urn="urn:adsk.eagle:library:6897166" deviceset="TP" device="SPRING_CONTACT_3.5X1.1" package3d_urn="urn:adsk.eagle:package:8763770/2" value="TPSPRING_CONTACT_3.5X1.1"/>
+<part name="D3" library="PiezoFFC" library_urn="urn:adsk.eagle:library:6897166" deviceset="DIODE_ZENER_PLZ5V1C" device="" package3d_urn="urn:adsk.eagle:package:8452796/2"/>
+<part name="PZ+" library="PiezoFFC" library_urn="urn:adsk.eagle:library:6897166" deviceset="TP" device="SPRING_CONTACT_3.5X1.1" package3d_urn="urn:adsk.eagle:package:8763770/3" value="TPSPRING_CONTACT_3.5X1.1"/>
+<part name="VCOM" library="PiezoFFC" library_urn="urn:adsk.eagle:library:6897166" deviceset="TP" device="SPRING_CONTACT_3.5X1.1" package3d_urn="urn:adsk.eagle:package:8763770/3" value="TPSPRING_CONTACT_3.5X1.1"/>
+<part name="GOUT" library="PiezoFFC" library_urn="urn:adsk.eagle:library:6897166" deviceset="TP" device="SPRING_CONTACT_3.5X1.1" package3d_urn="urn:adsk.eagle:package:8763770/3" value="TPSPRING_CONTACT_3.5X1.1"/>
 <part name="TJ1" library="PiezoFFC" library_urn="urn:adsk.eagle:library:6897166" deviceset="C-GRID-04" device="-70553" package3d_urn="urn:adsk.eagle:package:6902618/2"/>
-<part name="VFOL" library="PiezoFFC" library_urn="urn:adsk.eagle:library:6897166" deviceset="TP" device="SPRING_CONTACT_3.5X1.1" package3d_urn="urn:adsk.eagle:package:8763770/2" value="TPSPRING_CONTACT_3.5X1.1"/>
+<part name="VFOL" library="PiezoFFC" library_urn="urn:adsk.eagle:library:6897166" deviceset="TP" device="SPRING_CONTACT_3.5X1.1" package3d_urn="urn:adsk.eagle:package:8763770/3" value="TPSPRING_CONTACT_3.5X1.1"/>
 </parts>
 <sheets>
