File: Eagle_Files/Pyr0-Piezo_DIY-Boards/Pyr0-Piezo-v2-DIY-Standalone-Board_v1.0.0.brd (EAGLE design)
At the start: 45.6 x 18.3 mm, 37 parts, among them J1 PP-STANDALONE-HEADER, U1 LM2902D

Commit message: fixed polarity for trigger LED on DIY board #bugfix
Parts:
- turned TRIG to 180 degrees
Connections:
- net GND: now also TRIG.C
- net LED_VCC: no longer TRIG.A
- net Z_TRG: now also TRIG.A; no longer TRIG.C
Routing:
- net LED_VCC: track 3.89 -> 1.99 mm
Changed lines of the file:
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@@
 <attribute name="MF" value="MOLEX" x="57.149996875" y="9.525" size="1.778" layer="27" rot="R270" display="off"/>
 <attribute name="MPN" value="" x="57.149996875" y="9.525" size="1.778" layer="27" rot="R270" display="off"/>
-<attribute name="NAME" x="49.92325625" y="1.968028125" size="0.8128" layer="25" font="vector" rot="R180"/>
+<attribute name="NAME" x="40.62774375" y="7.683971875" size="1.27" layer="25" font="vector"/>
 <attribute name="OC_FARNELL" value="unknown" x="57.149996875" y="9.525" size="1.778" layer="27" rot="R270" display="off"/>
 <attribute name="OC_NEWARK" value="unknown" x="57.149996875" y="9.525" size="1.778" layer="27" rot="R270" display="off"/>
@@
 <attribute name="VALUE" x="12.7" y="8.89" size="1.27" layer="27" rot="R90"/>
 </element>
-<element name="TRIG" library="PiezoFFC" library_urn="urn:adsk.eagle:library:6897166" package="CHIP-LED0805" package3d_urn="urn:adsk.eagle:package:15818/2" value="" x="8.255" y="10.16" smashed="yes">
+<element name="TRIG" library="PiezoFFC" library_urn="urn:adsk.eagle:library:6897166" package="CHIP-LED0805" package3d_urn="urn:adsk.eagle:package:15818/2" value="" x="8.255" y="10.16" smashed="yes" rot="R180">
 <attribute name="NAME" x="7.62" y="8.128" size="1.27" layer="25" rot="R270"/>
-<attribute name="VALUE" x="10.795" y="8.89" size="1.27" layer="27" rot="R90"/>
+<attribute name="VALUE" x="5.715" y="11.43" size="1.27" layer="27" rot="R270"/>
 </element>
 <element name="R19" library="PiezoFFC" library_urn="urn:adsk.eagle:library:6897166" package="R0805" package3d_urn="urn:adsk.eagle:package:8443791/3" value="4K7" x="12.065" y="10.16" smashed="yes" rot="R90">
@@
 </polygon>
 <contactref element="PWR" pad="C"/>
+<contactref element="TRIG" pad="C"/>
 </signal>
 <signal name="Z_TRG">
@@
 <wire x1="8.421" y1="15.074" x2="8.255" y2="15.24" width="0.254" layer="1"/>
 <wire x1="8.255" y1="15.24" x2="6.985" y2="15.24" width="0.254" layer="1"/>
-<contactref element="TRIG" pad="C"/>
 <wire x1="6.985" y1="15.24" x2="5.08" y2="15.24" width="0.254" layer="1"/>
-<wire x1="8.255" y1="11.21" x2="6.985" y2="12.48" width="0.254" layer="1"/>
-<wire x1="6.985" y1="12.48" x2="6.985" y2="15.24" width="0.254" layer="1"/>
+<wire x1="6.985" y1="15.24" x2="6.985" y2="12.48" width="0.254" layer="1"/>
+<contactref element="TRIG" pad="A"/>
+<wire x1="6.985" y1="12.48" x2="8.255" y2="11.21" width="0.254" layer="1"/>
 </signal>
 <signal name="PZ+">
@@
 </signal>
 <signal name="LED_VCC">
-<contactref element="TRIG" pad="A"/>
 <contactref element="R19" pad="1"/>
 <contactref element="PWR" pad="A"/>
-<wire x1="8.255" y1="9.11" x2="10.16" y2="9.11" width="0.254" layer="1"/>
 <wire x1="12.065" y1="9.31" x2="10.36" y2="9.31" width="0.254" layer="1"/>
 <wire x1="10.36" y1="9.31" x2="10.16" y2="9.11" width="0.254" layer="1"/>
