File: Eagle_Files/Pyr0-Piezo_DIY-Boards/Pyr0-Piezo-v2-DIY-Standalone-Board_v1.0.0.sch (EAGLE design)
At the start: 37 parts, among them J1 PP-STANDALONE-HEADER, U1 LM2902D

Commit message: fixed polarity for trigger LED on DIY board #bugfix
Connections:
- net GND: now also TRIG.C
- net LED_VCC: no longer TRIG.A
- net Z_TRG: now also TRIG.A; no longer TRIG.C
Other:
- moved on the sheet: PWR, R19, TRIG
Changed lines of the file:
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@@
 <setting verticaltext="up"/>
 </settings>
-<grid distance="1.27" unitdist="mm" unit="mm" style="lines" multiple="1" display="no" altdistance="0.01" altunitdist="inch" altunit="mm"/>
+<grid distance="1.27" unitdist="mm" unit="mm" style="lines" multiple="1" display="no" altdistance="0.01" altunitdist="inch" altunit="inch"/>
 <layers>
 <layer number="1" name="Top" color="4" fill="1" visible="no" active="no"/>
@@
 <attribute name="VALUE" x="64.77" y="22.86" size="1.27" layer="96" ratio="10" rot="R180"/>
 </instance>
-<instance part="PWR" gate="G$1" x="189.23" y="114.3" smashed="yes">
-<attribute name="NAME" x="192.786" y="109.728" size="1.778" layer="95" rot="R90"/>
-<attribute name="VALUE" x="194.945" y="109.728" size="1.778" layer="96" rot="R90"/>
-</instance>
-<instance part="TRIG" gate="G$1" x="180.34" y="114.3" smashed="yes">
-<attribute name="NAME" x="183.896" y="109.728" size="1.778" layer="95" rot="R90"/>
-<attribute name="VALUE" x="186.055" y="109.728" size="1.778" layer="96" rot="R90"/>
-</instance>
-<instance part="R19" gate="G$1" x="180.34" y="123.19" smashed="yes" rot="R90">
-<attribute name="NAME" x="179.07" y="121.92" size="1.27" layer="95" ratio="10" rot="R90"/>
-<attribute name="VALUE" x="181.61" y="124.46" size="1.27" layer="96" ratio="10" rot="R270"/>
-</instance>
-<instance part="P+3" gate="1" x="180.34" y="133.35" smashed="yes">
-<attribute name="VALUE" x="177.8" y="128.27" size="1.778" layer="96" rot="R90"/>
-</instance>
-<instance part="SUPPLY7" gate="GND" x="189.23" y="106.68" smashed="yes">
-<attribute name="VALUE" x="187.325" y="103.505" size="1.778" layer="96"/>
+<instance part="PWR" gate="G$1" x="124.46" y="12.7" smashed="yes">
+<attribute name="NAME" x="128.016" y="8.128" size="1.778" layer="95" rot="R90"/>
+<attribute name="VALUE" x="130.175" y="8.128" size="1.778" layer="96" rot="R90"/>
+</instance>
+<instance part="TRIG" gate="G$1" x="114.3" y="12.7" smashed="yes">
+<attribute name="NAME" x="117.856" y="8.128" size="1.778" layer="95" rot="R90"/>
+<attribute name="VALUE" x="120.015" y="8.128" size="1.778" layer="96" rot="R90"/>
+</instance>
+<instance part="R19" gate="G$1" x="124.46" y="21.59" smashed="yes" rot="R90">
+<attribute name="NAME" x="123.19" y="20.32" size="1.27" layer="95" ratio="10" rot="R90"/>
+<attribute name="VALUE" x="125.73" y="22.86" size="1.27" layer="96" ratio="10" rot="R270"/>
+</instance>
+<instance part="P+3" gate="1" x="124.46" y="31.75" smashed="yes">
+<attribute name="VALUE" x="121.92" y="26.67" size="1.778" layer="96" rot="R90"/>
+</instance>
+<instance part="SUPPLY7" gate="GND" x="124.46" y="2.54" smashed="yes">
+<attribute name="VALUE" x="122.555" y="-0.635" size="1.778" layer="96"/>
 </instance>
 </instances>
@@
 <pinref part="SUPPLY7" gate="GND" pin="GND"/>
 <pinref part="PWR" gate="G$1" pin="C"/>
+<wire x1="124.46" y1="5.08" x2="124.46" y2="6.35" width="0.1524" layer="91"/>
+<pinref part="TRIG" gate="G$1" pin="C"/>
+<wire x1="124.46" y1="6.35" x2="124.46" y2="7.62" width="0.1524" layer="91"/>
+<wire x1="114.3" y1="7.62" x2="114.3" y2="6.35" width="0.1524" layer="91"/>
+<wire x1="114.3" y1="6.35" x2="124.46" y2="6.35" width="0.1524" layer="91"/>
+<junction x="124.46" y="6.35"/>
 </segment>
 </net>
@@
 <pinref part="J1" gate="G$2" pin="Z-TRG"/>
 <pinref part="R10" gate="G$1" pin="2"/>
-<pinref part="TRIG" gate="G$1" pin="C"/>
 <wire x1="180.34" y1="97.79" x2="182.88" y2="97.79" width="0.1524" layer="91"/>
-<wire x1="180.34" y1="109.22" x2="180.34" y2="97.79" width="0.1524" layer="91"/>
-<junction x="180.34" y="97.79"/>
+</segment>
+<segment>
+<pinref part="TRIG" gate="G$1" pin="A"/>
+<wire x1="114.3" y1="15.24" x2="114.3" y2="20.32" width="0.1524" layer="91"/>
+<label x="114.3" y="20.32" size="1.778" layer="95" rot="R90" xref="yes"/>
 </segment>
 </net>
@@
 <pinref part="R19" gate="G$1" pin="2"/>
 <pinref part="P+3" gate="1" pin="+5V"/>
-<wire x1="180.34" y1="127" x2="180.34" y2="130.81" width="0.1524" layer="91"/>
+<wire x1="124.46" y1="25.4" x2="124.46" y2="29.21" width="0.1524" layer="91"/>
 </segment>
 </net>
@@
 <net name="LED_VCC" class="0">
 <segment>
-<pinref part="TRIG" gate="G$1" pin="A"/>
 <pinref part="R19" gate="G$1" pin="1"/>
-<wire x1="180.34" y1="116.84" x2="180.34" y2="118.11" width="0.1524" layer="91"/>
 <pinref part="PWR" gate="G$1" pin="A"/>
-<wire x1="180.34" y1="118.11" x2="180.34" y2="119.38" width="0.1524" layer="91"/>
-<wire x1="189.23" y1="116.84" x2="189.23" y2="118.11" width="0.1524" layer="91"/>
-<wire x1="189.23" y1="118.11" x2="180.34" y2="118.11" width="0.1524" layer="91"/>
-<junction x="180.34" y="118.11"/>
-</segment>
-</net>
+<wire x1="124.46" y1="16.51" x2="124.46" y2="17.78" width="0.1524" layer="91"/>
+<wire x1="124.46" y1="15.24" x2="124.46" y2="16.51" width="0.1524" layer="91"/>
+</segment>
+</net>
