File: Eagle_Files/Pyr0-Piezo_DIY-Boards/Pyr0-Piezo-v2-DIY-Business-Card.brd (EAGLE design)
At the start: 88.9 x 50.8 mm, 48 parts, among them J1 PP-STANDALONE-HEADER, U1 LM2902N, U2 ATMEGA328P

Commit message: Finished business card design
Parts:
- added U$5: (no value), PiezoFFC:LOGO-PYR0BALL-SS-6MM
- moved U$1 2.01 mm to (64.1, 41.9)
- moved U$2 2.01 mm to (64.1, 41.9)
- moved U$3 2.01 mm to (64.1, 41.9)
- moved U$4 2.01 mm to (64.1, 41.9)
- moved PZ-IN 1.91 mm to (85.7, 25.4)
- moved R2 1.91 mm to (74.9, 25.4)
Connections:
- net VCOMP_SENSE: now also J1.11
- net V_FOLLOW: now also J1.10
Routing:
- net V_FOLLOW: track 31.3 -> 62.3 mm, vias 0 -> 2
- net VCOMP_SENSE: track 15.9 -> 44.7 mm, vias 0 -> 1
- net Z_MIN_TRIG: track 42.5 -> 44.2 mm
- net PZ+: track 32.6 -> 31.8 mm
Other:
- board size 88.9 x 50.8 mm -> 88.9 x 49.5 mm
- board text added: "/u/pyr0ball"
- board text added: "1 - +5V 2 - GADJ_R0 3 - GADJ_R1 4 - GADJ_R2 5 - GADJ_R3 6 - PT100_OUT 7 - GND 8 - VCOMP_PWM 9 - VFOL_PWM 10 - VFOL_SENSE 11 - VCOMP_SENSE 12 - Z_TRIG"
- board text added: "@pyr0ball"
- board text added: "Comparator"
- board text added: "Gain Adjust"
- board text added: "Voltage Follower"
- board text removed: "1 - +5V 2 - GADJ_R0 3 - GADJ_R1 4 - GADJ_R2 5 - GADJ_R3 6 - PT100_OUT 7 - GND 8 - VCOMP_PWM 9 - VFOL_PWM 10 - N/C 11 - N/C 12 - Z_TRIG"
