File: Eagle_Files/Pyr0-Piezo_DIY-Boards/Pyr0-Piezo-v2-DIY-Business-Card.sch (EAGLE design)
At the start: 44 parts, among them J1 PP-STANDALONE-HEADER, U1 LM2902N, U2 ATMEGA328P

Commit message: Finished business card design
Connections:
- net VCOMP_SENSE: now also J1G$5.FOL_S
- net V_FOLLOW: now also J1G$5.COMP_S
Changed lines of the file:
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@@
 <setting verticaltext="up"/>
 </settings>
-<grid distance="1.27" unitdist="mm" unit="mm" style="lines" multiple="1" display="no" altdistance="0.01" altunitdist="inch" altunit="mm"/>
+<grid distance="0.1" unitdist="inch" unit="inch" style="lines" multiple="1" display="no" altdistance="0.01" altunitdist="inch" altunit="inch"/>
 <layers>
 <layer number="1" name="Top" color="4" fill="1" visible="no" active="no"/>
@@
 <attribute name="VALUE" x="109.22" y="127.2286" size="1.778" layer="96"/>
 </instance>
+<instance part="J1" gate="G$5" x="274.32" y="50.8" smashed="yes"/>
 </instances>
 <busses>
@@
 <label x="49.53" y="118.11" size="1.778" layer="95" xref="yes"/>
 </segment>
+<segment>
+<pinref part="J1" gate="G$5" pin="COMP_S"/>
+<wire x1="269.24" y1="45.72" x2="259.08" y2="45.72" width="0.1524" layer="91"/>
+<label x="256.54" y="45.72" size="1.778" layer="95"/>
+</segment>
 </net>
 <net name="VCOMP_SENSE" class="0">
@@
 <label x="49.53" y="115.57" size="1.778" layer="95" xref="yes"/>
 </segment>
+<segment>
+<pinref part="J1" gate="G$5" pin="FOL_S"/>
+<wire x1="269.24" y1="55.88" x2="259.08" y2="55.88" width="0.1524" layer="91"/>
+<label x="254" y="55.88" size="1.778" layer="95"/>
+</segment>
 </net>
