File: Eagle_Files/EasyPiezi/EasyPiezi_2.2.0.brd (EAGLE design)
At the start: 43 x 15.4 mm, 70 parts, among them J1 CON-MOLEX-6P-1.25MM048, U2 L78L05ACU, U3 LM2902QT, U4 ATMEGA48/88/168/328PB

Commit message: Fixed pad thermals, added url, fixed logo #bugfix
Parts:
- moved U$2 3.35 mm to (22.4, 12.3)
- moved U$1 3.30 mm to (22.2, 8.13)
- moved R15 0.89 mm to (20.0, 10.7)
- moved R21 0.25 mm to (27.2, 1.97)
- moved TP_F 0.13 mm to (23.6, 5.05)
Routing:
- net GND: track 6.13 -> 7.42 mm
- net PZ_AMP_OUT: track 7.17 -> 8.16 mm
- net Z_TRG: track 5.96 -> 5.19 mm
Other:
- board text added: "EasyPiezi v2.2.0"
- board text added: "docs.pyroballpcbs.com"
- board text removed: "EasyPiezi v2.1.2"
