File: Eagle_Files/PiezoDisk-PCB/Pyr0-Piezo_SingleDisk_Adapter_3pin.brd (EAGLE design)
At the start: 21.6 x 20 mm, 4 parts, among them J1 C-GRID-03-70553

Commit message: gave singledisk pcb a bit more flex for better sensitivity #bugfix
Parts:
- PZ1: value PIEZO-DISK12MM -> PIEZO-DISK12MM-OFFSET; device PiezoFFC:PIEZO-DISK-12MM -> PiezoFFC:PIEZO-DISK-12MM-OFFSET
- moved PZ1 0.64 mm to (0.00, 0.64)
Connections:
- net GND: no longer PZ1.GND4
Routing:
- net PZ+: track 12.1 -> 11.2 mm
Other:
- board size 21.6 x 20 mm -> 21.6 x 19 mm
Changed lines of the file:
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@@
 </layers>
 <board>
-<fusionsync huburn="a.cGVyc29uYWw6dWUyYTEyMDdh" projecturn="a.cGVyc29uYWw6dWUyYTEyMDdhIzIwMTgxMTI5MTYyOTY3NjMx" f3durn="urn:adsk.wipprod:dm.lineage:7ePR4_QuQeiO7QY8erFDCw" pcbguid="d4991351-07ad-4ba6-9d91-f49c73d368d4" lastpulledtime="" lastsyncedchangeguid="1955d288-6f82-8a71-617e-abfcb1f65f0e"/>
+<fusionsync huburn="a.cGVyc29uYWw6dWUyYTEyMDdh" projecturn="a.cGVyc29uYWw6dWUyYTEyMDdhIzIwMTgxMTI5MTYyOTY3NjMx" f3durn="urn:adsk.wipprod:dm.lineage:7ePR4_QuQeiO7QY8erFDCw" pcbguid="d4991351-07ad-4ba6-9d91-f49c73d368d4" lastpulledtime="" lastsyncedchangeguid="b91400a7-0863-90be-fe90-801656f4d338"/>
 <plain>
-<wire x1="-10.795" y1="-3.06" x2="-10.795" y2="-13.78" width="0" layer="20"/>
+<wire x1="-10.795" y1="-4.965" x2="-10.795" y2="-13.78" width="0" layer="20"/>
 <wire x1="-10.795" y1="-13.78" x2="-6.795" y2="-17.78" width="0" layer="20" curve="90"/>
 <wire x1="-6.795" y1="-17.78" x2="6.775" y2="-17.78" width="0" layer="20"/>
 <wire x1="6.775" y1="-17.78" x2="10.775" y2="-13.78" width="0" layer="20" curve="90"/>
-<wire x1="10.775" y1="-13.78" x2="10.775" y2="-3.06" width="0" layer="20"/>
-<wire x1="6.775" y1="2.21" x2="5.385" y2="2.21" width="0" layer="20"/>
-<wire x1="5.385" y1="2.21" x2="4.7625" y2="1.5875" width="0" layer="20"/>
-<wire x1="4.7625" y1="1.5875" x2="4.7625" y2="-1.5875" width="0" layer="20"/>
-<wire x1="4.7625" y1="-1.5875" x2="4.699" y2="-1.778" width="0" layer="20"/>
-<wire x1="4.699" y1="-1.778" x2="2.286" y2="-4.191" width="0" layer="20" curve="-53.130102"/>
-<wire x1="2.286" y1="-4.191" x2="2.032" y2="-4.191" width="0" layer="20"/>
-<wire x1="2.032" y1="-4.191" x2="1.27" y2="-3.429" width="0" layer="20" curve="-90"/>
-<wire x1="1.27" y1="-3.429" x2="1.27" y2="-1.651" width="0" layer="20"/>
-<wire x1="1.27" y1="-1.651" x2="1.397" y2="-1.524" width="0" layer="20"/>
-<wire x1="1.397" y1="-1.524" x2="0.889" y2="1.905" width="0" layer="20" curve="106.853992"/>
-<wire x1="0.889" y1="1.905" x2="-0.889" y2="1.905" width="0" layer="20"/>
-<wire x1="-6.775" y1="2.21" x2="-5.385" y2="2.21" width="0" layer="20"/>
-<wire x1="-5.385" y1="2.21" x2="-4.7625" y2="1.5875" width="0" layer="20"/>
-<wire x1="-4.7625" y1="1.5875" x2="-4.7625" y2="-1.5875" width="0" layer="20"/>
-<wire x1="-4.7625" y1="-1.5875" x2="-4.699" y2="-1.778" width="0" layer="20"/>
-<wire x1="-4.699" y1="-1.778" x2="-2.286" y2="-4.191" width="0" layer="20" curve="53.130102"/>
-<wire x1="-2.286" y1="-4.191" x2="-2.032" y2="-4.191" width="0" layer="20"/>
-<wire x1="-2.032" y1="-4.191" x2="-1.27" y2="-3.429" width="0" layer="20" curve="90"/>
-<wire x1="-1.27" y1="-3.429" x2="-1.27" y2="-1.651" width="0" layer="20"/>
-<wire x1="-1.27" y1="-1.651" x2="-1.397" y2="-1.524" width="0" layer="20"/>
-<wire x1="-1.397" y1="-1.524" x2="-0.889" y2="1.905" width="0" layer="20" curve="-106.853992"/>
-<wire x1="-10.795" y1="-3.06" x2="-6.775" y2="2.21" width="0" layer="20" curve="-75.323607"/>
-<wire x1="10.775" y1="-3.06" x2="6.775" y2="2.21" width="0" layer="20" curve="75.323607"/>
+<wire x1="10.775" y1="-13.78" x2="10.775" y2="-4.965" width="0" layer="20"/>
+<wire x1="6.775" y1="1.2575" x2="5.385" y2="1.2575" width="0" layer="20"/>
+<wire x1="5.385" y1="1.2575" x2="4.7625" y2="0.635" width="0" layer="20"/>
+<wire x1="4.7625" y1="0.635" x2="4.7625" y2="-0.635" width="0" layer="20"/>
+<wire x1="4.7625" y1="-0.635" x2="4.699" y2="-0.8255" width="0" layer="20"/>
+<wire x1="4.699" y1="-0.8255" x2="2.286" y2="-3.556" width="0" layer="20" curve="-40"/>
+<wire x1="2.286" y1="-3.556" x2="2.032" y2="-3.556" width="0" layer="20"/>
+<wire x1="2.032" y1="-3.556" x2="1.27" y2="-2.921" width="0" layer="20" curve="-90"/>
+<wire x1="1.27" y1="-2.921" x2="1.397" y2="-2.4765" width="0" layer="20"/>
+<wire x1="1.397" y1="-2.4765" x2="0.889" y2="0.9525" width="0" layer="20" curve="106.853992"/>
+<wire x1="0.889" y1="0.9525" x2="-0.889" y2="0.9525" width="0" layer="20"/>
+<wire x1="-6.775" y1="1.2575" x2="-5.385" y2="1.2575" width="0" layer="20"/>
+<wire x1="-5.385" y1="1.2575" x2="-4.7625" y2="0.635" width="0" layer="20"/>
+<wire x1="-4.7625" y1="0.635" x2="-4.7625" y2="-0.635" width="0" layer="20"/>
+<wire x1="-4.7625" y1="-0.635" x2="-4.699" y2="-0.8255" width="0" layer="20"/>
+<wire x1="-4.699" y1="-0.8255" x2="-2.286" y2="-3.556" width="0" layer="20" curve="30"/>
+<wire x1="-2.286" y1="-3.556" x2="-2.032" y2="-3.556" width="0" layer="20"/>
+<wire x1="-2.032" y1="-3.556" x2="-1.27" y2="-2.921" width="0" layer="20" curve="90"/>
+<wire x1="-1.27" y1="-2.921" x2="-1.397" y2="-2.4765" width="0" layer="20"/>
+<wire x1="-1.397" y1="-2.4765" x2="-0.889" y2="0.9525" width="0" layer="20" curve="-106.853992"/>
+<wire x1="-10.795" y1="-4.965" x2="-6.775" y2="1.2575" width="0" layer="20" curve="-75.323607"/>
+<wire x1="10.775" y1="-4.965" x2="6.775" y2="1.2575" width="0" layer="20" curve="75.323607"/>
 </plain>
 <attributes>
@@
 <attribute name="OC_NEWARK" value="unknown" x="-19.05" y="-9.525" size="1.778" layer="27" rot="R180" display="off"/>
 </element>
-<element name="PZ1" library="PiezoFFC" library_urn="urn:adsk.eagle:library:6897166" package="PIEZO-DISK-12MM" package3d_urn="urn:adsk.eagle:package:14393959/5" value="PIEZO-DISK12MM" x="0" y="0" smashed="yes" rot="R180"/>
+<element name="PZ1" library="PiezoFFC" library_urn="urn:adsk.eagle:library:6897166" package="PIEZO-DISK-12MM-OFFSET" package3d_urn="urn:adsk.eagle:package:16537148/2" value="PIEZO-DISK12MM-OFFSET" x="0" y="0.635" smashed="yes" rot="R180"/>
 <element name="H1" library="PiezoFFC" library_urn="urn:adsk.eagle:library:6897166" package="HOLES_3,2-PAD" package3d_urn="urn:adsk.eagle:package:5224590/3" value="HOLES_MOUNT-PAD-ROUND3.2" x="6.35" y="-8.255" smashed="yes"/>
 <element name="H2" library="PiezoFFC" library_urn="urn:adsk.eagle:library:6897166" package="HOLES_3,2-PAD" package3d_urn="urn:adsk.eagle:package:5224590/3" value="HOLES_MOUNT-PAD-ROUND3.2" x="-6.35" y="-8.255" smashed="yes"/>
@@
 <signals>
 <signal name="PZ+">
-<contactref element="PZ1" pad="PZ+" route="any" routetag="G$1.PZ+"/>
+<contactref element="PZ1" pad="PZ+"/>
 <contactref element="J1" pad="2"/>
-<wire x1="0" y1="0" x2="0" y2="-12.065" width="0.508" layer="16"/>
+<wire x1="0" y1="-0.865" x2="0" y2="-12.065" width="0.508" layer="16"/>
 </signal>
 <signal name="GND">
@@
 <contactref element="PZ1" pad="GND2"/>
 <contactref element="PZ1" pad="GND3"/>
-<contactref element="PZ1" pad="GND4"/>
 <polygon width="0.254" layer="1">
-<vertex x="-10.795" y="0.94"/>
+<vertex x="-10.795" y="-0.0125"/>
 <vertex x="-10.795" y="-17.78"/>
 <vertex x="10.775" y="-17.78"/>
-<vertex x="10.775" y="0.94"/>
-<vertex x="2.235" y="0.94"/>
-<vertex x="1.27" y="1.905"/>
-<vertex x="-1.27" y="1.905"/>
-<vertex x="-2.235" y="0.94"/>
+<vertex x="10.775" y="-0.0125"/>
+<vertex x="2.235" y="-0.0125"/>
+<vertex x="1.27" y="0.9525"/>
+<vertex x="-1.27" y="0.9525"/>
+<vertex x="-2.235" y="-0.0125"/>
 </polygon>
 <polygon width="0.254" layer="16">
-<vertex x="-10.795" y="0.94"/>
+<vertex x="-10.795" y="-0.0125"/>
 <vertex x="-10.795" y="-17.78"/>
 <vertex x="10.775" y="-17.78"/>
-<vertex x="10.775" y="0.94"/>
-<vertex x="2.235" y="0.94"/>
-<vertex x="1.27" y="1.905"/>
-<vertex x="-1.27" y="1.905"/>
-<vertex x="-2.235" y="0.94"/>
+<vertex x="10.775" y="-0.0125"/>
+<vertex x="2.235" y="-0.0125"/>
+<vertex x="1.27" y="0.9525"/>
+<vertex x="-1.27" y="0.9525"/>
+<vertex x="-2.235" y="-0.0125"/>
 </polygon>
 <contactref element="H2" pad="B3,2"/>
 <contactref element="H1" pad="B3,2"/>
 <contactref element="J1" pad="3"/>
-<wire x1="6" y1="0" x2="0" y2="6" width="0" layer="19" extent="1-1"/>
 </signal>
 </signals>
@@
 <mfgpreviewcolor name="substratecolor" color="0xFF786E46"/>
 </mfgpreviewcolors>
+<errors>
+</errors>
 </board>
 </drawing>

Commit message: updated piezoPCB singledisk for better actuation #bugfix
Parts:
- added GND, GND0, PZ+: TPTP12SQ, PiezoFFC:TP12SQ
- added TP1, TP2, TP3: TPTP16R_LONG, PiezoFFC:TP16R_LONG
- moved PZ1 0.32 mm to (0.00, 0.32)
Connections:
- net GND: now also GND.TP, GND0.TP, TP2.TP, TP3.TP
- net PZ+: now also PZ+.TP, TP1.TP
Routing:
- net PZ+: track 11.2 -> 18.8 mm
Other:
- board size 21.6 x 19 mm -> 21.6 x 18.4 mm
