File: Hardware/Eagle_Files/PiezoDisk-PCB/Pyr0-Piezo_Orion_Adapter_v1.0.0.brd (EAGLE design)
At the start: 32 x 43 mm, 5 parts, among them J1 C-GRID-02-70553

Commit message: Updated Orion Adapter PCB with 3-pin for PZDetect #featureadd
Parts:
- added U$5, U$6: (no value), PiezoFFC:LOGO-PYR0BALL-SS-6MM
- J1: value C-GRID-02-70553 -> C-GRID-03-70553; device PiezoFFC:70553-02 -> PiezoFFC:70553-03
Connections:
- net GND: now also J1.1, J1.3; no longer J1.2
- net PIEZO_OUT: now also J1.2; no longer J1.1
Routing:
- net PIEZO_OUT: track 44.8 -> 43.5 mm
Changed lines of the file:
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@@
 <?xml version="1.0" encoding="utf-8"?>
 <!DOCTYPE eagle SYSTEM "eagle.dtd">
-<eagle version="9.5.1">
+<eagle version="9.6.2">
 <drawing>
 <settings>
@@
 </layers>
 <board>
-<fusionsync huburn="a.cGVyc29uYWw6dWUyYTEyMDdh" projecturn="a.cGVyc29uYWw6dWUyYTEyMDdhIzIwMTgxMTI5MTYyOTY3NjMx" f3durn="urn:adsk.wipprod:dm.lineage:C-HqNGddSr69jsuWzaZLjw" pcbguid="d70e268b-0e59-4e39-8411-c2538c8efa20" lastpulledtime="" lastsyncedchangeguid="1387d4e4-ab54-07f4-efe3-34061caa9246"/>
+<fusionsync huburn="a.cGVyc29uYWw6dWUyYTEyMDdh" projecturn="a.cGVyc29uYWw6dWUyYTEyMDdhIzIwMTgxMTI5MTYyOTY3NjMx" f3durn="urn:adsk.wipprod:dm.lineage:C-HqNGddSr69jsuWzaZLjw" pcbguid="d70e268b-0e59-4e39-8411-c2538c8efa20" lastpulledtime="" lastsyncedchangeguid="1387d4e4-ab54-07f4-efe3-34061caa9246" latestrevisionid="" lastsyncedrevisionid="" lastboardhashguid="4dd1147d-6ac1-21f4-3d57-ac485abd95b7" lastpushedtime="2020-09-15T17:37:29Z" linktopcb3d="false"/>
 <plain>
 <wire x1="-14" y1="-27" x2="14" y2="-27" width="0" layer="20"/>
@@
 <hole x="-13" y="13" drill="3.2"/>
 <text x="-9" y="14" size="0.8128" layer="21">Pyr0-Piezo Orion Adapter v1.0.0</text>
-<text x="-10" y="-17" size="1.016" layer="21">https://docs.pyroballpcbs.com</text>
+<text x="-10" y="-16" size="1.016" layer="21">https://docs.pyroballpcbs.com</text>
 </plain>
 <attributes>
@@
 <element name="U$3" library="PiezoFFC" library_urn="urn:adsk.eagle:library:6897166" package="PIEZO-DISK-12MM" package3d_urn="urn:adsk.eagle:package:14393959/5" value="PIEZO-DISK12MM" x="-6.5" y="6.5" smashed="yes" rot="R225"/>
 <element name="U$4" library="PiezoFFC" library_urn="urn:adsk.eagle:library:6897166" package="PIEZO-DISK-12MM" package3d_urn="urn:adsk.eagle:package:14393959/5" value="PIEZO-DISK12MM" x="6.5" y="6.5" smashed="yes" rot="R135"/>
-<element name="J1" library="PiezoFFC" library_urn="urn:adsk.eagle:library:6897166" package="70553-02" package3d_urn="urn:adsk.eagle:package:7346257/2" value="C-GRID-02-70553" x="-1" y="-22" smashed="yes" rot="R90">
+<element name="J1" library="PiezoFFC" library_urn="urn:adsk.eagle:library:6897166" package="70553-03" package3d_urn="urn:adsk.eagle:package:7346260/2" value="C-GRID-03-70553" x="-1" y="-22" smashed="yes" rot="R90">
 <attribute name="MF" value="MOLEX" x="-1" y="-22" size="1.778" layer="27" rot="R90" display="off"/>
 <attribute name="MPN" value="" x="-1" y="-22" size="1.778" layer="27" rot="R90" display="off"/>
@@
 <attribute name="OC_NEWARK" value="unknown" x="-1" y="-22" size="1.778" layer="27" rot="R90" display="off"/>
 </element>
+<element name="U$5" library="PiezoFFC" library_urn="urn:adsk.eagle:library:6897166" package="LOGO-PYR0BALL-SS-6MM" package3d_urn="urn:adsk.eagle:package:14743021/2" value="" x="-12.7" y="-21.9" smashed="yes"/>
+<element name="U$6" library="PiezoFFC" library_urn="urn:adsk.eagle:library:6897166" package="LOGO-PYR0BALL-SS-6MM" package3d_urn="urn:adsk.eagle:package:14743021/2" value="" x="12.8" y="-23.5" smashed="yes" rot="R180"/>
 </elements>
 <signals>
@@
 <contactref element="U$4" pad="GND3"/>
 <contactref element="U$4" pad="GND4"/>
-<contactref element="J1" pad="2"/>
 <polygon width="0.1524" layer="16">
 <vertex x="-14" y="-27"/>
@@
 <vertex x="14" y="-27"/>
 </polygon>
+<contactref element="J1" pad="1"/>
+<contactref element="J1" pad="3"/>
 </signal>
 <signal name="PIEZO_OUT">
@@
 <contactref element="U$1" pad="PZ+" route="any" routetag="G$1.PZ+"/>
 <contactref element="U$4" pad="PZ+" route="any" routetag="G$1.PZ+"/>
-<contactref element="J1" pad="1"/>
-<wire x1="6.62" y1="-23.27" x2="2.54" y2="-23.27" width="0.4064" layer="16"/>
-<wire x1="2.54" y1="-23.27" x2="0" y2="-20.73" width="0.4064" layer="16" curve="-90"/>
-<wire x1="0" y1="-20.73" x2="0" y2="-4" width="0.4064" layer="16"/>
 <wire x1="-6.5" y1="-6.5" x2="-2.9" y2="-2.9" width="0.4064" layer="16"/>
 <wire x1="-6.5" y1="6.5" x2="-2.9" y2="2.9" width="0.4064" layer="16"/>
 <wire x1="6.5" y1="6.5" x2="2.9" y2="2.9" width="0.4064" layer="16"/>
 <wire x1="6.5" y1="-6.5" x2="2.9" y2="-2.9" width="0.4064" layer="16"/>
+<contactref element="J1" pad="2"/>
+<wire x1="6.62" y1="-22" x2="2.54" y2="-22" width="0.508" layer="16"/>
+<wire x1="2.54" y1="-22" x2="0" y2="-19.46" width="0.508" layer="16" curve="-90"/>
+<wire x1="0" y1="-19.46" x2="0" y2="-4" width="0.508" layer="16"/>
 <wire x1="0" y1="-4" x2="-2.9" y2="-2.9" width="0" layer="19" extent="16-16"/>
 <wire x1="2.9" y1="-2.9" x2="0" y2="-4" width="0" layer="19" extent="16-16"/>
