File: Hardware/Eagle_Files/PiezoDisk-PCB/Pyr0-Piezo_Orion_Adapter_v1.0.0.sch (EAGLE design)
At the start: 5 parts, among them J1 C-GRID-02-70553

Commit message: Updated Orion Adapter PCB with 3-pin for PZDetect #featureadd
Parts:
- J1: value C-GRID-02-70553 -> C-GRID-03-70553; device PiezoFFC:C-GRID-02-70553 -> PiezoFFC:C-GRID-03-70553
Connections:
- net GND: now also J1-1.S, J1-3.S; no longer J1-2.S
- net PIEZO_OUT: now also J1-2.S; no longer J1-1.S
Other:
- moved on the sheet: J1-1, J1-2
Changed lines of the file:
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@@
 <?xml version="1.0" encoding="utf-8"?>
 <!DOCTYPE eagle SYSTEM "eagle.dtd">
-<eagle version="9.5.1">
+<eagle version="9.6.2">
 <drawing>
 <settings>
@@
 <setting verticaltext="up"/>
 </settings>
-<grid distance="0.1" unitdist="inch" unit="inch" style="lines" multiple="1" display="no" altdistance="0.01" altunitdist="inch" altunit="inch"/>
+<grid distance="1.27" unitdist="mm" unit="mm" style="lines" multiple="1" display="no" altdistance="0.01" altunitdist="inch" altunit="inch"/>
 <layers>
 <layer number="1" name="Top" color="4" fill="1" visible="no" active="no"/>
@@
 <part name="U$4" library="PiezoFFC" library_urn="urn:adsk.eagle:library:6897166" deviceset="PIEZO-DISK" device="12MM" package3d_urn="urn:adsk.eagle:package:14393959/5"/>
 <part name="GND1" library="supply1" library_urn="urn:adsk.eagle:library:371" deviceset="GND" device=""/>
-<part name="J1" library="PiezoFFC" library_urn="urn:adsk.eagle:library:6897166" deviceset="C-GRID-02" device="-70553" package3d_urn="urn:adsk.eagle:package:7346257/2"/>
+<part name="J1" library="PiezoFFC" library_urn="urn:adsk.eagle:library:6897166" deviceset="C-GRID-03" device="-70553" package3d_urn="urn:adsk.eagle:package:7346260/2"/>
 </parts>
 <sheets>
@@
 <attribute name="VALUE" x="30.48" y="-12.7" size="1.778" layer="96"/>
 </instance>
-<instance part="J1" gate="-2" x="73.66" y="10.16" smashed="yes">
-<attribute name="NAME" x="76.2" y="9.398" size="1.524" layer="95"/>
-</instance>
-<instance part="J1" gate="-1" x="73.66" y="12.7" smashed="yes">
-<attribute name="NAME" x="76.2" y="11.938" size="1.524" layer="95"/>
-<attribute name="VALUE" x="72.898" y="14.097" size="1.778" layer="96"/>
+<instance part="J1" gate="-2" x="76.2" y="13.97" smashed="yes">
+<attribute name="NAME" x="78.74" y="13.208" size="1.524" layer="95"/>
+</instance>
+<instance part="J1" gate="-1" x="76.2" y="11.43" smashed="yes">
+<attribute name="NAME" x="78.74" y="10.668" size="1.524" layer="95"/>
+<attribute name="VALUE" x="77.978" y="15.367" size="1.778" layer="96"/>
+</instance>
+<instance part="J1" gate="-3" x="76.2" y="8.89" smashed="yes">
+<attribute name="NAME" x="78.74" y="8.128" size="1.524" layer="95"/>
 </instance>
 </instances>
@@
 <wire x1="55.88" y1="0" x2="38.1" y2="0" width="0.1524" layer="91"/>
 <junction x="38.1" y="0"/>
-<pinref part="J1" gate="-2" pin="S"/>
-<wire x1="71.12" y1="10.16" x2="71.12" y2="0" width="0.1524" layer="91"/>
 <wire x1="71.12" y1="0" x2="55.88" y2="0" width="0.1524" layer="91"/>
 <junction x="55.88" y="0"/>
+<wire x1="71.12" y1="0" x2="71.12" y2="8.89" width="0.1524" layer="91"/>
+<pinref part="J1" gate="-1" pin="S"/>
+<wire x1="71.12" y1="8.89" x2="71.12" y2="11.43" width="0.1524" layer="91"/>
+<wire x1="71.12" y1="11.43" x2="73.66" y2="11.43" width="0.1524" layer="91"/>
+<pinref part="J1" gate="-3" pin="S"/>
+<wire x1="73.66" y1="8.89" x2="71.12" y2="8.89" width="0.1524" layer="91"/>
+<junction x="71.12" y="8.89"/>
 </segment>
 </net>
@@
 <wire x1="53.34" y1="22.86" x2="33.02" y2="22.86" width="0.1524" layer="91"/>
 <label x="33.02" y="30.48" size="1.778" layer="95" rot="R90"/>
-<pinref part="J1" gate="-1" pin="S"/>
-<wire x1="71.12" y1="12.7" x2="71.12" y2="22.86" width="0.1524" layer="91"/>
 <wire x1="71.12" y1="22.86" x2="53.34" y2="22.86" width="0.1524" layer="91"/>
 <junction x="53.34" y="22.86"/>
+<wire x1="71.12" y1="22.86" x2="71.12" y2="13.97" width="0.1524" layer="91"/>
+<pinref part="J1" gate="-2" pin="S"/>
+<wire x1="71.12" y1="13.97" x2="73.66" y2="13.97" width="0.1524" layer="91"/>
 </segment>
 </net>
