File: Hardware/Eagle_Files/EzPzEffector/EzPz-Effector_v2.3.1.brd (EAGLE design)
At the start: 90.2 x 85.9 mm, 67 parts, among them J1 C-GRID-06-70543, U1 ATMEGA328PTQFP-32, U2 LM317DCYSOT223, U3 LM2902PT

Commit message: Fixed Heater trace to ground on EzPzEffector #bugfix
Connections:
- new net HE0-: HEATER.4, V/TH_IN.2
- net GND: no longer HEATER.4, V/TH_IN.2
Routing:
- net HE0-: track 0.00 -> 33.1 mm
Changed lines of the file:
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@@
 <via x="-24" y="13" extent="1-16" drill="0.35"/>
 <via x="-26.5" y="13" extent="1-16" drill="0.35"/>
-<contactref element="HEATER" pad="4"/>
-<contactref element="V/TH_IN" pad="2"/>
 <via x="-4.5" y="26.6" extent="1-16" drill="0.35"/>
 <via x="-12.25" y="25" extent="1-16" drill="0.35"/>
@@
 <wire x1="6.8048" y1="-26.6952" x2="4.98" y2="-28.52" width="0.1524" layer="1"/>
 </signal>
+<signal name="HE0-">
+<contactref element="HEATER" pad="4"/>
+<contactref element="V/TH_IN" pad="2"/>
+<wire x1="27.06843125" y1="-17.943653125" x2="27" y2="-18.012084375" width="0.8128" layer="1"/>
+<wire x1="27" y1="-18.012084375" x2="27" y2="-20.25715" width="0.8128" layer="1"/>
+<wire x1="24.5602" y1="-22.69695" x2="24.5602" y2="-23.697425" width="0.8128" layer="1"/>
+<wire x1="24.5602" y1="-23.697425" x2="20.582425" y2="-27.6752" width="0.8128" layer="1"/>
+<wire x1="20.582425" y1="-27.6752" x2="12.82323125" y2="-27.6752" width="0.8128" layer="1"/>
+<wire x1="12.82323125" y1="-27.6752" x2="11.20823125" y2="-26.0602" width="0.8128" layer="1"/>
+<wire x1="2.44" y1="-28.31" x2="2.44" y2="-29.25" width="0.8128" layer="1"/>
+<wire x1="27" y1="-20.25715" x2="24.5602" y2="-22.69695" width="0.8128" layer="1"/>
+<wire x1="11.20823125" y1="-26.0602" x2="4.6898" y2="-26.0602" width="0.8128" layer="1"/>
+<wire x1="4.6898" y1="-26.0602" x2="2.44" y2="-28.31" width="0.8128" layer="1"/>
+</signal>
 </signals>

Commit message: Added bypass jumper to allow powering EzPz direct from heater VCC #featureadd
Parts:
- added BYPASS: C-GRID-02-70543, PiezoFFC:70543-02
Connections:
- net VCC_REG: now also BYPASS.2
- net VIN_12/24: now also BYPASS.1
Routing:
- net VIN_12/24: track 25.9 -> 63.1 mm
- net VCC_REG: track 8.24 -> 20.8 mm
Changed lines of the file:
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@@
 </layers>
 <board>
-<fusionsync huburn="a.cGVyc29uYWw6dWUyYTEyMDdh" projecturn="a.cGVyc29uYWw6dWUyYTEyMDdhIzIwMTgxMTI5MTYyOTY3NjMx" f3durn="urn:adsk.wipprod:dm.lineage:qf6Wlt5RSPWK4r9tDMxusw" pcbguid="" lastpulledtime="2020-08-07T19:55:00Z" lastsyncedchangeguid="" latestrevisionid="8016aa98-db26-41a4-8108-f24e8ca86df1" lastsyncedrevisionid="8016aa98-db26-41a4-8108-f24e8ca86df1" lastboardhashguid="bd6e886d-fb3e-9dc2-1f69-de54a29e028e" lastpushedtime="2020-08-08T00:21:21Z" linktopcb3d="true"/>
+<fusionsync huburn="a.cGVyc29uYWw6dWUyYTEyMDdh" projecturn="a.cGVyc29uYWw6dWUyYTEyMDdhIzIwMTgxMTI5MTYyOTY3NjMx" f3durn="urn:adsk.wipprod:dm.lineage:qf6Wlt5RSPWK4r9tDMxusw" pcbguid="" lastpulledtime="2020-08-07T19:55:00Z" lastsyncedchangeguid="" latestrevisionid="d26613a3-daa6-4b98-b176-9e7509ba51ed" lastsyncedrevisionid="d26613a3-daa6-4b98-b176-9e7509ba51ed" lastboardhashguid="81052898-e767-1147-31a1-72f8a9b9b313" lastpushedtime="2020-09-14T19:50:01Z" linktopcb3d="true"/>
 <plain>
 <hole x="-8.765" y="15.493" drill="3.2"/>
@@
 <element name="U$5" library="PiezoFFC" library_urn="urn:adsk.eagle:library:6897166" package="OSHW_8MM" value="" x="31.5" y="-1.75" smashed="yes"/>
 <element name="U$6" library="PiezoFFC" library_urn="urn:adsk.eagle:library:6897166" package="OSHW_8MM" value="" x="10.75" y="36" smashed="yes" rot="MR0"/>
+<element name="BYPASS" library="PiezoFFC" library_urn="urn:adsk.eagle:library:6897166" package="70543-02" package3d_urn="urn:adsk.eagle:package:7346256/2" value="C-GRID-02-70543" x="-25.5" y="-30.25" smashed="yes" rot="R120">
+<attribute name="MF" value="MOLEX" x="-25.5" y="-30.25" size="1.778" layer="27" rot="R120" display="off"/>
+<attribute name="MPN" value="" x="-25.5" y="-30.25" size="1.778" layer="27" rot="R120" display="off"/>
+<attribute name="NAME" x="-21.07779375" y="-32.82948125" size="1.016" layer="25" ratio="10" rot="R210"/>
+<attribute name="OC_FARNELL" value="unknown" x="-25.5" y="-30.25" size="1.778" layer="27" rot="R120" display="off"/>
+<attribute name="OC_NEWARK" value="unknown" x="-25.5" y="-30.25" size="1.778" layer="27" rot="R120" display="off"/>
+</element>
 </elements>
 <signals>
@@
 <wire x1="-27" y1="-18.25" x2="-26.153725" y2="-18.7729" width="0.4064" layer="1"/>
 <via x="-28.75" y="-17.75" extent="1-16" drill="0.35"/>
+<contactref element="BYPASS" pad="2"/>
+<wire x1="-26.153725" y1="-18.7729" x2="-23" y2="-24.5" width="0.8128" layer="1"/>
+<wire x1="-23" y1="-24.5" x2="-24" y2="-28" width="0.8128" layer="1"/>
+<wire x1="-24" y1="-28" x2="-26.135" y2="-29.150146875" width="0.8128" layer="1"/>
 </signal>
 <signal name="TTL_RXD">
@@
 <wire x1="-32.265228125" y1="-7.520571875" x2="-33.594890625" y2="-5.129909375" width="0.3048" layer="1"/>
 <wire x1="-33.594890625" y1="-5.129909375" x2="-33.859" y2="-5.129909375" width="0.3048" layer="1"/>
-<wire x1="-32.265228125" y1="-7.520571875" x2="-28.75" y2="-13.5" width="0.4064" layer="1"/>
-<wire x1="-28.75" y1="-13.5" x2="-29.0172" y2="-14.4326875" width="0.4064" layer="1"/>
+<wire x1="-28.928215625" y1="-14.122103125" x2="-32.265228125" y2="-8.445821875" width="0.4064" layer="1"/>
+<wire x1="-32.265228125" y1="-7.520571875" x2="-32.265228125" y2="-8.445821875" width="0.4064" layer="1"/>
+<wire x1="-28.928215625" y1="-14.122103125" x2="-29.0172" y2="-14.4326875" width="0.4064" layer="1"/>
 </signal>
 <signal name="AMP_VCC">
@@
 <wire x1="21.25" y1="-29.25" x2="10.06" y2="-29.25" width="0.8128" layer="1"/>
 <wire x1="26.1608" y1="-24.3392" x2="21.25" y2="-29.25" width="0.8128" layer="1"/>
+<contactref element="BYPASS" pad="1"/>
+<wire x1="10.06" y1="-29.25" x2="10.06" y2="-30.19" width="0.8128" layer="1"/>
+<wire x1="-22.75" y1="-32" x2="-23.901296875" y2="-30.848703125" width="0.8128" layer="1"/>
+<wire x1="-23.901296875" y1="-30.848703125" x2="-24.865" y2="-31.34985" width="0.8128" layer="1"/>
+<wire x1="10.06" y1="-30.19" x2="8.25" y2="-32" width="0.8128" layer="1"/>
+<wire x1="8.25" y1="-32" x2="-22.75" y2="-32" width="0.8128" layer="1"/>
 </signal>
 <signal name="TH1">

Commit message: added additional mounting holes on EzPzEffector for accessories #featureadd
Parts:
- moved U$1 3.91 mm to (-20.8, 17.8)
- moved INT 2.76 mm to (-27.7, 14.4)
- moved H2 1.25 mm to (-29.7, -17.1)
- moved H3 1.25 mm to (29.7, -17.1)
Routing:
- net Z_TRG: track 33.4 -> 35.4 mm
Changed lines of the file:
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@@
 <wire x1="-24.75" y1="37.75" x2="-45" y2="3" width="0.1524" layer="20"/>
 <wire x1="-19.5" y1="-40.75" x2="19.5" y2="-40.75" width="0.1524" layer="20"/>
-<text x="-0.25" y="-39" size="1.4224" layer="21" align="bottom-center">https://docs.pyroballpcbs.com</text>
-<text x="-11.5" y="-36.5" size="1.778" layer="21">EzPz-Effector v2.3.1</text>
+<text x="-0.25" y="37.25" size="1.4224" layer="21" align="bottom-center">https://docs.pyroballpcbs.com</text>
+<text x="-11.5" y="-34.75" size="1.778" layer="21">EzPz-Effector v2.3.1</text>
 <wire x1="-20.6101" y1="-9.3014" x2="-20.6208" y2="-8.8734" width="0.1016" layer="20"/>
 <wire x1="-20.6208" y1="-8.8734" x2="-20.5941" y2="-8.4461" width="0.1016" layer="20"/>
@@
 <wire x1="21.142946875" y1="5.453365625" x2="26.7721125" y2="8.703365625" width="0.1524" layer="21"/>
 <wire x1="22.267946875" y1="3.504809375" x2="27.8971125" y2="6.754809375" width="0.1524" layer="21"/>
+<hole x="0" y="-37" drill="3.25"/>
+<hole x="32.476" y="18.75" drill="3.25"/>
+<hole x="-32.476" y="18.75" drill="3.25"/>
 </plain>
 <attributes>
@@
 <attribute name="NAME" x="0.765" y="27.205" size="0.8128" layer="26" font="vector" rot="MR180"/>
 </element>
-<element name="INT" library="testpad" library_urn="urn:adsk.eagle:library:385" package="TP06R" package3d_urn="urn:adsk.eagle:package:27954/1" value="TPTP06R" x="-27.91" y="17.2" smashed="yes" rot="R90">
-<attribute name="NAME" x="-28.3101" y="16.9" size="0.6096" layer="25" rot="R90"/>
-<attribute name="POPULARITY" value="1" x="14" y="42.6" size="1.778" layer="27" rot="R90" display="off"/>
-<attribute name="TP_SIGNAL_NAME" value="" x="-26.005" y="17.2" size="1" layer="37" rot="R90"/>
-<attribute name="VALUE" x="-27.529" y="16.946" size="0.0254" layer="27" rot="R90"/>
+<element name="INT" library="testpad" library_urn="urn:adsk.eagle:library:385" package="TP06R" package3d_urn="urn:adsk.eagle:package:27954/1" value="TPTP06R" x="-27.66" y="14.45" smashed="yes" rot="R90">
+<attribute name="NAME" x="-28.0601" y="14.15" size="0.6096" layer="25" rot="R90"/>
+<attribute name="POPULARITY" value="1" x="14.25" y="39.85" size="1.778" layer="27" rot="R90" display="off"/>
+<attribute name="TP_SIGNAL_NAME" value="" x="-25.755" y="14.45" size="1" layer="37" rot="R90"/>
+<attribute name="VALUE" x="-27.529" y="14.446" size="0.0254" layer="27" rot="R90"/>
 </element>
 <element name="LED" library="PiezoFFC" library_urn="urn:adsk.eagle:library:6897166" package="0606_LED" package3d_urn="urn:adsk.eagle:package:9308796/3" value="LED-RGB-COM_ANO0606" x="-32.895953125" y="-26.128159375" smashed="yes" rot="MR150">
@@
 <attribute name="NAME" x="-23.4" y="33.81" size="1.27" layer="21"/>
 </element>
-<element name="H2" library="PiezoFFC" library_urn="urn:adsk.eagle:library:6897166" package="EFFECTOR-45MM-ROD" package3d_urn="urn:adsk.eagle:package:22453934/1" value="EFFECTOR-ROD-MOUNT" x="-28.579" y="-16.5" smashed="yes" rot="R120">
-<attribute name="NAME" x="-16.428559375" y="-36.40204375" size="1.27" layer="21" rot="R120"/>
-</element>
-<element name="H3" library="PiezoFFC" library_urn="urn:adsk.eagle:library:6897166" package="EFFECTOR-45MM-ROD" package3d_urn="urn:adsk.eagle:package:22453934/1" value="EFFECTOR-ROD-MOUNT" x="28.579" y="-16.5" smashed="yes" rot="R240">
-<attribute name="NAME" x="39.828559375" y="4.092046875" size="1.27" layer="21" rot="R240"/>
+<element name="H2" library="PiezoFFC" library_urn="urn:adsk.eagle:library:6897166" package="EFFECTOR-45MM-ROD" package3d_urn="urn:adsk.eagle:package:22453934/1" value="EFFECTOR-ROD-MOUNT" x="-29.661" y="-17.125" smashed="yes" rot="R120">
+<attribute name="NAME" x="-17.510559375" y="-37.02704375" size="1.27" layer="21" rot="R120"/>
+</element>
+<element name="H3" library="PiezoFFC" library_urn="urn:adsk.eagle:library:6897166" package="EFFECTOR-45MM-ROD" package3d_urn="urn:adsk.eagle:package:22453934/1" value="EFFECTOR-ROD-MOUNT" x="29.661" y="-17.125" smashed="yes" rot="R240">
+<attribute name="NAME" x="40.910559375" y="3.467046875" size="1.27" layer="21" rot="R240"/>
 </element>
 <element name="U1" library="PiezoFFC" library_urn="urn:adsk.eagle:library:6897166" package="QFP80P900X900X120-32N" package3d_urn="urn:adsk.eagle:package:22517142/2" value="ATMEGA328PTQFP-32" x="-22" y="20" smashed="yes" rot="R90">
@@
 <attribute name="OC_NEWARK" value="unknown" x="6.25" y="-29.25" size="1.778" layer="27" rot="R180" display="off"/>
 </element>
-<element name="U$1" library="PiezoFFC" library_urn="urn:adsk.eagle:library:6897166" package="LOGO-PYR0BALL-SS-20MM" package3d_urn="urn:adsk.eagle:package:5522046/2" value="" x="-23.75" y="20.25" smashed="yes" rot="MR0"/>
+<element name="U$1" library="PiezoFFC" library_urn="urn:adsk.eagle:library:6897166" package="LOGO-PYR0BALL-SS-20MM" package3d_urn="urn:adsk.eagle:package:5522046/2" value="" x="-20.75" y="17.75" smashed="yes" rot="MR0"/>
 <element name="U$2" library="PiezoFFC" library_urn="urn:adsk.eagle:library:6897166" package="LOGO-PYR0BALL-SS-6MM" package3d_urn="urn:adsk.eagle:package:14743021/2" value="" x="14.5" y="8.75" smashed="yes"/>
 <element name="U$3" library="PiezoFFC" library_urn="urn:adsk.eagle:library:6897166" package="LOGO-PYR0BALL-SS-6MM" package3d_urn="urn:adsk.eagle:package:14743021/2" value="" x="-15" y="8.25" smashed="yes" rot="R120"/>
@@
 <attribute name="MF" value="MOLEX" x="-25.5" y="-30.25" size="1.778" layer="27" rot="R120" display="off"/>
 <attribute name="MPN" value="" x="-25.5" y="-30.25" size="1.778" layer="27" rot="R120" display="off"/>
-<attribute name="NAME" x="-21.07779375" y="-32.82948125" size="1.016" layer="25" ratio="10" rot="R210"/>
+<attribute name="NAME" x="-20.82779375" y="-32.82948125" size="1.016" layer="25" ratio="10" rot="R210"/>
 <attribute name="OC_FARNELL" value="unknown" x="-25.5" y="-30.25" size="1.778" layer="27" rot="R120" display="off"/>
 <attribute name="OC_NEWARK" value="unknown" x="-25.5" y="-30.25" size="1.778" layer="27" rot="R120" display="off"/>
@@
 <contactref element="U1" pad="27"/>
 <wire x1="-26.3" y1="21.2" x2="-26.5" y2="21" width="0.1524" layer="1"/>
-<wire x1="-26.5" y1="21" x2="-27.25" y2="21" width="0.1524" layer="1"/>
-<wire x1="-27.25" y1="21" x2="-27.75" y2="20.5" width="0.1524" layer="1"/>
-<wire x1="-27.75" y1="20.5" x2="-27.75" y2="20.43105625" width="0.1524" layer="1"/>
-<wire x1="-27.75" y1="20.43105625" x2="-28.8048" y2="19.37625625" width="0.1524" layer="1"/>
+<wire x1="-27.25" y1="21" x2="-26.5" y2="21" width="0.1524" layer="1"/>
 <wire x1="-37.3048" y1="-7.6262625" x2="-34.46553125" y2="-10.46553125" width="0.1524" layer="1"/>
-<wire x1="-28.8048" y1="5.4452" x2="-37.3048" y2="-3.0548" width="0.1524" layer="1"/>
+<wire x1="-37.3048" y1="-3.0548" x2="-28.8048" y2="5.4452" width="0.1524" layer="1"/>
 <wire x1="-37.3048" y1="-3.0548" x2="-37.3048" y2="-7.6262625" width="0.1524" layer="1"/>
-<wire x1="-28.8048" y1="19.37625625" x2="-28.8048" y2="5.4452" width="0.1524" layer="1"/>
 <wire x1="-34.46553125" y1="-10.46553125" x2="-34.46553125" y2="-11.745759375" width="0.1524" layer="1"/>
 <wire x1="-34.46553125" y1="-11.745759375" x2="-35.4968" y2="-12.7770375" width="0.1524" layer="16"/>
 <via x="-34.46553125" y="-11.745759375" extent="1-16" drill="0.35"/>
+<wire x1="-28.8048" y1="5.4452" x2="-28.8048" y2="16.0073125" width="0.1524" layer="1"/>
+<wire x1="-28.8048" y1="16.0073125" x2="-27.5834" y2="17.2287125" width="0.1524" layer="1"/>
+<wire x1="-27.5834" y1="20.6666" x2="-27.25" y2="21" width="0.1524" layer="1"/>
+<wire x1="-27.5834" y1="17.2287125" x2="-27.5834" y2="20.6666" width="0.1524" layer="1"/>
 </signal>
 <signal name="SCL">
@@
 <contactref element="U1" pad="28"/>
 <wire x1="-26.3" y1="20.4" x2="-26.45" y2="20.25" width="0.1524" layer="1"/>
-<wire x1="-26.45" y1="20.25" x2="-27.5" y2="20.25" width="0.1524" layer="1"/>
-<wire x1="-27.5" y1="20.25" x2="-28.5" y2="19.25" width="0.1524" layer="1"/>
-<wire x1="-28.5" y1="5.3189375" x2="-37" y2="-3.1810625" width="0.1524" layer="1"/>
+<wire x1="-27" y1="20.25" x2="-26.45" y2="20.25" width="0.1524" layer="1"/>
+<wire x1="-37" y1="-3.1810625" x2="-28.5" y2="5.3189375" width="0.1524" layer="1"/>
 <wire x1="-37" y1="-3.1810625" x2="-37" y2="-7.5" width="0.1524" layer="1"/>
-<wire x1="-28.5" y1="19.25" x2="-28.5" y2="5.3189375" width="0.1524" layer="1"/>
 <wire x1="-33.25" y1="-13.99993125" x2="-34.2268" y2="-14.976740625" width="0.1524" layer="16"/>
 <wire x1="-37" y1="-7.5" x2="-33.25" y2="-11.25" width="0.1524" layer="1"/>
 <wire x1="-33.25" y1="-11.25" x2="-33.25" y2="-13.99993125" width="0.1524" layer="1"/>
 <via x="-33.25" y="-13.99993125" extent="1-16" drill="0.35"/>
+<wire x1="-28.5" y1="5.3189375" x2="-28.5" y2="15.88105625" width="0.1524" layer="1"/>
+<wire x1="-28.5" y1="15.88105625" x2="-27.2786" y2="17.10245625" width="0.1524" layer="1"/>
+<wire x1="-27.2786" y1="19.9714" x2="-27" y2="20.25" width="0.1524" layer="1"/>
+<wire x1="-27.2786" y1="17.10245625" x2="-27.2786" y2="19.9714" width="0.1524" layer="1"/>
 </signal>
 <signal name="Z_TRG">
@@
 <wire x1="-22.8932" y1="22.1432" x2="-22.8932" y2="18.8568" width="0.1524" layer="1"/>
 <wire x1="-24.55" y1="17.2" x2="-26" y2="17.2" width="0.1524" layer="1"/>
+<wire x1="-26" y1="17.2" x2="-26.75" y2="17.2" width="0.1524" layer="1"/>
 <wire x1="-26" y1="17.2" x2="-26.3" y2="17.2" width="0.1524" layer="1"/>
 <wire x1="-24.0714" y1="23.3214" x2="-22.8932" y2="22.1432" width="0.1524" layer="1"/>
 <wire x1="-22.8932" y1="18.8568" x2="-24.55" y2="17.2" width="0.1524" layer="1"/>
-<wire x1="-27.91" y1="17.2" x2="-26" y2="17.2" width="0.1524" layer="1"/>
+<wire x1="-27.66" y1="16.29" x2="-26.75" y2="17.2" width="0.1524" layer="1"/>
+<wire x1="-27.66" y1="16.29" x2="-27.66" y2="14.45" width="0.1524" layer="1"/>
 </signal>
 <signal name="PZ+">
